File: template/template.sch (KiCad schematic (older format))
At the start: 13 parts, among them P1 Power, P10 CONN_01X04, P11 CONN_01X04, P12 CONN_01X03, P13 CONN_02X05, P14 CONN_01X04, P2 Analog, P3 Digital, P4 Digital, P9 CONN_01X04

Commit message: no message
Parts:
- R1: value R -> 47k
- R2: value R -> 10k
Changed lines of the file:
@@
 P 5450 3250
 F 0 "R1" V 5530 3250 40  0000 C CNN
-F 1 "R" V 5457 3251 40  0000 C CNN
+F 1 "47k" V 5457 3251 40  0000 C CNN
 F 2 "RP_KiCAD_Libs:C0603K" V 5380 3250 30  0001 C CNN
 F 3 "" H 5450 3250 30  0000 C CNN
@@
 P 5450 3650
 F 0 "R2" V 5530 3650 40  0000 C CNN
-F 1 "R" V 5457 3651 40  0000 C CNN
+F 1 "10k" V 5457 3651 40  0000 C CNN
 F 2 "RP_KiCAD_Libs:C0603K" V 5380 3650 30  0001 C CNN
 F 3 "" H 5450 3650 30  0000 C CNN

Commit message: no message
Parts:
- added C1, C2: C, RP_KiCAD_Libs:C1206K, symbol C
- added U1, U2: MC78L05ACD, Housings_SOIC:SOIJ-8_5.3x5.3mm_Pitch1.27mm, symbol MC78L05ACD
Connections:
- net labels added: 5V_rerays
- wire segments 56 -> 70
Changed lines of the file:
@@
 LIBS:special
 LIBS:transistors
+LIBS:regul
 LIBS:template-cache
 EELAYER 25 0
@@
 	0    1    1    0
 $EndComp
-$Comp
-L +5V #PWR08
-U 1 1 570CE43B
-P 3900 1750
-F 0 "#PWR08" H 3900 1840 20  0001 C CNN
-F 1 "+5V" H 3900 1840 30  0000 C CNN
-F 2 "" H 3900 1750 60  0000 C CNN
-F 3 "" H 3900 1750 60  0000 C CNN
-	1    3900 1750
-	0    -1   -1   0
-$EndComp
-$Comp
-L +5V #PWR09
-U 1 1 570CE7C0
-P 3900 2400
-F 0 "#PWR09" H 3900 2490 20  0001 C CNN
-F 1 "+5V" H 3900 2490 30  0000 C CNN
-F 2 "" H 3900 2400 60  0000 C CNN
-F 3 "" H 3900 2400 60  0000 C CNN
-	1    3900 2400
-	0    -1   -1   0
-$EndComp
-$Comp
-L +5V #PWR010
-U 1 1 570CE7EC
-P 3900 3000
-F 0 "#PWR010" H 3900 3090 20  0001 C CNN
-F 1 "+5V" H 3900 3090 30  0000 C CNN
-F 2 "" H 3900 3000 60  0000 C CNN
-F 3 "" H 3900 3000 60  0000 C CNN
-	1    3900 3000
-	0    -1   -1   0
-$EndComp
 Text Label 3900 3100 0    60   ~ 0
 1(Tx)
@@
 $EndComp
 $Comp
-L GND #PWR011
+L GND #PWR08
 U 1 1 570D0C2B
 P 5550 2450
-F 0 "#PWR011" H 5550 2450 30  0001 C CNN
+F 0 "#PWR08" H 5550 2450 30  0001 C CNN
 F 1 "GND" H 5550 2380 30  0001 C CNN
 F 2 "" H 5550 2450 60  0000 C CNN
@@
 PS_EN
 $Comp
-L +5V #PWR012
+L +5V #PWR09
 U 1 1 570D25B2
 P 6800 1300
-F 0 "#PWR012" H 6800 1390 20  0001 C CNN
+F 0 "#PWR09" H 6800 1390 20  0001 C CNN
 F 1 "+5V" H 6800 1390 30  0000 C CNN
 F 2 "" H 6800 1300 60  0000 C CNN
@@
 $EndComp
 $Comp
-L GND #PWR013
+L GND #PWR010
 U 1 1 570D2AEF
 P 6300 1300
-F 0 "#PWR013" H 6300 1300 30  0001 C CNN
+F 0 "#PWR010" H 6300 1300 30  0001 C CNN
 F 1 "GND" H 6300 1230 30  0001 C CNN
 F 2 "" H 6300 1300 60  0000 C CNN
@@
 0(Rx)
 $Comp
-L +5V #PWR014
+L +5V #PWR011
 U 1 1 570D3BC0
 P 7250 2050
-F 0 "#PWR014" H 7250 2140 20  0001 C CNN
+F 0 "#PWR011" H 7250 2140 20  0001 C CNN
 F 1 "+5V" H 7250 2140 30  0000 C CNN
 F 2 "" H 7250 2050 60  0000 C CNN
@@
 USB_DM
 $Comp
-L GND #PWR015
+L GND #PWR012
 U 1 1 570D3E38
 P 7250 2350
-F 0 "#PWR015" H 7250 2350 30  0001 C CNN
+F 0 "#PWR012" H 7250 2350 30  0001 C CNN
 F 1 "GND" H 7250 2280 30  0001 C CNN
 F 2 "" H 7250 2350 60  0000 C CNN
@@
 Vin
 $Comp
-L +5V #PWR016
+L +5V #PWR013
 U 1 1 570E925E
 P 6300 1400
-F 0 "#PWR016" H 6300 1490 20  0001 C CNN
+F 0 "#PWR013" H 6300 1490 20  0001 C CNN
 F 1 "+5V" H 6300 1490 30  0000 C CNN
 F 2 "" H 6300 1400 60  0000 C CNN
@@
 $EndComp
 $Comp
-L GND #PWR017
+L GND #PWR014
 U 1 1 571B0477
 P 6300 3350
-F 0 "#PWR017" H 6300 3350 30  0001 C CNN
+F 0 "#PWR014" H 6300 3350 30  0001 C CNN
 F 1 "GND" H 6300 3280 30  0001 C CNN
 F 2 "" H 6300 3350 60  0000 C CNN
@@
 	5450 3400 5450 3500
 $Comp
-L GND #PWR018
+L GND #PWR015
 U 1 1 572DD85C
 P 5450 3800
-F 0 "#PWR018" H 5450 3800 30  0001 C CNN
+F 0 "#PWR015" H 5450 3800 30  0001 C CNN
 F 1 "GND" H 5450 3730 30  0001 C CNN
 F 2 "" H 5450 3800 60  0000 C CNN
@@
 A2
 NoConn ~ 6800 1400
+Text GLabel 3900 1750 0    60   Input ~ 0
+5V_rerays
+Text GLabel 3900 2400 0    60   Input ~ 0
+5V_rerays
+Text GLabel 3900 3000 0    60   Input ~ 0
+5V_rerays
+Text GLabel 4400 3750 2    60   Input ~ 0
+5V_rerays
+$Comp
+L C C1
+U 1 1 57691EB1
+P 3300 3950
+F 0 "C1" H 3300 4050 40  0000 L CNN
+F 1 "C" H 3306 3865 40  0000 L CNN
+F 2 "RP_KiCAD_Libs:C1206K" H 3338 3800 30  0001 C CNN
+F 3 "" H 3300 3950 60  0000 C CNN
+	1    3300 3950
+	1    0    0    -1
+$EndComp
+$Comp
+L C C2
+U 1 1 57691F24
+P 4300 3950
+F 0 "C2" H 4300 4050 40  0000 L CNN
+F 1 "C" H 4306 3865 40  0000 L CNN
+F 2 "RP_KiCAD_Libs:C1206K" H 4338 3800 30  0001 C CNN
+F 3 "" H 4300 3950 60  0000 C CNN
+	1    4300 3950
+	1    0    0    -1
+$EndComp
+Text Label 3200 3750 2    60   ~ 0
+Vin
+Wire Wire Line
+	4200 3750 4400 3750
+Connection ~ 4300 3750
+$Comp
+L GND #PWR016
+U 1 1 576929F1
+P 3850 4250
+F 0 "#PWR016" H 3850 4250 30  0001 C CNN
+F 1 "GND" H 3850 4180 30  0001 C CNN
+F 2 "" H 3850 4250 60  0000 C CNN
+F 3 "" H 3850 4250 60  0000 C CNN
+	1    3850 4250
+	1    0    0    -1
+$EndComp
+$Comp
+L MC78L05ACD U1
+U 1 1 57692F76
+P 3800 3800
+F 0 "U1" H 3600 4000 40  0000 C CNN
+F 1 "MC78L05ACD" H 3800 4000 40  0000 L CNN
+F 2 "Housings_SOIC:SOIJ-8_5.3x5.3mm_Pitch1.27mm" H 3800 3900 30  0000 C CIN
+F 3 "" H 3800 3800 60  0000 C CNN
+	1    3800 3800
+	1    0    0    -1
+$EndComp
+Wire Wire Line
+	3200 3750 3400 3750
+Connection ~ 3300 3750
+Wire Wire Line
+	3300 4150 4300 4150
+Wire Wire Line
+	3650 4100 3650 4150
+Connection ~ 3650 4150
+Wire Wire Line
+	3750 4100 3750 4150
+Connection ~ 3750 4150
+Wire Wire Line
+	3850 4100 3850 4250
+Connection ~ 3850 4150
+Wire Wire Line
+	3950 4100 3950 4150
+Connection ~ 3950 4150
+Text GLabel 4400 4500 2    60   Input ~ 0
+5V_rerays
+Text Label 3200 4500 2    60   ~ 0
+Vin
+Wire Wire Line
+	4200 4500 4400 4500
+Connection ~ 4300 4500
+$Comp
+L GND #PWR017
+U 1 1 5769379B
+P 3850 5000
+F 0 "#PWR017" H 3850 5000 30  0001 C CNN
+F 1 "GND" H 3850 4930 30  0001 C CNN
+F 2 "" H 3850 5000 60  0000 C CNN
+F 3 "" H 3850 5000 60  0000 C CNN
+	1    3850 5000
+	1    0    0    -1
+$EndComp
+$Comp
+L MC78L05ACD U2
+U 1 1 576937A1
+P 3800 4550
+F 0 "U2" H 3600 4750 40  0000 C CNN
+F 1 "MC78L05ACD" H 3800 4750 40  0000 L CNN
+F 2 "Housings_SOIC:SOIJ-8_5.3x5.3mm_Pitch1.27mm" H 3800 4650 30  0000 C CIN
+F 3 "" H 3800 4550 60  0000 C CNN
+	1    3800 4550
+	1    0    0    -1
+$EndComp
+Wire Wire Line
+	3200 4500 3400 4500
+Connection ~ 3300 4500
+Wire Wire Line
+	3300 4900 4300 4900
+Wire Wire Line
+	3650 4850 3650 4900
+Connection ~ 3650 4900
+Wire Wire Line
+	3750 4850 3750 4900
+Connection ~ 3750 4900
+Wire Wire Line
+	3850 4850 3850 5000
+Connection ~ 3850 4900
+Wire Wire Line
+	3950 4850 3950 4900
+Connection ~ 3950 4900
 $EndSCHEMATC

Commit message: no message
Parts:
- removed C1, C2: C, RP_KiCAD_Libs:C1206K, symbol C
- removed U1, U2: MC78L05ACD, Housings_SOIC:SOIJ-8_5.3x5.3mm_Pitch1.27mm, symbol MC78L05ACD
- added P5: CONN_01X03, Pin_Headers:Pin_Header_Straight_1x03, symbol CONN_01X03
- added R3: 100, RP_KiCAD_Libs:0207_2f7, symbol R
Connections:
- wire segments 70 -> 56
Other:
- moved on the sheet: P12, SP1

Commit message: no message
Parts:
- P5: footprint Pin_Headers:Pin_Header_Straight_1x03 -> Pin_Headers:Pin_Header_Angled_1x03
Changed lines of the file:
@@
 F 0 "P5" H 5100 5150 50  0000 C CNN
 F 1 "CONN_01X03" V 5200 4950 50  0000 C CNN
-F 2 "Pin_Headers:Pin_Header_Straight_1x03" H 5100 4950 50  0001 C CNN
+F 2 "Pin_Headers:Pin_Header_Angled_1x03" H 5100 4950 50  0001 C CNN
 F 3 "" H 5100 4950 50  0000 C CNN
 	1    5100 4950
