File: KiCAD_Projects/template_test/template_test.sch (KiCad schematic (older format))
At the start: 0 parts

Commit message: no message
Parts:
- added R?: R, symbol R
Changed lines of the file:
@@
 LIBS:regul
 LIBS:user
+LIBS:template_test-cache
 EELAYER 25 0
 EELAYER END
@@
 Comment4 ""
 $EndDescr
+$Comp
+L R R?
+U 1 1 57743B49
+P 5800 2900
+F 0 "R?" V 5880 2900 40  0000 C CNN
+F 1 "R" V 5807 2901 40  0000 C CNN
+F 2 "" V 5730 2900 30  0000 C CNN
+F 3 "" H 5800 2900 30  0000 C CNN
+	1    5800 2900
+	1    0    0    -1
+$EndComp
 $EndSCHEMATC
