File: KiCAD_Projects/regulPCB/regulPCB.kicad_pcb (KiCad board)
At the start: 2 copper layers, 31.8 x 25.4 mm, 4 parts, among them P1 CONN_01X03, U1 LM1084IT-5.0/NOPB

Commit message: no message
Parts:
- moved C1 149.0 mm to (0.00, 8.89)
- moved C2 149.0 mm to (1.27, 3.81)
- moved P1 149.0 mm to (2.54, 6.35)
- moved U1 149.0 mm to (0.00, 0.00)
Other:
- board size 31.8 x 25.4 mm -> 30 x 26 mm
Changed lines of the file:
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@@
     (links 7)
     (no_connects 0)
-    (area 95.149999 76.734999 130.275001 109.248333)
+    (area -15.075001 -15.075001 15.075001 11.075001)
     (thickness 1.6)
-    (drawings 12)
+    (drawings 10)
     (tracks 15)
     (zones 0)
@@
   )
   (setup
-    (last_trace_width 0.25)
+    (last_trace_width 1)
     (user_trace_width 1)
     (trace_clearance 0.2)
@@
   )
   (module RP_KiCAD_Libs:C3216 (layer B.Cu)
-    (at 112.395 106.68)
+    (at 0 8.89)
     (descr <b>CAPACITOR</b>)
     (fp_text reference C1 (at -1.27 1.27) (layer B.SilkS)
@@
   )
   (module RP_KiCAD_Libs:C3216 (layer B.Cu)
-    (at 113.665 101.6)
+    (at 1.27 3.81)
     (descr <b>CAPACITOR</b>)
     (fp_text reference C2 (at -1.27 1.27) (layer B.SilkS)
@@
   )
   (module Pin_Headers:Pin_Header_Angled_1x03 (layer B.Cu)
-    (at 114.935 104.14 90)
+    (at 2.54 6.35 90)
     (descr "Through hole pin header")
     (tags "pin header")
@@
   )
   (module TO_SOT_Packages_SMD:TO-263-3Lead (layer B.Cu)
-    (at 112.395 97.79 90)
+    (at 0 0 90)
     (descr "D2PAK / TO-263 3-lead smd package")
     (tags "D2PAK D2PAK-3 TO-263AB TO-263")
@@
     )
   )
-  (gr_line (start 128.27 90.17) (end 128.27 82.55) (angle 90) (layer Edge.Cuts) (width 0.15))
-  (gr_line (start 96.52 90.17) (end 96.52 82.55) (angle 90) (layer Edge.Cuts) (width 0.15))
-  (gr_line (start 106.68 100.33) (end 106.68 107.95) (angle 90) (layer Edge.Cuts) (width 0.15))
-  (gr_line (start 96.52 90.17) (end 106.68 100.33) (angle 90) (layer Edge.Cuts) (width 0.15))
-  (gr_line (start 118.11 100.33) (end 118.11 107.95) (angle 90) (layer Edge.Cuts) (width 0.15))
-  (gr_line (start 128.27 90.17) (end 118.11 100.33) (angle 90) (layer Edge.Cuts) (width 0.15))
-  (gr_line (start 106.68 107.95) (end 118.11 107.95) (angle 90) (layer Edge.Cuts) (width 0.15))
-  (gr_line (start 96.52 82.55) (end 128.27 82.55) (angle 90) (layer Edge.Cuts) (width 0.15))
-  (gr_circle (center 123.19 87.63) (end 118.11 87.63) (layer F.SilkS) (width 0.2))
-  (gr_circle (center 101.6 87.63) (end 106.68 87.63) (layer F.SilkS) (width 0.2))
-  (gr_circle (center 112.395 87.63) (end 123.19 87.63) (layer F.SilkS) (width 0.2))
-  (gr_line (start 95.25 87.63) (end 130.175 87.63) (angle 90) (layer F.SilkS) (width 0.2))
-  (via (at 101.6 87.63) (size 5) (drill 3) (layers F.Cu B.Cu) (net 0))
-  (via (at 123.19 87.63) (size 5) (drill 3) (layers F.Cu B.Cu) (net 0))
-  (segment (start 109.855 97.79) (end 109.855 104.14) (width 1) (layer B.Cu) (net 1))
-  (segment (start 109.855 104.14) (end 109.855 105.74) (width 1) (layer B.Cu) (net 1))
-  (segment (start 109.855 105.74) (end 110.795 106.68) (width 1) (layer B.Cu) (net 1))
-  (segment (start 113.995 106.68) (end 114.935 105.74) (width 1) (layer B.Cu) (net 2))
-  (segment (start 114.935 105.74) (end 114.935 104.14) (width 1) (layer B.Cu) (net 2))
-  (segment (start 115.265 101.6) (end 114.935 101.93) (width 1) (layer B.Cu) (net 2))
-  (segment (start 114.935 101.93) (end 114.935 102.87) (width 1) (layer B.Cu) (net 2))
-  (segment (start 114.935 97.79) (end 114.935 102.87) (width 1) (layer B.Cu) (net 2))
-  (segment (start 114.935 102.87) (end 114.935 104.14) (width 1) (layer B.Cu) (net 2))
-  (segment (start 112.065 101.6) (end 112.395 101.93) (width 1) (layer B.Cu) (net 3))
-  (segment (start 112.395 101.93) (end 112.395 102.87) (width 1) (layer B.Cu) (net 3))
-  (segment (start 112.395 97.79) (end 112.395 102.87) (width 1) (layer B.Cu) (net 3))
-  (segment (start 112.395 102.87) (end 112.395 104.14) (width 1) (layer B.Cu) (net 3))
+  (gr_line (start 15 -9) (end 5 1) (angle 90) (layer Edge.Cuts) (width 0.15))
+  (gr_line (start 15 -11) (end 11 -15) (angle 90) (layer Edge.Cuts) (width 0.15))
+  (gr_line (start -15 -9) (end -5 1) (angle 90) (layer Edge.Cuts) (width 0.15))
+  (gr_line (start -15 -11) (end -11 -15) (angle 90) (layer Edge.Cuts) (width 0.15))
+  (gr_line (start -15 -11) (end -15 -9) (angle 90) (layer Edge.Cuts) (width 0.15))
+  (gr_line (start 15 -11) (end 15 -9) (angle 90) (layer Edge.Cuts) (width 0.15))
+  (gr_line (start -11 -15) (end 11 -15) (angle 90) (layer Edge.Cuts) (width 0.15))
+  (gr_line (start -5 11) (end -5 1) (angle 90) (layer Edge.Cuts) (width 0.15))
+  (gr_line (start 5 11) (end -5 11) (angle 90) (layer Edge.Cuts) (width 0.15))
+  (gr_line (start 5 1) (end 5 11) (angle 90) (layer Edge.Cuts) (width 0.15))
+  (via (at -11 -10) (size 5) (drill 3) (layers F.Cu B.Cu) (net 0))
+  (via (at 11 -10) (size 5) (drill 3) (layers F.Cu B.Cu) (net 0))
+  (segment (start -2.54 6.35) (end -2.54 7.95) (width 1) (layer B.Cu) (net 1))
+  (segment (start -2.54 7.95) (end -1.6 8.89) (width 1) (layer B.Cu) (net 1))
+  (segment (start -2.54 0) (end -2.54 6.35) (width 1) (layer B.Cu) (net 1))
+  (segment (start 2.87 3.81) (end 2.54 4.14) (width 1) (layer B.Cu) (net 2))
+  (segment (start 2.54 4.14) (end 2.54 5.08) (width 1) (layer B.Cu) (net 2))
+  (segment (start 2.54 0) (end 2.54 5.08) (width 1) (layer B.Cu) (net 2))
+  (segment (start 2.54 5.08) (end 2.54 6.35) (width 1) (layer B.Cu) (net 2))
+  (segment (start 2.54 6.35) (end 2.54 7.95) (width 1) (layer B.Cu) (net 2))
+  (segment (start 2.54 7.95) (end 1.6 8.89) (width 1) (layer B.Cu) (net 2))
+  (segment (start -0.33 3.81) (end 0 4.14) (width 1) (layer B.Cu) (net 3))
+  (segment (start 0 4.14) (end 0 5.08) (width 1) (layer B.Cu) (net 3))
+  (segment (start 0 0) (end 0 5.08) (width 1) (layer B.Cu) (net 3))
+  (segment (start 0 5.08) (end 0 6.35) (width 1) (layer B.Cu) (net 3))
   (zone (net 0) (net_name "") (layer B.Cu) (hatch edge 0.508)
     (connect_pads (clearance 0.4))
     (min_thickness 0.0254)
-    (fill yes (arc_segments 16) (thermal_gap 0.508) (thermal_bridge_width 0.508))
+    (fill yes (arc_segments 16) (thermal_gap 0.4) (thermal_bridge_width 0.4))
     (polygon
       (pts
-        (xy 128.27 90.17) (xy 118.11 100.33) (xy 118.11 107.95) (xy 106.68 107.95) (xy 106.68 100.33)
-        (xy 96.52 90.17) (xy 96.52 82.55) (xy 128.27 82.55) (xy 128.27 90.17)
+        (xy 16 11) (xy -16 11) (xy -16 -15) (xy 16 -15) (xy 16 11)
       )
     )
