File: KiCAD_Projects/3phaseDriver/3phaseDriver.kicad_pcb (KiCad board)
At the start: 2 copper layers, 50 x 50 mm, 26 parts, among them P1 CONN_01X06, P2 CONN_01X06, P3 CONN_01X01, P4 CONN_01X01, P5 CONN_01X01, Q1 MOSFET_N, Q2 MOSFET_N, Q3 MOSFET_N, Q4 MOSFET_N, Q5 MOSFET_N, Q6 MOSFET_N, U1 NCP5104, U2 NCP5104, U3 NCP5104

Commit message: no message
Parts:
- removed Q1, Q2, Q3, Q4, Q5, Q6: MOSFET_N, TO_SOT_Packages_SMD:D2-PAK
- removed R1, R2, R3, R4, R5, R6: R, RP_KiCAD_Libs:0204_2f7
- added C4: C, RP_KiCAD_Libs:C3216, B.Cu at (156.8, 73.0)
- C1: footprint RP_KiCAD_Libs:C3216 -> Capacitors_ThroughHole:C_Radial_D5_L11_P2; moved to F.Cu
- P3, P4: value CONN_01X01 -> CONN_01X02; footprint Connect:1pin -> Pin_Headers:Pin_Header_Straight_1x02
- P5: value CONN_01X01 -> CONN_01X09; footprint Connect:1pin -> Pin_Headers:Pin_Header_Straight_1x09_Pitch2.00mm
- moved P5 153.4 mm to (152.4, 58.4)
- moved U3 150.4 mm to (162.6, 73.7), turned to 180 degrees
- moved P2 148.3 mm to (170.2, 72.4), turned to 90 degrees
- moved D3 145.7 mm to (162.6, 69.8), turned to 180 degrees
- moved C3 143.8 mm to (156.8, 65.4), turned to 270 degrees
- moved U2 134.5 mm to (162.6, 66.0), turned to 180 degrees
- moved D2 129.8 mm to (162.6, 62.2), turned to 180 degrees
- moved C2 127.9 mm to (156.8, 57.8), turned to 270 degrees
- moved U1 118.8 mm to (162.6, 58.4), turned to 180 degrees
- moved D1 114.3 mm to (162.6, 54.6), turned to 180 degrees
- moved P4 106.4 mm to (105.0, 83.0)
- moved C1 98.8 mm to (142.2, 63.5)
- moved P1 98.3 mm to (146.1, 88.9), turned to 180 degrees
- moved P3 83.1 mm to (105.0, 64.0)
Connections:
- C1 pad 1: Net-(C1-Pad1) -> +12V
- C1 pad 2: Net-(C1-Pad2) -> GND
- D1 pad 2: Net-(C1-Pad1) -> Net-(C2-Pad1)
- D2 pad 2: Net-(C2-Pad1) -> Net-(C3-Pad1)
- D3 pad 2: Net-(C3-Pad1) -> Net-(C4-Pad1)
- P3 pad 1: Net-(C1-Pad2) -> +BATT
- P4 pad 1: Net-(C2-Pad2) -> GND
- P5 pad 1: Net-(C3-Pad2) -> Net-(P5-Pad1)
- U1 pad 5: Net-(R2-Pad2) -> Net-(P5-Pad3)
- U1 pad 6: Net-(C1-Pad2) -> Net-(C2-Pad2)
- U1 pad 7: Net-(R1-Pad2) -> Net-(P5-Pad1)
- U1 pad 8: Net-(C1-Pad1) -> Net-(C2-Pad1)
- U2 pad 5: Net-(R4-Pad2) -> Net-(P5-Pad6)
- U2 pad 6: Net-(C2-Pad2) -> Net-(C3-Pad2)
- U2 pad 7: Net-(R3-Pad2) -> Net-(P5-Pad4)
- U2 pad 8: Net-(C2-Pad1) -> Net-(C3-Pad1)
- U3 pad 5: Net-(R6-Pad2) -> Net-(P5-Pad9)
- U3 pad 6: Net-(C3-Pad2) -> Net-(C4-Pad2)
- U3 pad 7: Net-(R5-Pad2) -> Net-(P5-Pad7)
- U3 pad 8: Net-(C3-Pad1) -> Net-(C4-Pad1)
Routing:
- net GND: track 98.1 -> 0.00 mm, vias 4 -> 0
- net +BATT: track 53.5 -> 0.00 mm
- net +12V: track 47.2 -> 7.09 mm
- net Net-(C1-Pad2): track 27.1 -> 0.00 mm, vias 2 -> 0
- net Net-(Q3-PadG): track 25.8 -> 0.00 mm
- net Net-(Q1-PadG): track 25.8 -> 0.00 mm
- net Net-(Q5-PadG): track 25.8 -> 0.00 mm
- net Net-(C3-Pad2): track 27.1 -> 7.84 mm, vias 2 -> 0
- net Net-(C2-Pad2): track 27.1 -> 8.03 mm, vias 2 -> 0
- net Net-(P5-Pad7): track 0.00 -> 8.54 mm
- net Net-(C4-Pad2): track 0.00 -> 8.51 mm
- net Net-(P5-Pad9): track 0.00 -> 8.46 mm
- net Net-(P5-Pad3): track 0.00 -> 8.33 mm
- net Net-(P5-Pad4): track 0.00 -> 7.87 mm
- net Net-(P5-Pad1): track 0.00 -> 7.72 mm
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- removed copper zone on B.Cu, net +BATT
- removed copper zone on B.Cu, net GND
- removed copper zone on B.Cu, net Net-(C1-Pad2)
- removed copper zone on B.Cu, net Net-(C2-Pad2)
- removed copper zone on B.Cu, net Net-(C3-Pad2)
Other:
- board outline removed
