File: KiCAD_Projects/CNC_GRBL_Controller/CNC_GRBL_Controller.kicad_pcb (KiCad board)
At the start: 2 copper layers, 100 x 50 mm, 10 parts, among them IC1 ATMEGA328-P, J1 DB25, P1 CONN_01X06, P2 CONN_01X02, SW1 SW_PUSH_SMALL, X1 CRYSTAL

Commit message: no message
Parts:
- removed P1: CONN_01X06, Pin_Headers:Pin_Header_Straight_1x06
- added C4: C, RP_KiCAD_Libs:C1608, B.Cu at (71.8, 12.7)
- added D1: LED, LEDs:LED-3MM, F.Cu at (94.0, 10.2)
- added D2: LED, LEDs:LED-3MM, F.Cu at (94.0, 15.2)
- added R2: R, RP_KiCAD_Libs:C1608, B.Cu at (75.6, 10.2)
- added R3: R, RP_KiCAD_Libs:C1608, B.Cu at (71.8, 20.3)
- added R4: R, RP_KiCAD_Libs:C1608, B.Cu at (95.9, 10.2)
- added R5: R, RP_KiCAD_Libs:C1608, B.Cu at (95.9, 15.2)
- added U1: AE-UM232R, Housings_DIP:DIP-24_W15.24mm_LongPads, F.Cu at (73.7, 10.2)
- P2: value CONN_01X02 -> CONN_01X07; footprint Pin_Headers:Pin_Header_Straight_1x02 -> Pin_Headers:Pin_Header_Straight_1x07
- moved P2 9.69 mm to (53.3, 27.9), turned to 270 degrees
Connections:
- net Net-(IC1-Pad1) renamed /Arduino_RESET
- P2 pad 1: /Arduino_TX -> +5V
- P2 pad 2: /Arduino_RX -> GND
Routing:
- net +5V: track 41.2 -> 83.6 mm
- net GND: track 49.0 -> 89.5 mm, vias 0 -> 2
- net /Arduino_RX: track 26.3 -> 64.8 mm, vias 0 -> 2
- net /Arduino_RESET: track 34.4 -> 64.3 mm, vias 0 -> 2
- net /Arduino_TX: track 25.1 -> 52.9 mm, vias 0 -> 2
- net Net-(D1-Pad2): track 0.00 -> 3.59 mm
- net Net-(D2-Pad2): track 0.00 -> 2.54 mm
- net Net-(D2-Pad1): track 0.00 -> 1.05 mm
- net Net-(D1-Pad1): track 0.00 -> 1.05 mm
- net (no net): vias 0 -> 4
Other:
- board size 100 x 50 mm -> 85 x 50 mm

Commit message: no message
Parts:
- C4: footprint RP_KiCAD_Libs:C1608 -> RP_KiCAD_Libs:C2012
Changed lines of the file:
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@@
     (links 57)
     (no_connects 0)
-    (area 14.924999 -11.578001 100.075001 50.075001)
+    (area 14.924999 -0.075001 100.075001 50.075001)
     (thickness 1.6)
     (drawings 4)
@@
   )
   (setup
-    (last_trace_width 0.5)
+    (last_trace_width 0.25)
     (user_trace_width 0.5)
     (user_trace_width 1)
@@
     )
   )
-  (module RP_KiCAD_Libs:C1608 (layer B.Cu)
-    (at 71.755 12.7 180)
-    (descr <b>CAPACITOR</b>)
-    (fp_text reference C4 (at -0.635 0.635 180) (layer B.SilkS)
-      (effects (font (size 1.2065 1.2065) (thickness 0.1016)) (justify left bottom mirror))
-    )
-    (fp_text value C (at -0.635 -1.905 180) (layer B.SilkS)
-      (effects (font (size 1.2065 1.2065) (thickness 0.1016)) (justify left bottom mirror))
-    )
-    (fp_line (start -0.356 0.432) (end 0.356 0.432) (layer Dwgs.User) (width 0.1016))
-    (fp_line (start -0.356 -0.419) (end 0.356 -0.419) (layer Dwgs.User) (width 0.1016))
-    (fp_poly (pts (xy -0.8382 -0.4699) (xy -0.3381 -0.4699) (xy -0.3381 0.4801) (xy -0.8382 0.4801)) (layer Dwgs.User) (width 0))
-    (fp_poly (pts (xy 0.3302 -0.4699) (xy 0.8303 -0.4699) (xy 0.8303 0.4801) (xy 0.3302 0.4801)) (layer Dwgs.User) (width 0))
-    (fp_poly (pts (xy -0.1999 -0.3) (xy 0.1999 -0.3) (xy 0.1999 0.3) (xy -0.1999 0.3)) (layer B.Adhes) (width 0))
-    (pad 1 smd rect (at -0.85 0 180) (size 1.1 1) (layers B.Cu B.Paste B.Mask)
-      (net 23 "Net-(C4-Pad1)"))
-    (pad 2 smd rect (at 0.85 0 180) (size 1.1 1) (layers B.Cu B.Paste B.Mask)
-      (net 24 /Arduino_RESET))
-    (model Resistors_SMD.3dshapes/R_0603.wrl
-      (at (xyz 0 0 0))
-      (scale (xyz 1 1 1))
-      (rotate (xyz 0 0 0))
-    )
-  )
   (module LEDs:LED-3MM (layer F.Cu)
     (at 93.98 10.16 180)
@@
       (scale (xyz 1 1 1))
       (rotate (xyz 0 0 90))
+    )
+  )
+  (module RP_KiCAD_Libs:C2012 (layer B.Cu)
+    (at 71.755 12.7 180)
+    (descr <b>CAPACITOR</b>)
+    (fp_text reference C4 (at -1.27 1.27 180) (layer B.SilkS)
+      (effects (font (size 1.2065 1.2065) (thickness 0.1016)) (justify left bottom mirror))
+    )
+    (fp_text value C (at -1.27 -2.54 180) (layer B.SilkS)
+      (effects (font (size 1.2065 1.2065) (thickness 0.1016)) (justify left bottom mirror))
+    )
+    (fp_line (start -0.381 0.66) (end 0.381 0.66) (layer Dwgs.User) (width 0.1016))
+    (fp_line (start -0.356 -0.66) (end 0.381 -0.66) (layer Dwgs.User) (width 0.1016))
+    (fp_poly (pts (xy -1.0922 -0.7239) (xy -0.3421 -0.7239) (xy -0.3421 0.7262) (xy -1.0922 0.7262)) (layer Dwgs.User) (width 0))
+    (fp_poly (pts (xy 0.3556 -0.7239) (xy 1.1057 -0.7239) (xy 1.1057 0.7262) (xy 0.3556 0.7262)) (layer Dwgs.User) (width 0))
+    (fp_poly (pts (xy -0.1001 -0.4001) (xy 0.1001 -0.4001) (xy 0.1001 0.4001) (xy -0.1001 0.4001)) (layer B.Adhes) (width 0))
+    (pad 1 smd rect (at -1.25 0 180) (size 1.3 1.5) (layers B.Cu B.Paste B.Mask)
+      (net 23 "Net-(C4-Pad1)"))
+    (pad 2 smd rect (at 1.25 0 180) (size 1.3 1.5) (layers B.Cu B.Paste B.Mask)
+      (net 24 /Arduino_RESET))
+    (model Resistors_SMD.3dshapes/R_0805.wrl
+      (at (xyz 0 0 0))
+      (scale (xyz 1 1 1))
+      (rotate (xyz 0 0 0))
     )
   )
@@
   (segment (start 53.34 33.02) (end 50.8 35.56) (width 0.5) (layer F.Cu) (net 1))
   (via (at 53.34 33.02) (size 1.2) (drill 0.8) (layers F.Cu B.Cu) (net 1))
-  (segment (start 73.66 25.4) (end 76.2 25.4) (width 0.5) (layer B.Cu) (net 2) (status 400000))
-  (segment (start 85.09 10.16) (end 88.9 10.16) (width 0.5) (layer B.Cu) (net 2) (status 800000))
+  (segment (start 73.66 25.4) (end 76.2 25.4) (width 0.5) (layer B.Cu) (net 2))
+  (segment (start 85.09 10.16) (end 88.9 10.16) (width 0.5) (layer B.Cu) (net 2))
   (segment (start 81.28 13.97) (end 85.09 10.16) (width 0.5) (layer B.Cu) (net 2))
   (segment (start 81.28 20.32) (end 81.28 13.97) (width 0.5) (layer B.Cu) (net 2))
   (segment (start 76.2 25.4) (end 81.28 20.32) (width 0.5) (layer B.Cu) (net 2))
-  (segment (start 55.46 41.91) (end 55.46 43.6) (width 0.5) (layer B.Cu) (net 2) (status 400000))
+  (segment (start 55.46 41.91) (end 55.46 43.6) (width 0.5) (layer B.Cu) (net 2))
   (segment (start 55.245 43.815) (end 53.555 43.815) (width 0.5) (layer B.Cu) (net 2))
   (segment (start 55.46 43.6) (end 55.245 43.815) (width 0.5) (layer B.Cu) (net 2))
-  (segment (start 53.34 38.1) (end 53.34 40.005) (width 0.5) (layer B.Cu) (net 2) (status 400000))
+  (segment (start 53.34 38.1) (end 53.34 40.005) (width 0.5) (layer B.Cu) (net 2))
   (segment (start 53.34 40.005) (end 51.435 40.005) (width 0.5) (layer B.Cu) (net 2))
-  (segment (start 50.8 27.94) (end 50.8 25.4) (width 0.5) (layer B.Cu) (net 2) (status 400000))
+  (segment (start 50.8 27.94) (end 50.8 25.4) (width 0.5) (layer B.Cu) (net 2))
   (segment (start 52.07 24.13) (end 54.61 24.13) (width 0.5) (layer B.Cu) (net 2))
   (segment (start 50.8 25.4) (end 52.07 24.13) (width 0.5) (layer B.Cu) (net 2))

Commit message: no message
Routing:
- added copper zone on B.Cu, net (none)
Changed lines of the file:
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@@
   (general
     (links 57)
-    (no_connects 0)
+    (no_connects 1)
     (area 14.924999 -0.075001 100.075001 50.075001)
     (thickness 1.6)
@@
   (segment (start 93.98 15.24) (end 95.035 15.24) (width 0.5) (layer B.Cu) (net 27))
   (segment (start 88.9 15.24) (end 91.44 15.24) (width 0.5) (layer B.Cu) (net 28))
-  (zone (net 2) (net_name GND) (layer B.Cu) (hatch edge 0.508)
+  (zone (net 0) (net_name "") (layer B.Cu) (hatch edge 0.508)
     (connect_pads (clearance 0.4))
     (min_thickness 0.2)
@@
     (polygon
       (pts
-        (xy 100 50) (xy 15 50) (xy 15 0) (xy 100 0) (xy 100 50)
+        (xy 100 0) (xy 100 50) (xy 15 50) (xy 15 0) (xy 33 0)
+        (xy 33 6) (xy 66 6) (xy 66 0)
       )
     )
+  )
+  (zone (net 2) (net_name GND) (layer B.Cu) (hatch edge 0.508)
+    (connect_pads yes (clearance 0.4))
+    (min_thickness 0.2)
+    (fill yes (arc_segments 16) (thermal_gap 0.508) (thermal_bridge_width 0.508))
+    (polygon
+      (pts
+        (xy 65 5) (xy 44 5) (xy 44 0) (xy 65 0) (xy 65 5)
+      )
+    )

Commit message: no message
Parts:
- removed SW1: SW_PUSH_SMALL, Buttons_Switches_ThroughHole:SW_DIP_x1_Slide
- added C5: C, RP_KiCAD_Libs:C1608, B.Cu at (67.3, 37.5)
- added P1: CONN_01X05, RP_KiCAD_Connector:XA_5L, F.Cu at (9.53, 25.4)
- added P3: CONN_01X02, RP_KiCAD_Connector:XA_2L, F.Cu at (38.1, 40.6)
- added P4: CONN_01X02, RP_KiCAD_Connector:XA_2L, F.Cu at (27.9, 40.6)
- added P5: CONN_01X02, RP_KiCAD_Connector:XA_2L, F.Cu at (17.8, 40.6)
- added P6: CONN_01X02, RP_KiCAD_Connector:XA_2L, F.Cu at (76.2, 40.6)
- added P7: CONN_01X02, RP_KiCAD_Connector:XA_2L, F.Cu at (66.0, 40.6)
- added Q1: MOSFET_N, TO_SOT_Packages_THT:TO-220_Neutral123_Vertical, F.Cu at (59.1, 37.5)
- added R6: R, RP_KiCAD_Libs:0204_2f5, F.Cu at (50.2, 34.9)
- added R7: R, RP_KiCAD_Libs:C1608, B.Cu at (52.7, 37.5)
- C4: footprint RP_KiCAD_Libs:C2012 -> RP_KiCAD_Libs:0204_2f5; moved to F.Cu
- P2: value CONN_01X07 -> CONN_01X02; footprint Pin_Headers:Pin_Header_Straight_1x07 -> RP_KiCAD_Connector:XA_2L
- R1, R2, R3: footprint RP_KiCAD_Libs:C1608 -> RP_KiCAD_Libs:0204_2f5; moved to F.Cu
- moved C2 41.3 mm to (24.1, 17.1), turned to 180 degrees
- moved X1 38.9 mm to (25.4, 17.8), turned to 180 degrees
- moved C3 37.3 mm to (26.7, 17.1), turned to 0 degrees
- moved R1 34.3 mm to (66.0, 20.3), turned to 270 degrees
- moved U1 28.7 mm to (53.3, 30.5), turned to 90 degrees
- moved R2 26.9 mm to (53.3, 25.4), turned to 90 degrees
- moved C1 21.1 mm to (35.6, 26.7)
- moved D1 20.9 mm to (73.7, 5.08)
- moved D2 20.9 mm to (73.7, 10.2)
- moved R4 20.3 mm to (76.2, 5.08)
- moved R5 20.3 mm to (76.2, 10.2)
- moved C4 20.3 mm to (55.9, 25.4), turned to 90 degrees
- moved IC1 19.8 mm to (48.3, 22.9), turned to 270 degrees
- moved J1 15.0 mm to (34.5, 0.00)
- moved P2 13.7 mm to (48.3, 40.6), turned to 0 degrees
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Connections:
- J1 pad 11: /Limit_X -> (no net)
- J1 pad 12: /Limit_Y -> (no net)
- J1 pad 13: /Limit_Z -> (no net)
- J1 pad 15: /Reset/Abort -> (no net)
- P2 pad 1: +5V -> GND
- P2 pad 2: GND -> /Probe
Routing:
- net GND: track 89.5 -> 258.9 mm
- net /Stepper_~EN: track 108.0 -> 28.3 mm, vias 4 -> 0
- net /X_Dir: track 86.6 -> 24.7 mm, vias 3 -> 1
- net /Y_Dir: track 88.9 -> 29.5 mm, vias 3 -> 1
- net /Arduino_RX: track 64.8 -> 9.20 mm, vias 2 -> 0
- net /Z_Dir: track 91.1 -> 36.8 mm
- net /Arduino_RESET: track 64.3 -> 20.9 mm, vias 2 -> 0
- net /Z_Step: track 60.9 -> 21.8 mm
- net /Y_Step: track 60.5 -> 29.0 mm
- net /Arduino_TX: track 52.9 -> 23.0 mm, vias 2 -> 0
- net /Limit_X: track 33.3 -> 5.75 mm, vias 3 -> 0
- net +5V: track 83.6 -> 106.6 mm, vias 2 -> 4
- net /Spindle_EN: track 57.5 -> 37.1 mm, vias 3 -> 1
- net /Limit_Y: track 29.0 -> 9.26 mm, vias 1 -> 0
- net /Limit_Z: track 32.2 -> 12.8 mm, vias 3 -> 0
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