File: KiCAD_Projects/CNC_LIMIT_AND/CNC_LIMIT_AND.sch (KiCad schematic (older format))
At the start: 19 parts, among them P1 CONN_01X03, P2 CONN_01X03, P3 CONN_01X03, P4 CONN_01X03, P5 CONN_01X05, Q1 MOSFET_N, Q2 MOSFET_N, Q3 MOSFET_N, Q4 MOSFET_N

Commit message: no message
Parts:
- P1, P2, P3, P4: footprint (none) -> RP_KiCAD_Connector:XA_3L
- P5: footprint (none) -> RP_KiCAD_Connector:XA_5L
- Q1, Q2, Q3, Q4: footprint (none) -> TO_SOT_Packages_SMD:SOT-23_Handsoldering
- R1, R2, R3, R4: footprint (none) -> RP_KiCAD_Libs:C1608
- R10, R5, R6, R7, R8, R9: footprint (none) -> RP_KiCAD_Libs:0204_2f5
Changed lines of the file:
@@
 F 0 "P1" H 4750 2450 50  0000 C CNN
 F 1 "CONN_01X03" V 4850 2250 50  0000 C CNN
-F 2 "" H 4750 2250 50  0000 C CNN
+F 2 "RP_KiCAD_Connector:XA_3L" H 4750 2250 50  0001 C CNN
 F 3 "" H 4750 2250 50  0000 C CNN
 	1    4750 2250
@@
 F 0 "P3" H 4800 3300 50  0000 C CNN
 F 1 "CONN_01X03" V 4900 3100 50  0000 C CNN
-F 2 "" H 4800 3100 50  0000 C CNN
+F 2 "RP_KiCAD_Connector:XA_3L" H 4800 3100 50  0001 C CNN
 F 3 "" H 4800 3100 50  0000 C CNN
 	1    4800 3100
@@
 F 0 "Q1" H 6310 2320 60  0000 R CNN
 F 1 "MOSFET_N" H 6310 2000 60  0000 R CNN
-F 2 "" H 6300 2150 60  0000 C CNN
+F 2 "TO_SOT_Packages_SMD:SOT-23_Handsoldering" H 6300 2150 60  0001 C CNN
 F 3 "" H 6300 2150 60  0000 C CNN
 	1    6300 2150
@@
 F 0 "Q2" H 6310 3170 60  0000 R CNN
 F 1 "MOSFET_N" H 6310 2850 60  0000 R CNN
-F 2 "" H 6300 3000 60  0000 C CNN
+F 2 "TO_SOT_Packages_SMD:SOT-23_Handsoldering" H 6300 3000 60  0001 C CNN
 F 3 "" H 6300 3000 60  0000 C CNN
 	1    6300 3000
@@
 F 0 "R1" V 5730 2150 40  0000 C CNN
 F 1 "R" V 5657 2151 40  0000 C CNN
-F 2 "" V 5580 2150 30  0000 C CNN
+F 2 "RP_KiCAD_Libs:C1608" V 5580 2150 30  0001 C CNN
 F 3 "" H 5650 2150 30  0000 C CNN
 	1    5650 2150
@@
 F 0 "R5" V 6030 2300 40  0000 C CNN
 F 1 "R" V 5957 2301 40  0000 C CNN
-F 2 "" V 5880 2300 30  0000 C CNN
+F 2 "RP_KiCAD_Libs:0204_2f5" V 5880 2300 30  0001 C CNN
 F 3 "" H 5950 2300 30  0000 C CNN
 	1    5950 2300
@@
 F 0 "R2" V 5730 3000 40  0000 C CNN
 F 1 "R" V 5657 3001 40  0000 C CNN
-F 2 "" V 5580 3000 30  0000 C CNN
+F 2 "RP_KiCAD_Libs:C1608" V 5580 3000 30  0001 C CNN
 F 3 "" H 5650 3000 30  0000 C CNN
 	1    5650 3000
@@
 F 0 "R6" V 6030 3150 40  0000 C CNN
 F 1 "R" V 5957 3151 40  0000 C CNN
-F 2 "" V 5880 3150 30  0000 C CNN
+F 2 "RP_KiCAD_Libs:0204_2f5" V 5880 3150 30  0001 C CNN
 F 3 "" H 5950 3150 30  0000 C CNN
 	1    5950 3150
@@
 F 0 "P2" H 4750 4300 50  0000 C CNN
 F 1 "CONN_01X03" V 4850 4100 50  0000 C CNN
-F 2 "" H 4750 4100 50  0000 C CNN
+F 2 "RP_KiCAD_Connector:XA_3L" H 4750 4100 50  0001 C CNN
 F 3 "" H 4750 4100 50  0000 C CNN
 	1    4750 4100
@@
 F 0 "P4" H 4800 5150 50  0000 C CNN
 F 1 "CONN_01X03" V 4900 4950 50  0000 C CNN
-F 2 "" H 4800 4950 50  0000 C CNN
+F 2 "RP_KiCAD_Connector:XA_3L" H 4800 4950 50  0001 C CNN
 F 3 "" H 4800 4950 50  0000 C CNN
 	1    4800 4950
@@
 F 0 "Q3" H 6310 4170 60  0000 R CNN
 F 1 "MOSFET_N" H 6310 3850 60  0000 R CNN
-F 2 "" H 6300 4000 60  0000 C CNN
+F 2 "TO_SOT_Packages_SMD:SOT-23_Handsoldering" H 6300 4000 60  0001 C CNN
 F 3 "" H 6300 4000 60  0000 C CNN
 	1    6300 4000
@@
 F 0 "Q4" H 6310 5020 60  0000 R CNN
 F 1 "MOSFET_N" H 6310 4700 60  0000 R CNN
-F 2 "" H 6300 4850 60  0000 C CNN
+F 2 "TO_SOT_Packages_SMD:SOT-23_Handsoldering" H 6300 4850 60  0001 C CNN
 F 3 "" H 6300 4850 60  0000 C CNN
 	1    6300 4850
@@
 F 0 "R3" V 5730 4000 40  0000 C CNN
 F 1 "R" V 5657 4001 40  0000 C CNN
-F 2 "" V 5580 4000 30  0000 C CNN
+F 2 "RP_KiCAD_Libs:C1608" V 5580 4000 30  0001 C CNN
 F 3 "" H 5650 4000 30  0000 C CNN
 	1    5650 4000
@@
 F 0 "R7" V 6030 4150 40  0000 C CNN
 F 1 "R" V 5957 4151 40  0000 C CNN
-F 2 "" V 5880 4150 30  0000 C CNN
+F 2 "RP_KiCAD_Libs:0204_2f5" V 5880 4150 30  0001 C CNN
 F 3 "" H 5950 4150 30  0000 C CNN
 	1    5950 4150
@@
 F 0 "R4" V 5730 4850 40  0000 C CNN
 F 1 "R" V 5657 4851 40  0000 C CNN
-F 2 "" V 5580 4850 30  0000 C CNN
+F 2 "RP_KiCAD_Libs:C1608" V 5580 4850 30  0001 C CNN
 F 3 "" H 5650 4850 30  0000 C CNN
 	1    5650 4850
@@
 F 0 "R8" V 6030 5000 40  0000 C CNN
 F 1 "R" V 5957 5001 40  0000 C CNN
-F 2 "" V 5880 5000 30  0000 C CNN
+F 2 "RP_KiCAD_Libs:0204_2f5" V 5880 5000 30  0001 C CNN
 F 3 "" H 5950 5000 30  0000 C CNN
 	1    5950 5000
@@
 F 0 "P5" H 7650 3250 50  0000 C CNN
 F 1 "CONN_01X05" V 7750 2950 50  0000 C CNN
-F 2 "" H 7650 2950 50  0000 C CNN
+F 2 "RP_KiCAD_Connector:XA_5L" H 7650 2950 50  0001 C CNN
 F 3 "" H 7650 2950 50  0000 C CNN
 	1    7650 2950
@@
 F 0 "R10" V 8180 2600 40  0000 C CNN
 F 1 "R" V 8107 2601 40  0000 C CNN
-F 2 "" V 8030 2600 30  0000 C CNN
+F 2 "RP_KiCAD_Libs:0204_2f5" V 8030 2600 30  0001 C CNN
 F 3 "" H 8100 2600 30  0000 C CNN
 	1    8100 2600
@@
 F 0 "R9" V 8030 2700 40  0000 C CNN
 F 1 "R" V 7957 2701 40  0000 C CNN
-F 2 "" V 7880 2700 30  0000 C CNN
+F 2 "RP_KiCAD_Libs:0204_2f5" V 7880 2700 30  0001 C CNN
 F 3 "" H 7950 2700 30  0000 C CNN
 	1    7950 2700
