File: KiCAD_Projects/F303_SI8234/F303_SI8234.kicad_pcb (KiCad board)
At the start: 2 copper layers, 68 parts, among them IC1 TLP785F, IC2 ATTINY85-P, P1 CONN_01X06, P2 CONN_01X06, P3 CONN_01X04, P4 CONN_01X04, P5 CONN_01X02, P6 CONN_01X04, Q1 MOSFET_N, Q2 MOSFET_N, Q3 MOSFET_N, Q4 MOSFET_N, SW1 SW_PUSH, U1 STM32F303K8, U2 MCP2551, U3 SI8234, U4 ACS714, U5 SI8234, U6 NCP1117ST50T3G, U7 MC78L15ACP, U8 NCP1117ST33T3G, U9 NCP1117ST50T3G, X1 CRYSTAL

Commit message: no message
Parts:
- removed L1, L2: INDUCTOR_SMALL, Choke_SMD:Choke_SMD_1206_Standard
- added C25: 220u, Capacitors_SMD:c_elec_8x6.5, F.Cu at (44.5, 52.7)
- added R14: 10k, RP_KiCAD_Libs:C1608, F.Cu at (59.7, 49.5)
- added R15: 10k, RP_KiCAD_Libs:C1608, F.Cu at (63.5, 49.5)
- added R16: 47k, RP_KiCAD_Libs:C1608, F.Cu at (59.7, 52.1)
- added R17: 10k, RP_KiCAD_Libs:C1608, F.Cu at (63.5, 52.1)
- C1, C16, C2, C3, C4, C7, C8: value C -> 0.1u
- C10, C11, C12, C13, C17, C18, C19, C20: value C -> 10u
- C14, C15: value C -> 470u
- C5, C6: value C -> 22p
- C9: value C -> 1n; moved to B.Cu
- P3, P4: footprint RP_KiCAD_Connector:XA_4L -> RP_KiCAD_Connector:XA_4T
- R1: value R -> 10kR
- R10, R11, R8, R9: value R -> 10
- R12: value R -> 1k
- R13, R5, R6, R7: value R -> 10k
- RP1: value R_PACK4 -> 10k
- RP2: value R_PACK4 -> 2.2k
- U7: footprint TO_SOT_Packages_SMD:SOT89-3_Housing -> TO_SOT_Packages_SMD:TO-252-2Lead
- moved U6 157.1 mm to (0.00, 100.3)
- moved Q1 126.5 mm to (7.62, 27.9)
- moved U3 126.5 mm to (7.62, 66.0)
- moved Q2 126.3 mm to (7.62, 47.0)
- moved U4 126.1 mm to (7.62, 22.9)
- moved R2 117.6 mm to (27.9, 109.2)
- moved P3 114.2 mm to (44.5, 102.9), turned to 270 degrees
- moved P5 111.9 mm to (17.8, 11.4)
- moved C16 110.2 mm to (44.5, 59.7)
- moved C15 109.7 mm to (38.1, 35.6), turned to 0 degrees
- moved C14 109.4 mm to (38.1, 24.1), turned to 0 degrees
- moved P6 109.4 mm to (40.6, 11.4)
- moved R4 108.3 mm to (40.0, 102.9)
- moved C5 105.1 mm to (3.17, 90.8)
- moved C24 102.9 mm to (16.5, 101.6), turned to 270 degrees
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Connections:
- C17 pad 1: Net-(C17-Pad1) -> /GP_PS
- C18 pad 1: Net-(C18-Pad1) -> +BATT
- U1 pad 10: /~EN -> /CURRENT_SENSE
- U1 pad 11: (no net) -> /12V_SENSE
- U1 pad 14: (no net) -> /5V_SENSE
- U1 pad 20: (no net) -> /~EN
- U4 pad 7: (no net) -> /CURRENT_SENSE
- U7 pad 1: Net-(C18-Pad1) -> +BATT
- U9 pad 3: Net-(C17-Pad1) -> /GP_PS
Routing:
- net GNDPWR: track 0.00 -> 84.0 mm
- net +BATT: track 0.00 -> 83.6 mm
- net /GD_PS: track 0.00 -> 27.9 mm
- net Net-(C13-Pad1): track 0.00 -> 8.88 mm
- net Net-(C11-Pad1): track 0.00 -> 8.88 mm
- net Net-(C10-Pad1): track 0.00 -> 4.49 mm
- net Net-(C12-Pad1): track 0.00 -> 4.49 mm
- net /OUT_B: track 0.00 -> 2.52 mm
- net /OUT_A_CS: track 0.00 -> 2.52 mm
Other:
- board outline added: 50 x 100 mm
