File: KiCAD_Projects/0.5_48_pitchAdabter/0.5_48_pitchAdabter.kicad_pcb (KiCad board)
At the start: 2 copper layers, 30.5 x 63.5 mm, 5 parts, among them P1 CONN_01X12, P2 CONN_01X12, P3 CONN_01X12, P4 CONN_01X12, U1 STM32F103_48

Commit message: no message
Routing:
- added copper zone on B.Cu, net (none)
