File: KiCAD_Projects/STMF303test/STMF303test.kicad_pcb (KiCad board)
At the start: 2 copper layers, 40 x 50 mm, 19 parts, among them P1 CONN_01X03, P2 CONN_01X07, P3 CONN_01X05, P4 CONN_01X06, P5 CONN_01X02, P6 CONN_01X02, P7 CONN_01X02, P8 CONN_01X02, SW1 SW_PUSH, U1 STM32F303K8, X1 CRYSTAL

Commit message: no message
Routing:
- added copper zone on B.Cu, net (none)
- removed copper zone on B.Cu, net GND
Changed lines of the file:
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@@
-(kicad_pcb (version 4) (host pcbnew 4.0.2-stable)
+(kicad_pcb (version 4) (host pcbnew 4.0.3-stable)
   (general
     (links 52)
     (no_connects 0)
-    (area 129.924999 54.107 172.240334 107.724333)
+    (area 129.924999 54.257 172.165334 107.649333)
     (thickness 1.6)
     (drawings 4)
@@
   )
   (setup
-    (last_trace_width 0.5)
+    (last_trace_width 0.25)
     (user_trace_width 0.5)
     (user_trace_width 1)
@@
   (segment (start 144.272 62.992) (end 141.732 60.452) (width 0.5) (layer B.Cu) (net 5))
   (segment (start 161.036 62.992) (end 158.863 62.992) (width 0.5) (layer B.Cu) (net 6))
-  (segment (start 167.132 83.312) (end 161.036 83.312) (width 0.5) (layer B.Cu) (net 7) (status C00000))
-  (segment (start 161.036 80.772) (end 167.132 80.772) (width 0.5) (layer B.Cu) (net 8) (status C00000))
+  (segment (start 167.132 83.312) (end 161.036 83.312) (width 0.5) (layer B.Cu) (net 7))
+  (segment (start 161.036 80.772) (end 167.132 80.772) (width 0.5) (layer B.Cu) (net 8))
   (segment (start 142.748 73.152) (end 145.796 73.152) (width 0.5) (layer B.Cu) (net 9))
   (segment (start 142.748 75.692) (end 145.796 75.692) (width 0.5) (layer B.Cu) (net 10))
@@
   (segment (start 161.036 68.072) (end 164.084 68.072) (width 0.5) (layer B.Cu) (net 28))
   (segment (start 164.084 65.532) (end 161.036 65.532) (width 0.5) (layer B.Cu) (net 29))
-  (zone (net 2) (net_name GND) (layer B.Cu) (hatch edge 0.508)
-    (connect_pads (clearance 0.4))
+  (zone (net 0) (net_name "") (layer B.Cu) (hatch edge 0.508)
+    (connect_pads yes (clearance 0.4))
     (min_thickness 0.2)
     (fill yes (arc_segments 16) (thermal_gap 0.508) (thermal_bridge_width 0.508))
     (polygon
       (pts
-        (xy 170 105) (xy 130 105) (xy 130 55) (xy 170 55) (xy 170 105)
+        (xy 170 105) (xy 130 105) (xy 130 55) (xy 170 55)
       )
     )
