File: KiCAD_Projects/QFPN_32_pitchAdapter/QFPN_32_pitchAdapter.kicad_pcb (KiCad board)
At the start: 2 copper layers, 16.5 x 41.9 mm, 3 parts, among them P1 CONN_01X32, P2 CONN_01X16, P3 CONN_01X16

Commit message: no message
Parts:
- moved P2 2.54 mm to (152.4, 83.8)
- moved P1 1.27 mm to (144.8, 102.9)
Routing:
- net Net-(P1-Pad7): track 5.01 -> 7.05 mm
- net Net-(P1-Pad10): track 5.01 -> 7.05 mm
- net Net-(P1-Pad9): track 3.75 -> 5.02 mm
- net Net-(P1-Pad8): track 3.75 -> 5.02 mm
- net Net-(P1-Pad23): track 5.01 -> 6.28 mm
- net Net-(P1-Pad26): track 5.01 -> 6.28 mm
- net Net-(P1-Pad25): track 3.75 -> 5.02 mm
- net Net-(P1-Pad24): track 3.75 -> 5.02 mm
- net Net-(P1-Pad6): track 6.89 -> 7.54 mm
- net Net-(P1-Pad11): track 6.89 -> 7.54 mm
- net Net-(P1-Pad27): track 6.89 -> 7.54 mm
- net Net-(P1-Pad22): track 6.89 -> 7.54 mm
- net Net-(P1-Pad29): track 11.6 -> 12.1 mm
- net Net-(P1-Pad5): track 9.22 -> 9.75 mm
- net Net-(P1-Pad28): track 9.22 -> 9.75 mm
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Other:
- board size 16.5 x 41.9 mm -> 19.1 x 41.9 mm
