File: KiCAD_Projects/STM32F103C8T_temp/STM32F103C8T_temp.sch (KiCad schematic (older format))
At the start: 11 parts, among them SW1 SW_PUSH, U1 STM32F103_48, X1 CRYSTAL, X2 CRYSTAL

Commit message: no message
Parts:
- removed C2, C3: C, symbol C
- removed X1: CRYSTAL, symbol CRYSTAL
Connections:
- net OSC32_IN: no longer names the net of U1.3 (PC14/OSC32_IN)
- net OSC32_OUT: no longer names the net of U1.4 (PC15/OSC_OUT)
Changed lines of the file:
@@
 LIBS:user
 LIBS:power
-LIBS:STMtemp-cache
+LIBS:STM32F103C8T_temp-cache
 EELAYER 25 0
 EELAYER END
@@
 VBAT
 $Comp
-L C C2
-U 1 1 5773BD64
-P 2200 3100
-F 0 "C2" H 2200 3200 40  0000 L CNN
-F 1 "C" H 2206 3015 40  0000 L CNN
-F 2 "" H 2238 2950 30  0000 C CNN
-F 3 "" H 2200 3100 60  0000 C CNN
-	1    2200 3100
-	0    1    1    0
-$EndComp
-$Comp
-L C C3
-U 1 1 5773BDBB
-P 2200 3700
-F 0 "C3" H 2200 3800 40  0000 L CNN
-F 1 "C" H 2206 3615 40  0000 L CNN
-F 2 "" H 2238 3550 30  0000 C CNN
-F 3 "" H 2200 3700 60  0000 C CNN
-	1    2200 3700
-	0    1    1    0
-$EndComp
-$Comp
-L CRYSTAL X1
-U 1 1 5773BE02
-P 2400 3400
-F 0 "X1" H 2400 3550 60  0000 C CNN
-F 1 "CRYSTAL" H 2400 3250 60  0000 C CNN
-F 2 "" H 2400 3400 60  0000 C CNN
-F 3 "" H 2400 3400 60  0000 C CNN
-	1    2400 3400
-	0    1    1    0
-$EndComp
-$Comp
-L GND #PWR01
-U 1 1 5773BEAD
-P 2000 3100
-F 0 "#PWR01" H 2000 3100 30  0001 C CNN
-F 1 "GND" H 2000 3030 30  0001 C CNN
-F 2 "" H 2000 3100 60  0000 C CNN
-F 3 "" H 2000 3100 60  0000 C CNN
-	1    2000 3100
-	0    1    1    0
-$EndComp
-$Comp
-L GND #PWR02
-U 1 1 5773BEEB
-P 2000 3700
-F 0 "#PWR02" H 2000 3700 30  0001 C CNN
-F 1 "GND" H 2000 3630 30  0001 C CNN
-F 2 "" H 2000 3700 60  0000 C CNN
-F 3 "" H 2000 3700 60  0000 C CNN
-	1    2000 3700
-	0    1    1    0
-$EndComp
-Text Label 2400 3100 0    60   ~ 0
-OSC32_IN
-Text Label 2400 3700 0    60   ~ 0
-OSC32_OUT
-Text Label 4000 3350 2    60   ~ 0
-OSC32_IN
-Text Label 4000 3450 2    60   ~ 0
-OSC32_OUT
-$Comp
 L C C4
