File: KiCAD_Projects/3WS_MD/3WS_MD.sch (KiCad schematic (older format))
At the start: 11 parts, among them SW1 SW_PUSH, U1 STM32F103_48, X1 CRYSTAL, X2 CRYSTAL

Commit message: no message
Parts:
- removed C2, C3: C, symbol C
- removed X1: CRYSTAL, symbol CRYSTAL
- added C? (x3): C, symbol C
- added P?: CONN_01X02, symbol CONN_01X02
- added P?: CONN_01X04, symbol CONN_01X04
- added R?: R, symbol R
- added U?: MCP2551, symbol MCP2551
- C1: value C -> 0.01u
- C4, C5: value C -> 22p
- R1: value R -> 10k
- R2: value R -> 1k
Connections:
- net +3.3V: now also C?.2, C?.2, C?.2
- net GND: now also C?.1, C?.1, C?.1, U?.2 (Vss), U?.8 (Rs)
- net ENC_Aa: now reaches U1.10 (PA0/WKUP/ADC12_IN0)
- net ENC_Ab: now reaches U1.11 (PA1/ADC12_IN1)
- net CURRENT_A: now reaches U1.12 (PA2/USART2_TX)
- net CURRENT_B: now reaches U1.13 (PA3/USART2_RX)
- net POT_A: now reaches U1.14 (PA4/SPI1_NSS)
- net POT_B: now reaches U1.15 (PA5/SPI1_SCK)
- net ENC_Ba: now reaches U1.16 (PA6/SPI1_MISO)
- net ENC_Bb: now reaches U1.17 (PA7/SPI1_MOSI)
- net LED: now reaches U1.18 (PB0/ADC12_IN8)
- net MOTOR_EN: now reaches U1.25 (PB12/SPI2_NSS)
- net LIMIT_A1: now reaches U1.26 (PB13/SPI2_SCK)
- net LIMIT_A2: now reaches U1.27 (PB14/SPI2_MISO)
- net LIMIT_B1: now reaches U1.28 (PB15/SPI2_MOSI)
- net LIMIT_B2: now reaches U1.29 (PA8)
- net USART_TX: now reaches U1.30 (PA9/USART1_TX)
- net USART_RX: now reaches U1.31 (PA10/USART_RX)
- net CAN_RX: now reaches U1.32 (PA11/CAN_RX/USBDM)
- net CAN_RX: now also U?.4 (RXD)
- net CAN_XT: now reaches U1.33 (PA12/CAN_TX/USBDP)
- net SPI_NSS: now reaches U1.38 (PA15/TDI)
- net SPI_SCK: now reaches U1.39 (PB3/TDO)
- net SPI_MOSI: now reaches U1.40 (PB4/NTRST)
- net SPI_MISO: now reaches U1.41 (PB5/I2C1_SMBAI)
- net PWM_A: now reaches U1.42 (PB6/I2C_SCL)
- net PWM_AN: now reaches U1.43 (PB7/I2C_SDA)
- net PWM_B: now reaches U1.45 (PB8/TIM4_CH3)
- net PWM_BN: now reaches U1.46 (PB9/TIM4_CH4)
- new net: P?.2 (P2), R?.2
- new net +5V: U?.3 (Vdd)
- new net CANH: P?.2 (P2), R?.1, U?.7 (CANH)
- new net CANL: P?.1 (P1), P?.1 (P1), U?.6 (CANL)
- new net CAN_TX: U?.1 (TXD)
- new net DGND: P?.4 (P4)
- no-connect marks 0 -> 1

Commit message: no message
Parts:
- removed C?: C, symbol C
- removed U?: MCP2551, symbol MCP2551
- added C10, C11, C12, C16, C17, C18, C19, C24, C26, C27, C28, C9: 4.7u, RP_KiCAD_Libs:C3216, symbol C
- added C13, C6: 1n, RP_KiCAD_Libs:C1608_WP, symbol C
- added C14, C15, C2, C20, C29, C3, C30, C31: 0.1u, RP_KiCAD_Libs:C1608_WP, symbol C
- added C21, C22: 470u, Capacitors_ThroughHole:C_Radial_D12.5_L25_P5, symbol C
- added C23: 100u, Capacitors_ThroughHole:C_Radial_D6.3_L11.2_P2.5, symbol C
- added C25: 100u, Capacitors_ThroughHole:C_Radial_D8_L11.5_P3.5, symbol C
- added D1, D10, D11, D12, D14: LED, RP_KiCAD_Libs:C3216, symbol LED
- added D13: DIODE, Diodes_SMD:SMA_Standard, symbol DIODE-RESCUE-3WS_MD
- added D2, D3, D4, D5, D6, D7, D8, D9: DIODE, RP_KiCAD_Libs:C3216, symbol DIODE-RESCUE-3WS_MD
- added FB1, FB2, FB3, FB4, FB5, FB6, FB7, FB8: FILTER, RP_KiCAD_Libs:C1608_WP, symbol FILTER
- added JP1, JP2: JUMPER, Connect:GS2, symbol JUMPER
- added P1, P10, P11, P12, P2, P4, P5, P9: TST, Connect:PINTST, symbol TST
- added P13: CONN_01X06, RP_KiCAD_Connector:ZH_6T, symbol CONN_01X06
- added P14, P15: CONN_01X02, RP_KiCAD_Connector:D-3200S_2L, symbol CONN_01X02
- added P16: CONN_01X04, RP_KiCAD_Connector:XA_4LC, symbol CONN_01X04
- added P3: CONN_01X18, RP_KiCAD_Connector:CardEdge_22(44type)_3.96mm_M, symbol CONN_01X18
- added P6: CONN_01X04, RP_KiCAD_Connector:D-3500D_4S, symbol CONN_01X04
- added Q1, Q2, Q3, Q4, Q5, Q6, Q7, Q8: MOSFET_N, TO_SOT_Packages_SMD:D2-PAK, symbol MOSFET_N
- added Q9: MOSFET_N, TO_SOT_Packages_SMD:SOT-23_Handsoldering, symbol MOSFET_N
- added R10, R11, R33, R4, R5: 10k, RP_KiCAD_Libs:C1608_WP, symbol R
- added R12, R13, R14, R15, R21, R22, R23, R24, R25, R26, R27, R28, R6, R7, R8, R9: 10, RP_KiCAD_Libs:C1608_WP, symbol R
- added R17, R29, R30, R31: 0, RP_KiCAD_Libs:C1608_WP, symbol R
- added R18: 470, RP_KiCAD_Libs:C1608_WP, symbol R
- added R19, R20: 4.7k, RP_KiCAD_Libs:C1608_WP, symbol R
- added R3, R34: 1k, RP_KiCAD_Libs:C1608_WP, symbol R
- added R32: 100, RP_KiCAD_Libs:C1608_WP, symbol R
- added SP1: SPEAKER, Buzzers_Beepers:Buzzer_12x9.5RM7.6, symbol SPEAKER
- added U10: NCP1117ST33T3G, TO_SOT_Packages_SMD:TO-223, symbol NCP1117ST33T3G
- added U11: NCP1117ST12T3G, TO_SOT_Packages_SMD:SOT-428, symbol NCP1117ST12T3G
- added U2, U3, U5, U6: SI8234, Housings_SOIC:SOIC-16_3.9x9.9mm_Pitch1.27mm, symbol SI8234
- added U4, U7: ACS722, Housings_SOIC:SOIC-8_3.9x4.9mm_Pitch1.27mm_ACS, symbol ACS722
- added U8: MAX3051, Housings_SOIC:SOIC-8_3.9x4.9mm_Pitch1.27mm, symbol MAX3051
- added U9: SW_ROTARY_16, Buttons_Switches_ThroughHole:rotary_0F, symbol SW_ROTARY_16
- C1: value 0.01u -> 0.1u; footprint (none) -> RP_KiCAD_Libs:C1608_WP
- C4, C5, R1, R2: footprint (none) -> RP_KiCAD_Libs:C1608_WP
- C7, C8: renamed from C?; value C -> 0.1u; footprint (none) -> RP_KiCAD_Libs:C1608_WP
- P7: renamed from P?; footprint (none) -> Pin_Headers:Pin_Header_Straight_1x02
- P8: renamed from P?; footprint (none) -> RP_KiCAD_Connector:XA_4LC
- R16: renamed from R?; value R -> 60; footprint (none) -> RP_KiCAD_Libs:C1608_WP
- SW1: footprint (none) -> Buttons_Switches_SMD:RP_SMD_Button
- U1: footprint MODULE -> Housings_QFP:LQFP-48_7x7mm_Pitch0.5mm
- X2: footprint (none) -> Crystals:ABM3_2pads
Connections:
- net CAN_XT is gone; now on net CAN_TX: U1.33 (PA12/CAN_TX/USBDP)
- net DGND is gone; now on net CANL: P8.4 (P4)
- net VBAT is gone; now on net +3.3V: U1.1 (VBAT)
- net +3.3V: now also C13.2, C14.2, C15.2, C2.2, C20.2, C26.1, C29.2, C3.2, C30.2, C31.2, C6.2, D10.1 (A), P13.2 (P2), P3.2 (P2), P5.1, R17.1, R30.1, U10.2 (VO), U2.3 (VDDI), U2.8 (VDDI), U3.3 (VDDI), U3.8 (VDDI), U4.8 (VCC), U5.3 (VDDI), U5.8 (VDDI), U6.3 (VDDI), U6.8 (VDDI), U7.8 (VCC), U8.3 (VCC)
- net CANH: now also P8.3 (P3), JP1.1, P16.3 (P3), U8.7 (CANH); no longer P8.2 (P2)
- net CANL: now also JP2.1, P16.4 (P4), U8.6 (CANL); no longer P8.1 (P1)
- net CAN_RX: now also U8.4 (RXD)
- net CAN_TX: now also U8.1 (TXD)
- net CURRENT_A: now also C6.1, P1.1, U4.7 (VIOUT)
- net CURRENT_B: now also C13.1, P2.1, U7.7 (VIOUT)
- net ENC_Aa: now also P3.5 (P5)
- net ENC_Ab: now also P3.6 (P6)
- net ENC_Ba: now also P3.9 (P9)
- net ENC_Bb: now also P3.10 (P10)
- net GND: now also P8.1 (P1), C14.1, C15.1, C2.1, C20.1, C23.2, C24.2, C26.2, C29.1, C3.1, C30.1, C31.1, P13.1 (P1), P16.1 (P1), P3.1 (P1), P9.1, Q9.S, R10.2, R11.2, R18.2, R19.2, R29.2, R3.2, R31.2, R33.2, R34.2, R4.2, R5.2, U10.1 (GND), U2.4 (GNDI), U3.4 (GNDI), U4.5 (GND), U5.4 (GNDI), U6.4 (GNDI), U7.5 (GND), U8.2 (GND), U8.8 (RS), U9.2 (C), U9.5 (C)
- net LIMIT_A1: now also P3.3 (P3)
- net LIMIT_A2: now also P3.4 (P4)
- net LIMIT_B1: now also P3.7 (P7)
- net LIMIT_B2: now also P3.8 (P8)
- net MOTOR_EN: now also U2.5 (DISABLE), U3.5 (DISABLE), U5.5 (DISABLE), U6.5 (DISABLE)
- net PWM_A: now also U1.45 (PB8/TIM4_CH3), U2.1 (PWM); no longer U1.42 (PB6/I2C_SCL)
- net PWM_AN: now also U1.46 (PB9/TIM4_CH4), U3.1 (PWM); no longer U1.43 (PB7/I2C_SDA)
- net PWM_B: now also U1.42 (PB6/I2C_SCL), U5.1 (PWM); no longer U1.45 (PB8/TIM4_CH3)
- net PWM_BN: now also U1.43 (PB7/I2C_SDA), U6.1 (PWM); no longer U1.46 (PB9/TIM4_CH4)
- net SWCLK: now also P13.3 (P3)
- net SWDIO: now also P13.4 (P4)
- net USART_RX: now also P13.6 (P6)
- net USART_TX: now also P13.5 (P5)
- net SEL_1: now reaches U1.19 (PB1/ADC12_IN9)
- net SEL_1: now also U9.3 (1)
- net SEL_2: now reaches U1.20 (PB2/BOOT1)
- net SEL_2: now also U9.1 (2)
- net SEL_4: now reaches U1.21 (PB10/USART3_TX/I2C_SCL)
- net SEL_4: now also U9.4
- net SEL_8: now reaches U1.22 (PB11/USART3_RX/I2C2_SDA)
- net SEL_8: now also U9.6 (8)
- net LED renamed BUZZER
- net BUZZER: now also R32.2
- net OSC32_IN: no longer names the net of U1.3 (PC14/OSC32_IN)
- net OSC32_OUT: no longer names the net of U1.4 (PC15/OSC_OUT)
- net POT_A renamed LED_A
- net LED_A: now also D14.1 (A)
- net POT_B renamed LED_B
- net LED_B: now also D1.1 (A)
- new net: R7.2, U2.10 (VOB)
- new net: C10.1, D6.2 (K), U2.11 (VDDB)
- new net: C9.2, Q1.S, Q2.D, U2.14 (GNDA), U4.1 (IP+), U4.2 (IP+)
- new net: R6.2, U2.15 (VOA)
- new net: C9.1, D2.2 (K), U2.16 (VDDA)
- new net: R4.1, U2.6 (DT)
- new net: FB1.2, Q1.G
- new net: FB2.2, Q2.G
- new net: D2.1 (A), R21.2
- new net: FB2.1, R7.1
- new net: FB1.1, R6.1
- new net: R9.2, U3.10 (VOB)
- new net: C12.1, D7.2 (K), U3.11 (VDDB)
- new net: R8.2, U3.15 (VOA)
- new net: C11.1, D3.2 (K), U3.16 (VDDA)
- new net: R5.1, U3.6 (DT)
- new net: FB3.2, Q3.G
- new net: FB4.2, Q4.G
- new net: D3.1 (A), R22.2
- new net: FB4.1, R9.1
- new net: FB3.1, R8.1
- new net: R13.2, U5.10 (VOB)
- new net: C17.1, D8.2 (K), U5.11 (VDDB)
- new net: C16.2, Q5.S, Q6.D, U5.14 (GNDA), U7.1 (IP+), U7.2 (IP+)
- new net: R12.2, U5.15 (VOA)
- new net: C16.1, D4.2 (K), U5.16 (VDDA)
- new net: R10.1, U5.6 (DT)
- new net: FB5.2, Q5.G
- new net: FB6.2, Q6.G
- new net: D4.1 (A), R24.2
- new net: FB6.1, R13.1
- new net: FB5.1, R12.1
- new net: R15.2, U6.10 (VOB)
- new net: C19.1, D9.2 (K), U6.11 (VDDB)
- new net: R14.2, U6.15 (VOA)
- new net: C18.1, D5.2 (K), U6.16 (VDDA)
- new net: R11.1, U6.6 (DT)
- new net: FB7.2, Q7.G
- new net: FB8.2, Q8.G
- new net: D5.1 (A), R25.2
- new net: FB8.1, R15.1
- new net: FB7.1, R14.1
- new net: C23.1, C24.1, D13.2 (K), P4.1, U10.3 (VI)
- new net: D1.2 (K), R3.1
- new net: D7.1 (A), R27.2
- new net: D6.1 (A), R23.2
- new net: D9.1 (A), R26.2
- new net: D8.1 (A), R28.2
- new net: D10.2 (K), R18.1
- new net: D11.2 (K), R19.1
- new net: D12.2 (K), R20.1
- new net: JP1.2, P3.11 (P11)
- new net: JP2.2, P3.12 (P12)
- new net: R17.2, R29.1, U4.6 (BW_SEL)
- new net: R30.2, R31.1, U7.6 (BW_SEL)
- new net: Q9.D, SP1.2
- new net: Q9.G, R32.1, R33.1
- new net: D14.2 (K), R34.1
- new net +12V: D11.1 (A), D13.1 (A), P16.2 (P2), P3.13 (P13), P8.2 (P2), SP1.1
- new net +BATT: C21.1, C22.1, C27.1, P10.1, P6.2 (P2), P6.4 (P4), Q1.D, Q3.D, Q5.D, Q7.D, U11.3 (VI)
- new net GD_12V: C25.1, C28.1, D12.1 (A), P12.1, R21.1, R22.1, R23.1, R24.1, R25.1, R26.1, R27.1, R28.1, U11.2 (VO)
- new net GNDPWR: C10.2, C12.2, C17.2, C19.2, C21.2, C22.2, C25.2, C27.2, C28.2, P11.1, P6.1 (P1), P6.3 (P3), Q2.S, Q4.S, Q6.S, Q8.S, R20.2, U11.1 (GND), U2.9 (GNCB), U3.9 (GNCB), U5.9 (GNCB), U6.9 (GNCB)
- new net OUT_A: P14.1 (P1), U4.3 (IP-), U4.4 (IP-)
- new net OUT_AN: C11.2, P14.2 (P2), Q3.S, Q4.D, U3.14 (GNDA)
- new net OUT_B: P15.1 (P1), U7.3 (IP-), U7.4 (IP-)
- new net OUT_BN: C18.2, P15.2 (P2), Q7.S, Q8.D, U6.14 (GNDA)
- no-connect marks 1 -> 25
Other:
- note added: "ACS"
- note added: "STM"
- moved on the sheet: C1, C4, C5, C7, C8, P7, P8, R1, R16, R2, SW1, U1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
