File: KiCAD_Projects/IRswitch/IRswitch.kicad_pcb (KiCad board)
At the start: 2 copper layers, 39.4 x 45.7 mm, 14 parts, among them IC1 ATMEGA168-P, P1 CONN_01X02, P2 CONN_01X03, P3 CONN_01X05, Q1 MOSFET_N, X1 CRYSTAL

Commit message: no message
Routing:
- net Net-(RL1-Pad10): track 0.00 -> 8.89 mm
- net Net-(RL1-Pad7): track 0.00 -> 8.26 mm
- net Net-(RL1-Pad12): track 0.00 -> 5.72 mm
Changed lines of the file:
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@@
     (thickness 1.6)
     (drawings 4)
-    (tracks 69)
+    (tracks 73)
     (zones 0)
     (modules 14)
@@
   )
   (setup
-    (last_trace_width 0.5)
+    (last_trace_width 1)
     (user_trace_width 0.5)
     (user_trace_width 1)
+    (user_trace_width 3)
     (trace_clearance 0.2)
-    (zone_clearance 0.508)
+    (zone_clearance 0.4)
     (zone_45_only no)
     (trace_min 0.2)
@@
   (segment (start 143.51 62.23) (end 139.7 66.04) (width 0.5) (layer B.Cu) (net 1))
   (segment (start 139.7 66.04) (end 139.7 69.83) (width 0.5) (layer B.Cu) (net 1))
-  (segment (start 140.97 71.1) (end 139.7 69.83) (width 0.5) (layer B.Cu) (net 1) (status 400000))
-  (segment (start 149.225 67.945) (end 151.13 69.85) (width 0.5) (layer B.Cu) (net 1) (status 400000))
+  (segment (start 140.97 71.1) (end 139.7 69.83) (width 0.5) (layer B.Cu) (net 1))
+  (segment (start 149.225 67.945) (end 151.13 69.85) (width 0.5) (layer B.Cu) (net 1))
   (segment (start 151.13 69.85) (end 153.035 69.85) (width 0.5) (layer B.Cu) (net 1))
-  (segment (start 154.285 65.405) (end 153.035 66.655) (width 0.5) (layer B.Cu) (net 1) (status 400000))
+  (segment (start 154.285 65.405) (end 153.035 66.655) (width 0.5) (layer B.Cu) (net 1))
   (segment (start 153.035 66.655) (end 153.035 69.85) (width 0.5) (layer B.Cu) (net 1))
   (segment (start 151.13 85.09) (end 153.035 83.185) (width 0.5) (layer B.Cu) (net 1))
   (segment (start 153.035 69.85) (end 153.035 83.185) (width 0.5) (layer B.Cu) (net 1))
-  (segment (start 138.43 80.645) (end 136.525 82.55) (width 0.5) (layer B.Cu) (net 1) (status 400000))
+  (segment (start 138.43 80.645) (end 136.525 82.55) (width 0.5) (layer B.Cu) (net 1))
   (segment (start 136.525 82.55) (end 136.525 83.82) (width 0.5) (layer B.Cu) (net 1))
   (segment (start 136.525 83.82) (end 137.795 85.09) (width 0.5) (layer B.Cu) (net 1))
   (segment (start 137.795 85.09) (end 151.13 85.09) (width 0.5) (layer B.Cu) (net 1))
-  (segment (start 140.97 71.1) (end 140.97 72.41) (width 1) (layer B.Cu) (net 1) (status C00000))
-  (segment (start 141.29 80.24114) (end 140.88614 80.645) (width 0.5) (layer B.Cu) (net 1) (status 400000))
-  (segment (start 140.88614 80.645) (end 138.43 80.645) (width 0.5) (layer B.Cu) (net 1) (status 800000))
+  (segment (start 140.97 71.1) (end 140.97 72.41) (width 1) (layer B.Cu) (net 1))
+  (segment (start 141.29 80.24114) (end 140.88614 80.645) (width 0.5) (layer B.Cu) (net 1))
+  (segment (start 140.88614 80.645) (end 138.43 80.645) (width 0.5) (layer B.Cu) (net 1))
   (segment (start 143.51 57.785) (end 143.51 62.23) (width 0.5) (layer B.Cu) (net 1))
   (segment (start 143.51 62.23) (end 149.225 67.945) (width 0.5) (layer B.Cu) (net 1))
@@
   (segment (start 154.305 65.385) (end 154.285 65.405) (width 1) (layer B.Cu) (net 1))
   (segment (start 154.285 65.405) (end 156.845 65.405) (width 0.5) (layer B.Cu) (net 1))
-  (segment (start 144.145 69.31406) (end 145.31594 70.485) (width 0.5) (layer B.Cu) (net 2) (status 400000))
-  (segment (start 145.31594 70.485) (end 149.225 70.485) (width 0.5) (layer B.Cu) (net 2) (status 800000))
-  (segment (start 140.97 68.6) (end 143.43094 68.6) (width 0.5) (layer B.Cu) (net 2) (status 400000))
-  (segment (start 143.43094 68.6) (end 144.145 69.31406) (width 0.5) (layer B.Cu) (net 2) (status 800000))
-  (segment (start 144.145 74.19594) (end 143.43094 74.91) (width 0.5) (layer B.Cu) (net 3) (status 400000))
-  (segment (start 143.43094 74.91) (end 140.97 74.91) (width 0.5) (layer B.Cu) (net 3) (status 800000))
-  (segment (start 149.225 73.025) (end 145.31594 73.025) (width 0.5) (layer B.Cu) (net 3) (status 400000))
-  (segment (start 145.31594 73.025) (end 144.145 74.19594) (width 0.5) (layer B.Cu) (net 3) (status 800000))
-  (segment (start 151.785 65.405) (end 151.765 65.425) (width 0.5) (layer B.Cu) (net 4) (status C00000))
-  (segment (start 151.765 65.425) (end 151.765 67.945) (width 0.5) (layer B.Cu) (net 4) (status 400000))
-  (segment (start 154.305 67.945) (end 156.845 67.945) (width 0.5) (layer B.Cu) (net 4) (status 800000))
+  (segment (start 144.145 69.31406) (end 145.31594 70.485) (width 0.5) (layer B.Cu) (net 2))
+  (segment (start 145.31594 70.485) (end 149.225 70.485) (width 0.5) (layer B.Cu) (net 2))
+  (segment (start 140.97 68.6) (end 143.43094 68.6) (width 0.5) (layer B.Cu) (net 2))
+  (segment (start 143.43094 68.6) (end 144.145 69.31406) (width 0.5) (layer B.Cu) (net 2))
+  (segment (start 144.145 74.19594) (end 143.43094 74.91) (width 0.5) (layer B.Cu) (net 3))
+  (segment (start 143.43094 74.91) (end 140.97 74.91) (width 0.5) (layer B.Cu) (net 3))
+  (segment (start 149.225 73.025) (end 145.31594 73.025) (width 0.5) (layer B.Cu) (net 3))
+  (segment (start 145.31594 73.025) (end 144.145 74.19594) (width 0.5) (layer B.Cu) (net 3))
+  (segment (start 151.785 65.405) (end 151.765 65.425) (width 0.5) (layer B.Cu) (net 4))
+  (segment (start 151.765 65.425) (end 151.765 67.945) (width 0.5) (layer B.Cu) (net 4))
+  (segment (start 154.305 67.945) (end 156.845 67.945) (width 0.5) (layer B.Cu) (net 4))
   (via (at 154.305 67.945) (size 1.2) (drill 0.8) (layers F.Cu B.Cu) (net 4))
   (segment (start 151.765 67.945) (end 154.305 67.945) (width 0.5) (layer F.Cu) (net 4))
   (via (at 151.765 67.945) (size 1.2) (drill 0.8) (layers F.Cu B.Cu) (net 4))
-  (segment (start 156.845 67.945) (end 156.845 70.485) (width 0.5) (layer B.Cu) (net 4) (status C00000))
+  (segment (start 156.845 67.945) (end 156.845 70.485) (width 0.5) (layer B.Cu) (net 4))
   (segment (start 138.43 62.865) (end 140.97 60.325) (width 0.5) (layer B.Cu) (net 4))
   (segment (start 151.765 45.085) (end 151.765 43.18) (width 0.5) (layer B.Cu) (net 4))
@@
   (segment (start 151.765 65.385) (end 151.785 65.405) (width 1) (layer B.Cu) (net 4))
   (segment (start 151.765 45.085) (end 151.765 45.72) (width 1) (layer B.Cu) (net 4))
-  (segment (start 138.43 75.565) (end 140.10386 77.23886) (width 0.5) (layer B.Cu) (net 5) (status 400000))
-  (segment (start 140.10386 77.23886) (end 142.24 77.23886) (width 0.5) (layer B.Cu) (net 5) (status 800000))
+  (segment (start 138.43 75.565) (end 140.10386 77.23886) (width 0.5) (layer B.Cu) (net 5))
+  (segment (start 140.10386 77.23886) (end 142.24 77.23886) (width 0.5) (layer B.Cu) (net 5))
   (segment (start 133.35 60.325) (end 138.43 65.405) (width 0.5) (layer B.Cu) (net 5))
   (segment (start 138.43 65.405) (end 138.43 75.565) (width 0.5) (layer B.Cu) (net 5))
@@
   (segment (start 146.05 83.185) (end 149.225 83.185) (width 0.5) (layer B.Cu) (net 10))
   (segment (start 146.05 83.185) (end 146.05 80.645) (width 0.5) (layer B.Cu) (net 10))
-  (segment (start 143.19 80.24114) (end 143.19 81.6) (width 0.5) (layer B.Cu) (net 26) (status 400000))
+  (segment (start 143.19 80.24114) (end 143.19 81.6) (width 0.5) (layer B.Cu) (net 26))
   (segment (start 143.19 81.6) (end 141.605 83.185) (width 0.5) (layer B.Cu) (net 26))
-  (segment (start 141.605 83.185) (end 138.43 83.185) (width 0.5) (layer B.Cu) (net 26) (status 800000))
+  (segment (start 141.605 83.185) (end 138.43 83.185) (width 0.5) (layer B.Cu) (net 26))
+  (segment (start 130.81 70.485) (end 130.81 64.77) (width 1) (layer B.Cu) (net 27) (status 400000))
+  (segment (start 130.81 70.485) (end 130.81 73.66) (width 1) (layer B.Cu) (net 27) (status 400000))
+  (segment (start 130.81 62.865) (end 130.81 54.61) (width 1) (layer B.Cu) (net 28) (status 400000))
+  (segment (start 130.81 75.565) (end 130.81 81.28) (width 1) (layer B.Cu) (net 30) (status 400000))
   (zone (net 1) (net_name GND) (layer B.Cu) (hatch edge 0.508)
-    (connect_pads (clearance 0.508))
-    (min_thickness 0.254)
+    (connect_pads (clearance 0.4))
+    (min_thickness 0.2)
     (fill yes (arc_segments 16) (thermal_gap 0.508) (thermal_bridge_width 0.508))
     (polygon

Commit message: no message
Parts:
- added P4: CONN_01X02, Connect:bornier2, F.Cu at (124.5, 59.1)
- added P5: CONN_01X02, Connect:bornier2, F.Cu at (124.5, 71.8)
Connections:
- IC1 pad 11: Net-(IC1-Pad11) -> (no net)
- IC1 pad 12: Net-(IC1-Pad12) -> (no net)
- IC1 pad 13: Net-(IC1-Pad13) -> (no net)
- IC1 pad 15: Net-(IC1-Pad15) -> (no net)
- IC1 pad 16: Net-(IC1-Pad16) -> (no net)
- IC1 pad 17: Net-(IC1-Pad17) -> (no net)
- IC1 pad 18: Net-(IC1-Pad18) -> (no net)
- IC1 pad 19: Net-(IC1-Pad19) -> (no net)
- IC1 pad 23: Net-(IC1-Pad23) -> (no net)
- IC1 pad 24: Net-(IC1-Pad24) -> (no net)
- IC1 pad 25: Net-(IC1-Pad25) -> (no net)
- IC1 pad 26: Net-(IC1-Pad26) -> (no net)
- IC1 pad 27: Net-(IC1-Pad27) -> (no net)
- IC1 pad 28: Net-(IC1-Pad28) -> (no net)
- IC1 pad 5: Net-(IC1-Pad5) -> (no net)
- IC1 pad 6: Net-(IC1-Pad6) -> (no net)
- RL1 pad 1: Net-(D1-Pad1) -> +5V
- RL1 pad 10: Net-(RL1-Pad10) -> (no net)
- RL1 pad 6: +5V -> Net-(D1-Pad1)
Routing:
- net Net-(P4-Pad2): track 0.00 -> 14.8 mm
- net +5V: track 80.8 -> 93.5 mm
- net Net-(RL1-Pad10): track 8.89 -> 0.00 mm
- net Net-(D1-Pad1): track 21.8 -> 29.8 mm
- net Net-(P5-Pad1): track 5.72 -> 8.98 mm
- net GND: track 101.8 -> 104.7 mm
- net Net-(P4-Pad1): track 8.26 -> 8.98 mm
- net (no net): vias 0 -> 4
Other:
- board size 39.4 x 45.7 mm -> 50 x 50 mm

Commit message: no message
Routing:
- added copper zone on B.Cu, net (none)
- removed copper zone on B.Cu, net GND
Changed lines of the file:
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@@
-(kicad_pcb (version 4) (host pcbnew 4.0.2-stable)
+(kicad_pcb (version 4) (host pcbnew 4.0.3-stable)
   (general
     (links 35)
     (no_connects 0)
-    (area 119.924999 39.924999 170.075001 90.075001)
+    (area 118.405 34.209999 170.075001 90.075001)
     (thickness 1.6)
     (drawings 4)
@@
   )
   (setup
-    (last_trace_width 0.5)
+    (last_trace_width 0.25)
     (user_trace_width 0.5)
     (user_trace_width 1)
@@
   (via (at 125 45) (size 4) (drill 3) (layers F.Cu B.Cu) (net 0))
   (via (at 165 45) (size 4) (drill 3) (layers F.Cu B.Cu) (net 0))
-  (segment (start 140.97 71.1) (end 139.72 71.1) (width 0.5) (layer B.Cu) (net 1) (status 400000))
+  (segment (start 140.97 71.1) (end 139.72 71.1) (width 0.5) (layer B.Cu) (net 1))
   (segment (start 139.7 71.08) (end 139.7 69.83) (width 0.5) (layer B.Cu) (net 1))
   (segment (start 139.72 71.1) (end 139.7 71.08) (width 0.5) (layer B.Cu) (net 1))
-  (segment (start 154.285 65.405) (end 154.285 66.655) (width 0.5) (layer B.Cu) (net 1) (status 400000))
+  (segment (start 154.285 65.405) (end 154.285 66.655) (width 0.5) (layer B.Cu) (net 1))
   (segment (start 154.285 66.655) (end 153.035 66.655) (width 0.5) (layer B.Cu) (net 1))
-  (segment (start 149.225 67.945) (end 146.685 67.945) (width 0.5) (layer B.Cu) (net 1) (status 400000))
+  (segment (start 149.225 67.945) (end 146.685 67.945) (width 0.5) (layer B.Cu) (net 1))
   (segment (start 143.51 64.77) (end 143.51 62.23) (width 0.5) (layer B.Cu) (net 1))
   (segment (start 146.685 67.945) (end 143.51 64.77) (width 0.5) (layer B.Cu) (net 1))
@@
   (segment (start 143.19 81.6) (end 141.605 83.185) (width 0.5) (layer B.Cu) (net 11))
   (segment (start 141.605 83.185) (end 138.43 83.185) (width 0.5) (layer B.Cu) (net 11))
-  (segment (start 124.46 56.515) (end 130.81 62.865) (width 1) (layer B.Cu) (net 12) (status C00000))
-  (segment (start 124.46 61.595) (end 121.92 64.135) (width 1) (layer B.Cu) (net 13) (status 400000))
-  (segment (start 121.92 71.755) (end 124.46 74.295) (width 1) (layer B.Cu) (net 13) (status 800000))
+  (segment (start 124.46 56.515) (end 130.81 62.865) (width 1) (layer B.Cu) (net 12))
+  (segment (start 124.46 61.595) (end 121.92 64.135) (width 1) (layer B.Cu) (net 13))
+  (segment (start 121.92 71.755) (end 124.46 74.295) (width 1) (layer B.Cu) (net 13))
   (segment (start 121.92 64.135) (end 121.92 71.755) (width 1) (layer B.Cu) (net 13))
   (segment (start 124.46 69.215) (end 130.81 75.565) (width 1) (layer B.Cu) (net 14))
-  (zone (net 1) (net_name GND) (layer B.Cu) (hatch edge 0.508)
+  (zone (net 0) (net_name "") (layer B.Cu) (hatch edge 0.508)
     (connect_pads (clearance 0.4))
     (min_thickness 0.2)
@@
     (polygon
       (pts
-        (xy 170 90) (xy 120 90) (xy 120 40) (xy 170 40) (xy 170 90)
+        (xy 170 90) (xy 120 90) (xy 120 40) (xy 170 40)
       )
     )
