File: KiCAD_Projects/ISO_DCDC/_saved_ISO_DCDC.sch (KiCad schematic (older format))
At the start: 64 parts, among them IC1 PC817, IC2 PC817, IC3 PC817, IC4 PC817, P1 CONN_01X01, P10 CONN_01X02, P11 CONN_01X02, P12 CONN_01X02, P19 CONN_01X01, P20 CONN_01X01, P21 CONN_01X02, P22 CONN_01X01, P23 CONN_01X01, P25 CONN_01X01, P26 CONN_01X01, P27 CONN_01X02, P30 CONN_01X01, P4 CONN_01X02, P5 CONN_01X02, P6 CONN_01X04, P7 CONN_01X04, P8 CONN_01X01, Q1 MOSFET_N, U1 V23076-D3001-D142, U3 V23076-D3001-D142

Commit message: no message
Parts:
- removed P12, P27: CONN_01X02, RP_KiCAD_Connector:XA_2T, symbol CONN_01X02
- added D6: LED, LEDs:LED-3MM, symbol LED
- added IC5: PC817, Opto-Devices:Optocoupler_SMD_HandSoldering_KPC357_LTV35x_PC357_SingleChannel, symbol PC817
- added P12, P2, P3, P9: CONN_01X01, Connect:1pin, symbol CONN_01X01
- added P13: CONN_01X04, RP_KiCAD_Connector:XA_4LC, symbol CONN_01X04
- added P14, P15, P16: CONN_01X02, RP_KiCAD_Connector:XA_2T, symbol CONN_01X02
- added R5: 2.2k, RP_KiCAD_Libs:C1608_WP, symbol R
- added U2: V23076-D3001-D142, Relays_ThroughHole:V23076-A3001-D142, symbol V23076-D3001-D142
- DCDC4: footprint Converters_DCDC_ACDC:MGS15 -> RP_KiCAD_Libs:MGS30
- L1: footprint Choke_Toroid_ThroughHole:Choke_Toroid_10x25mm_Vertical -> Choke_Toroid_ThroughHole:Choke_Toroid_horizontal_Diameter26mm
- R19: footprint RP_KiCAD_Libs:C1608_WP -> RP_KiCAD_Libs:0204_2f5
- R3, R4: footprint RP_KiCAD_Libs:0204_2f7 -> RP_KiCAD_Libs:0204_2f5
Connections:
- net 15V: now also DCDC3.6 (+Vin), IC4.4; no longer IC3.4
- net 5V: now also P15.2 (P2)
- net 5V_GND: now also P15.1 (P1)
- net GNDPWR: now also IC5.2, P12.1 (P1), P3.1 (P1), R5.2
- net POWER_EN_HIGH: now also IC5.1, U2.2 (A2)
- net POWER_EN_LOW: now also U2.1 (A1)
- net at C3.1, C4.1, C6.1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: no longer DCDC3.6 (+Vin)
- net at IC2.3: now also IC3.4; no longer IC1.4
- net at IC2.4: now also IC1.3; no longer IC3.3
- net at IC4.3: now also IC1.4; no longer R19.1
- net at IC4.2: now also P13.2 (P2)
- net at R22.1: now also P13.1 (P1)
- net 12V renamed 12V_CAN
- net 12V_CAN: now also P14.2 (P2)
- net 12V_GND renamed 12V_CAN_GND
- net 12V_CAN_GND: now also P14.1 (P1)
- net 5V_RasPi renamed 12V_RasPi
- net 12V_RasPi: now also P16.2 (P2)
- net 5V_RasPi_GND renamed 12V_RasPi_GND
- net 12V_RasPi_GND: now also P16.1 (P1)
- new net: IC3.3, R19.1
- new net: P9.1 (P1), U2.4 (COM)
- new net: D6.1 (A), P2.1 (P1), U2.5 (NO)
- new net: D6.2 (K), R5.1
- new net: IC5.3, P13.4 (P4)
- new net: IC5.4, P13.3 (P3)
Other:
- moved on the sheet: D1, D9, P10, P11, P25, P26, R1, R18
