File: KiCAD_Projects/CNC_LIMIT/CNC_LIMIT.sch (KiCad schematic (older format))
At the start: 0 parts

Commit message: no message
Parts:
- added D1, D2, D3, D4: LED, LEDs:LED-3MM, symbol LED
- added P1, P2: CONN_01X03, RP_KiCAD_Connector:XH_3L, symbol CONN_01X03
- added R1, R2, R3, R4: R, RP_KiCAD_Libs:0204_2f5, symbol R
Connections:
- new net: D2.2 (K), R2.1
- new net: D4.2 (K), R4.1
- new net +5V: D1.1 (A), D2.1 (A), D3.1 (A), D4.1 (A), P1.2 (P2), P2.2 (P2)
- new net GND: P1.1 (P1), P2.1 (P1), R1.1, R2.2, R3.1, R4.2
- new net OUT: D1.2 (K), D3.2 (K), P1.3 (P3), P2.3 (P3), R1.2, R3.2

Commit message: no message
Parts:
- P1, P2: footprint RP_KiCAD_Connector:XH_3L -> Crystals:Resonator_7.2x3mm
- R2, R4: footprint RP_KiCAD_Libs:0204_2f5 -> RP_KiCAD_Libs:C1608
Changed lines of the file:
@@
 F 0 "R2" V 6730 3000 40  0000 C CNN
 F 1 "R" V 6657 3001 40  0000 C CNN
-F 2 "RP_KiCAD_Libs:0204_2f5" V 6580 3000 30  0001 C CNN
+F 2 "RP_KiCAD_Libs:C1608" V 6580 3000 30  0001 C CNN
 F 3 "" H 6650 3000 30  0000 C CNN
 	1    6650 3000
@@
 F 0 "P1" H 5100 2600 50  0000 C CNN
 F 1 "CONN_01X03" V 5200 2400 50  0000 C CNN
-F 2 "RP_KiCAD_Connector:XH_3L" H 5100 2400 50  0001 C CNN
+F 2 "Crystals:Resonator_7.2x3mm" H 5100 2400 50  0001 C CNN
 F 3 "" H 5100 2400 50  0000 C CNN
 	1    5100 2400
@@
 F 0 "R4" V 6880 4600 40  0000 C CNN
 F 1 "R" V 6807 4601 40  0000 C CNN
-F 2 "RP_KiCAD_Libs:0204_2f5" V 6730 4600 30  0001 C CNN
+F 2 "RP_KiCAD_Libs:C1608" V 6730 4600 30  0001 C CNN
 F 3 "" H 6800 4600 30  0000 C CNN
 	1    6800 4600
@@
 F 0 "P2" H 5250 4200 50  0000 C CNN
 F 1 "CONN_01X03" V 5350 4000 50  0000 C CNN
-F 2 "RP_KiCAD_Connector:XH_3L" H 5250 4000 50  0001 C CNN
+F 2 "Crystals:Resonator_7.2x3mm" H 5250 4000 50  0001 C CNN
 F 3 "" H 5250 4000 50  0000 C CNN
 	1    5250 4000

Commit message: no message
Parts:
- removed D3, D4: LED, LEDs:LED-3MM, symbol LED
- removed P2: CONN_01X03, Crystals:Resonator_7.2x3mm, symbol CONN_01X03
- removed R3: R, RP_KiCAD_Libs:0204_2f5, symbol R
- removed R4: R, RP_KiCAD_Libs:C1608, symbol R
- P1: footprint Crystals:Resonator_7.2x3mm -> Pin_Headers:Pin_Header_Straight_1x03
- R1: footprint RP_KiCAD_Libs:0204_2f5 -> RP_KiCAD_Libs:C1608_WP
- R2: footprint RP_KiCAD_Libs:C1608 -> RP_KiCAD_Libs:C1608_WP
Changed lines of the file:
@@
 F 0 "R2" V 6730 3000 40  0000 C CNN
 F 1 "R" V 6657 3001 40  0000 C CNN
-F 2 "RP_KiCAD_Libs:C1608" V 6580 3000 30  0001 C CNN
+F 2 "RP_KiCAD_Libs:C1608_WP" V 6580 3000 30  0001 C CNN
 F 3 "" H 6650 3000 30  0000 C CNN
 	1    6650 3000
@@
 F 0 "R1" V 6130 2300 40  0000 C CNN
 F 1 "R" V 6057 2301 40  0000 C CNN
-F 2 "RP_KiCAD_Libs:0204_2f5" V 5980 2300 30  0001 C CNN
+F 2 "RP_KiCAD_Libs:C1608_WP" V 5980 2300 30  0001 C CNN
 F 3 "" H 6050 2300 30  0000 C CNN
 	1    6050 2300
@@
 F 0 "P1" H 5100 2600 50  0000 C CNN
 F 1 "CONN_01X03" V 5200 2400 50  0000 C CNN
-F 2 "Crystals:Resonator_7.2x3mm" H 5100 2400 50  0001 C CNN
+F 2 "Pin_Headers:Pin_Header_Straight_1x03" H 5100 2400 50  0001 C CNN
 F 3 "" H 5100 2400 50  0000 C CNN
 	1    5100 2400
@@
 	0    -1   -1   0
 $EndComp
-$Comp
-L LED D4
-U 1 1 57A31437
-P 6800 4250
-F 0 "D4" H 6800 4350 50  0000 C CNN
-F 1 "LED" H 6800 4150 50  0000 C CNN
-F 2 "LEDs:LED-3MM" H 6800 4250 60  0001 C CNN
-F 3 "" H 6800 4250 60  0000 C CNN
-	1    6800 4250
-	0    1    1    0
-$EndComp
-$Comp
-L LED D3
-U 1 1 57A3143D
-P 6200 4250
-F 0 "D3" H 6200 4350 50  0000 C CNN
-F 1 "LED" H 6200 4150 50  0000 C CNN
-F 2 "LEDs:LED-3MM" H 6200 4250 60  0001 C CNN
-F 3 "" H 6200 4250 60  0000 C CNN
-	1    6200 4250
-	0    -1   -1   0
-$EndComp
-$Comp
-L R R4
-U 1 1 57A31443
-P 6800 4600
-F 0 "R4" V 6880 4600 40  0000 C CNN
-F 1 "R" V 6807 4601 40  0000 C CNN
-F 2 "RP_KiCAD_Libs:C1608" V 6730 4600 30  0001 C CNN
-F 3 "" H 6800 4600 30  0000 C CNN
-	1    6800 4600
-	1    0    0    -1
-$EndComp
-$Comp
-L R R3
-U 1 1 57A31449
-P 6200 3900
-F 0 "R3" V 6280 3900 40  0000 C CNN
-F 1 "R" V 6207 3901 40  0000 C CNN
-F 2 "RP_KiCAD_Libs:0204_2f5" V 6130 3900 30  0001 C CNN
-F 3 "" H 6200 3900 30  0000 C CNN
-	1    6200 3900
-	1    0    0    -1
-$EndComp
-Wire Wire Line
-	6450 4450 6200 4450
-Wire Wire Line
-	6450 3950 6450 4450
-Wire Wire Line
-	6450 4050 6800 4050
-Connection ~ 6450 4050
-Wire Wire Line
-	6200 3750 7000 3750
-Wire Wire Line
-	7000 3750 7000 4750
-Wire Wire Line
-	7000 4750 6800 4750
-Wire Wire Line
-	6100 4050 6200 4050
-$Comp
-L GND #PWR05
-U 1 1 57A31457
-P 6800 4800
-F 0 "#PWR05" H 6800 4800 30  0001 C CNN
-F 1 "GND" H 6800 4730 30  0001 C CNN
-F 2 "" H 6800 4800 60  0000 C CNN
-F 3 "" H 6800 4800 60  0000 C CNN
-	1    6800 4800
-	1    0    0    -1
-$EndComp
-$Comp
-L +5V #PWR06
-U 1 1 57A3145D
-P 6450 3950
-F 0 "#PWR06" H 6450 4040 20  0001 C CNN
-F 1 "+5V" H 6450 4040 30  0000 C CNN
-F 2 "" H 6450 3950 60  0000 C CNN
-F 3 "" H 6450 3950 60  0000 C CNN
-	1    6450 3950
-	1    0    0    -1
-$EndComp
-Wire Wire Line
-	6800 4750 6800 4800
-Text Label 6100 4050 2    60   ~ 0
-OUT
-Connection ~ 6200 4050
-Connection ~ 6800 4750
-$Comp
-L CONN_01X03 P2
-U 1 1 57A31467
-P 5250 4000
-F 0 "P2" H 5250 4200 50  0000 C CNN
-F 1 "CONN_01X03" V 5350 4000 50  0000 C CNN
-F 2 "Crystals:Resonator_7.2x3mm" H 5250 4000 50  0001 C CNN
-F 3 "" H 5250 4000 50  0000 C CNN
-	1    5250 4000
-	-1   0    0    1
-$EndComp
-Text Label 5450 3900 0    60   ~ 0
-OUT
-$Comp
-L +5V #PWR07
-U 1 1 57A3146E
-P 5450 4000
-F 0 "#PWR07" H 5450 4090 20  0001 C CNN
-F 1 "+5V" H 5450 4090 30  0000 C CNN
-F 2 "" H 5450 4000 60  0000 C CNN
-F 3 "" H 5450 4000 60  0000 C CNN
-	1    5450 4000
-	0    1    1    0
-$EndComp
-$Comp
-L GND #PWR08
-U 1 1 57A31474
-P 5450 4100
-F 0 "#PWR08" H 5450 4100 30  0001 C CNN
-F 1 "GND" H 5450 4030 30  0001 C CNN
-F 2 "" H 5450 4100 60  0000 C CNN
-F 3 "" H 5450 4100 60  0000 C CNN
-	1    5450 4100
-	0    -1   -1   0
-$EndComp
