File: KiCAD_Projects/3WS_MD_rev3.0/3WS_MD_rev3.0.kicad_pcb (KiCad board)
At the start: 2 copper layers, 76 x 93 mm, 140 parts, among them P1 CONN_01X01, P11 TST, P12 TST, P13 CONN_01X06, P14 CONN_01X02, P15 CONN_01X02, P16 CONN_01X04, P17 CONN_01X04, P18 CONN_01X04, P19 CONN_01X04, P2 CONN_01X01, P20 CONN_01X06, P3 CONN_01X04, P4 CONN_02X02, P5 TST, P6 CONN_01X04, P7 CONN_01X02, P8 CONN_01X04, P9 TST, Q1 MOSFET_N, Q2 MOSFET_N, Q3 MOSFET_N, Q4 MOSFET_N, Q5 MOSFET_N, Q6 MOSFET_N, Q7 MOSFET_N, Q8 MOSFET_N, Q9 MOSFET_N, SW1 SW_PUSH, SW2 SW_PUSH, SW3 SW_PUSH, U1 STM32F103_48, U10 NCP1117ST33T3G, U2 SI8234, U3 SI8234, U4 LM7812, U5 SI8234, U6 SI8234, U7 NCP1117ST33T3G, U8 MAX3051, U9 SW_ROTARY_16, X2 CRYSTAL

Commit message: no message
Parts:
- G***: footprint RP_KiCAD_Libs:Raiden -> RP_KiCAD_Libs:hien_2
- G***: footprint RP_KiCAD_Libs:Raiden_text -> RP_KiCAD_Libs:hien_2_text
- moved G*** 18.4 mm to (13.5, 61.9)
- moved G*** 2.20 mm to (10.1, 74.0), turned to 270 degrees
