File: KiCAD_Projects/DEF_encoder/_saved_DEF_encoder.sch (KiCad schematic (older format))
At the start: 7 parts, among them P1 CONN_01X04, P2 CONN_01X04, U1 SN75175

Commit message: no message
Parts:
- added R2, R3, R4, R5: 120, RP_KiCAD_Libs:C1608_WP, symbol R
Changed lines of the file:
@@
 Text Label 5350 2100 2    60   ~ 0
 OUT1_A
+$Comp
+L R R2
+U 1 1 583F8365
+P 2750 1600
+F 0 "R2" V 2830 1600 40  0000 C CNN
+F 1 "120" V 2757 1601 40  0000 C CNN
+F 2 "RP_KiCAD_Libs:C1608_WP" V 2680 1600 30  0001 C CNN
+F 3 "" H 2750 1600 30  0000 C CNN
+	1    2750 1600
+	1    0    0    -1
+$EndComp
+$Comp
+L R R3
+U 1 1 583F83AD
+P 2750 2100
+F 0 "R3" V 2830 2100 40  0000 C CNN
+F 1 "120" V 2757 2101 40  0000 C CNN
+F 2 "RP_KiCAD_Libs:C1608_WP" V 2680 2100 30  0001 C CNN
+F 3 "" H 2750 2100 30  0000 C CNN
+	1    2750 2100
+	1    0    0    -1
+$EndComp
+$Comp
+L R R4
+U 1 1 583F8433
+P 3350 1600
+F 0 "R4" V 3430 1600 40  0000 C CNN
+F 1 "120" V 3357 1601 40  0000 C CNN
+F 2 "RP_KiCAD_Libs:C1608_WP" V 3280 1600 30  0001 C CNN
+F 3 "" H 3350 1600 30  0000 C CNN
+	1    3350 1600
+	1    0    0    -1
+$EndComp
+$Comp
+L R R5
+U 1 1 583F8439
+P 3350 2100
+F 0 "R5" V 3430 2100 40  0000 C CNN
+F 1 "120" V 3357 2101 40  0000 C CNN
+F 2 "RP_KiCAD_Libs:C1608_WP" V 3280 2100 30  0001 C CNN
+F 3 "" H 3350 2100 30  0000 C CNN
+	1    3350 2100
+	1    0    0    -1
+$EndComp
+Text Label 2750 1750 0    60   ~ 0
+IN1_AA
+Text Label 2750 1450 0    60   ~ 0
+IN1_AB
+Text Label 2750 1950 0    60   ~ 0
+IN1_BB
+Text Label 2750 2250 0    60   ~ 0
+IN1_BA
+Text Label 3350 1450 0    60   ~ 0
+IN2_AB
+Text Label 3350 1750 0    60   ~ 0
+IN2_AA
+Text Label 3350 1950 0    60   ~ 0
+IN2_BB
+Text Label 3350 2250 0    60   ~ 0
+IN2_BA
 $EndSCHEMATC
