File: KiCAD_Projects/ACS758_test/ACS758_test.sch (KiCad schematic (older format))
At the start: 6 parts, among them P1 CONN_01X03, P2 CONN_01X01, P3 CONN_01X01, P4 CONN_01X01, P5 CONN_01X01, U1 ACS758

Commit message: no message
Parts:
- added C1: C, RP_KiCAD_Libs:C2012, symbol C
Connections:
- net at P1.2 (P2), U1.1 (VCC): now also C1.2
- net at P1.1 (P1), U1.2 (GND): now also C1.1
Changed lines of the file:
@@
 Wire Wire Line
 	5300 3250 5750 3250
+$Comp
+L C C1
+U 1 1 5841AF29
+P 5550 2750
+F 0 "C1" H 5550 2850 40  0000 L CNN
+F 1 "C" H 5556 2665 40  0000 L CNN
+F 2 "RP_KiCAD_Libs:C2012" H 5588 2600 30  0001 C CNN
+F 3 "" H 5550 2750 60  0000 C CNN
+	1    5550 2750
+	1    0    0    -1
+$EndComp
+Connection ~ 5550 2950
+Wire Wire Line
+	5550 2550 5700 2550
+Wire Wire Line
+	5700 2550 5700 3100
+Connection ~ 5700 3100
 $EndSCHEMATC
