File: KiCAD_Projects/3WS_MD_rev4.0/3WS_MD_rev4.0.kicad_pcb (KiCad board)
At the start: 2 copper layers, 76 x 93 mm, 140 parts, among them P1 CONN_01X01, P11 TST, P12 TST, P13 CONN_01X06, P14 CONN_01X02, P15 CONN_01X02, P16 CONN_01X04, P17 CONN_01X04, P18 CONN_01X04, P19 CONN_01X04, P2 CONN_01X01, P20 CONN_01X06, P3 CONN_01X04, P4 CONN_02X02, P5 TST, P6 CONN_01X04, P7 CONN_01X02, P8 CONN_01X04, P9 TST, Q1 MOSFET_N, Q2 MOSFET_N, Q3 MOSFET_N, Q4 MOSFET_N, Q5 MOSFET_N, Q6 MOSFET_N, Q7 MOSFET_N, Q8 MOSFET_N, Q9 MOSFET_N, SW1 SW_PUSH, SW2 SW_PUSH, SW3 SW_PUSH, U1 STM32F103_48, U10 NCP1117ST33T3G, U2 SI8234, U3 SI8234, U4 LM7812, U5 SI8234, U6 SI8234, U7 NCP1117ST33T3G, U8 MAX3051, U9 SW_ROTARY_16, X2 CRYSTAL

Commit message: no message
Parts:
- removed G***: LOGO, RP_KiCAD_Libs:hien_2
- removed G***: LOGO, RP_KiCAD_Libs:hien_2_text
- added R40: 10, RP_KiCAD_Libs:C3216, F.Cu at (38.0, 103.1)
- C21: value 470u -> 100u; footprint Capacitors_ThroughHole:C_Radial_D12.5_L25_P5 -> Capacitors_ThroughHole:C_Radial_D6.3_L11.2_P2.5
- Q1, Q2, Q3, Q4, Q5, Q6, Q7, Q8: footprint TO_SOT_Packages_SMD:D2-PAK -> TO_SOT_Packages_SMD:D2-PAK_compact
- moved C22 13.0 mm to (10.0, 25.0)
- moved C21 10.8 mm to (13.5, 35.0)
- moved Q1 6.52 mm to (38.0, 38.5)
- moved Q5 6.52 mm to (64.0, 38.5)
- moved Q3 6.50 mm to (24.5, 38.5)
- moved Q7 6.50 mm to (50.5, 38.5)
- moved Q6 5.02 mm to (64.0, 21.0)
- moved Q2 5.00 mm to (37.5, 21.0)
- moved Q4 5.00 mm to (24.5, 21.0)
- moved Q8 5.00 mm to (50.5, 21.0)
- moved U4 4.61 mm to (13.0, 45.5), turned to 180 degrees
- moved C25 3.04 mm to (17.0, 48.5)
Connections:
- C21 pad 1: +BATT -> Net-(C21-Pad1)
- C27 pad 1: Net-(C27-Pad1) -> Net-(C21-Pad1)
- D15 pad 1: +BATT -> Net-(D15-Pad1)
- D15 pad 2: Net-(C27-Pad1) -> Net-(C21-Pad1)
- U4 pad VI: Net-(C27-Pad1) -> Net-(C21-Pad1)
Routing:
- net GNDPWR: track 316.7 -> 1.00 mm, vias 58 -> 0
- net /OUT_A: track 145.5 -> 0.00 mm, vias 62 -> 0
- net +BATT: track 141.6 -> 0.00 mm, vias 50 -> 0
- net /OUT_AN: track 139.1 -> 0.00 mm, vias 62 -> 0
- net /OUT_B: track 106.3 -> 0.00 mm, vias 41 -> 0
- net /GD_12V: track 86.4 -> 0.00 mm, vias 9 -> 0
- net /OUT_BN: track 84.8 -> 0.00 mm, vias 41 -> 0
- net GND: track 378.3 -> 312.8 mm
- net +3.3V: track 287.8 -> 226.5 mm
- net Net-(R9-Pad2): track 34.8 -> 0.00 mm, vias 2 -> 0
- net Net-(R7-Pad2): track 34.8 -> 0.00 mm, vias 2 -> 0
- net Net-(R15-Pad2): track 34.8 -> 0.00 mm, vias 2 -> 0
- net Net-(R13-Pad2): track 34.8 -> 0.00 mm, vias 2 -> 0
- net /EXIO_3: track 63.1 -> 49.7 mm
- net /EXIO_2: track 61.1 -> 50.2 mm
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
Commit message: no message
Parts:
- moved Q9 7.00 mm to (50.4, 59.9)
- moved R32 7.00 mm to (55.3, 59.9)
- moved R33 7.00 mm to (53.8, 59.9)
- moved C1 7.00 mm to (4.80, 70.9)
- moved C13 7.00 mm to (59.7, 68.3)
- moved C14 7.00 mm to (66.0, 52.0)
- moved C15 7.00 mm to (53.0, 52.0)
- moved C2 7.00 mm to (40.0, 52.0)
- moved C20 7.00 mm to (63.1, 58.0)
- moved C23 7.00 mm to (59.0, 76.5)
- moved C26 7.00 mm to (53.8, 68.8)
- moved C29 7.00 mm to (30.3, 64.5)
- moved C3 7.00 mm to (27.0, 52.0)
- moved C4 7.00 mm to (13.7, 70.2)
- moved C5 7.00 mm to (16.1, 72.6)
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
Commit message: no message
Parts:
- moved R40 62.9 mm to (10.5, 39.5)
- moved P12 13.0 mm to (83.5, 39.5)
- moved D15 11.0 mm to (9.50, 34.5)
- moved D12 9.85 mm to (14.5, 41.0)
- moved R20 5.52 mm to (13.0, 40.5)
- moved C27 5.50 mm to (14.5, 38.0)
- moved C25 4.03 mm to (15.0, 43.0)
- moved U4 3.35 mm to (11.5, 40.5)
- moved Q4 3.04 mm to (27.5, 19.5)
- moved Q3 3.00 mm to (27.5, 36.5)
- moved C21 2.92 mm to (16.0, 34.5), turned to 90 degrees
- moved FB4 2.06 mm to (32.0, 18.5)
- moved Q2 2.06 mm to (39.5, 19.5)
- moved R9 2.00 mm to (33.5, 22.5)
- moved FB2 1.58 mm to (44.5, 19.5)
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Routing:
- removed copper zone on B.Cu, net +BATT
- removed copper zone on B.Cu, net /OUT_A
- removed copper zone on B.Cu, net /OUT_AN
- removed copper zone on B.Cu, net /OUT_B
- removed copper zone on B.Cu, net /OUT_BN

Commit message: no message
Parts:
- added U1: ACS758, RP_KiCAD_Libs:ACS785xCB, F.Cu at (113.0, 7.50)
- FB4, R9: moved to B.Cu
- moved Q2 59.7 mm to (93.4, 45.2), turned to 0 degrees
- moved Q1 56.0 mm to (95.2, 30.9), turned to 0 degrees
- moved FB4 28.2 mm to (21.0, 44.5), turned to 45 degrees
- moved R9 28.0 mm to (21.0, 47.5), turned to 315 degrees
- moved Q4 23.5 mm to (27.5, 43.0), turned to 0 degrees
- moved P2 11.2 mm to (-7.50, 14.0)
- moved P1 11.1 mm to (-7.50, 12.5)
- moved Q3 10.5 mm to (27.5, 26.0), turned to 0 degrees
- moved U2 7.00 mm to (37.5, 55.0)
- moved U3 7.00 mm to (24.5, 55.0)
- moved U5 7.00 mm to (63.5, 55.0)
- moved U6 7.00 mm to (50.5, 55.0)
- moved Q9 6.00 mm to (50.4, 66.9)
- moved R32 6.00 mm to (55.3, 66.9)
- moved R33 6.00 mm to (53.8, 66.9)
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Routing:
- net Net-(FB4-Pad2): track 0.00 -> 4.66 mm, vias 0 -> 1
- net Net-(R9-Pad2): track 0.00 -> 4.29 mm
- net Net-(FB4-Pad1): track 0.00 -> 1.73 mm
- net GNDPWR: track 1.00 -> 0.00 mm
- removed copper zone on F.Cu, net +BATT
- removed copper zone on B.Cu, net GND
- removed copper zone on B.Cu, net GNDPWR
