File: KiCAD_Projects/STM32F103_CanNode_rev1.1/STM32F103_CanNode_rev1.1.sch (KiCad schematic (older format))
At the start: 69 parts, among them P1 CONN_01X04, P10 CONN_01X04, P11 CONN_01X04, P2 CONN_01X04, P3 CONN_01X08, P4 CONN_01X08, P5 CONN_01X06, P6 CONN_01X02, P7 CONN_01X08, P8 CONN_01X04, P9 CONN_01X04, SW1 SW_PUSH, U1 STM32F103_48, U2 NCP1117ST33T3G, U3 MAX3051, U4 NCP1117ST50T3G, U5 TBD62083A, X2 CRYSTAL

Commit message: no message
Parts:
- removed C6: C, RP_KiCAD_Libs:C1608_WP, symbol C
- added D11: DIODE, Diodes_SMD:SMA_Standard, symbol DIODE
- added JP12, JP13: JUMPER3, Connect:GS3, symbol JUMPER3
- C1, C8, C9: value C -> 0.1u
- C2, C3, C7: value C -> 4.7u
- C4, C5: value C -> 22p
- R1, R2: value R -> 10k
- R5: value R -> 120
Connections:
- net +12V: now also D11.1 (K); no longer P1.2 (P2), P2.2 (P2)
- net +3.3V: now also JP12.3, JP13.3; no longer JP11.3, JP9.3
- net +5V: now also JP12.1, JP13.1
- net PA4: now also JP2.2; no longer JP6.2
- net PA5: now also JP4.2; no longer JP8.2
- net PB0: now also JP6.2; no longer JP2.2
- net PB1: now also JP8.2; no longer JP4.2
- new net: D11.2 (A), P1.2 (P2), P2.2 (P2)
- new net: JP13.2, JP9.3
- new net: JP11.3, JP12.2
Other:
- moved on the sheet: P1, P2
