File: KiCAD_Projects/SingleCanEncoder_compact/SingleCanEncoder_compact.sch (KiCad schematic (older format))
At the start: 34 parts, among them P1 CONN_01X04, P2 CONN_01X04, P3 CONN_01X04, P5 CONN_01X06, P6 CONN_01X02, SW1 SW_PUSH, U1 STM32F103_48, U2 NCP1117ST33T3G, U3 MAX3051, U4 LM7805CT, U5 SW_ROTARY_16, X2 CRYSTAL

Commit message: 単発エンコーダ基板のアドレスセレクタ変更
Parts:
- removed U4: LM7805CT, TO_SOT_Packages_SMD:SOT89-3_Housing, symbol LM7805CT
- added U4: SOT-89-3regul, TO_SOT_Packages_SMD:SOT89-3_Housing, symbol SOT-89-3regul
- U5: footprint Buttons_Switches_SMD:SW_ROTARY_16 -> Buttons_Switches_ThroughHole:rotary_0F
Changed lines of the file:
@@
 F 0 "U5" H 9350 4550 60  0000 C CNN
 F 1 "SW_ROTARY_16" H 9350 3950 60  0000 C CNN
-F 2 "Buttons_Switches_SMD:SW_ROTARY_16" H 9350 4250 60  0001 C CNN
+F 2 "Buttons_Switches_ThroughHole:rotary_0F" H 9350 4250 60  0001 C CNN
 F 3 "" H 9350 4250 60  0001 C CNN
 	1    9350 4250
 	1    0    0    -1
 $EndComp
+Text Label 8900 4100 2    60   ~ 0
+SEL_1
 Text Label 8900 4400 2    60   ~ 0
-SEL_1
-Text Label 8900 4100 2    60   ~ 0
 SEL_2
 Text Label 9800 4100 0    60   ~ 0
@@
 	0    1    1    0
 $EndComp
-Text Label 4000 3250 2    60   ~ 0
+Text Label 4000 4050 2    60   ~ 0
 SEL_1
-Text Label 4000 3350 2    60   ~ 0
+Text Label 4000 4150 2    60   ~ 0
 SEL_2
+Text Label 5100 5350 3    60   ~ 0
+SEL_8
 Text Label 4000 4250 2    60   ~ 0
-SEL_8
-Text Label 4000 3450 2    60   ~ 0
 SEL_4
 Text Label 12850 4350 2    60   ~ 0
@@
 $EndComp
 $Comp
-L LM7805CT U4
-U 1 1 587C1A85
-P 2500 7050
-F 0 "U4" H 2300 7250 40  0000 C CNN
-F 1 "LM7805CT" H 2500 7250 40  0000 L CNN
-F 2 "TO_SOT_Packages_SMD:SOT89-3_Housing" H 2500 7150 30  0000 C CIN
-F 3 "" H 2500 7050 60  0000 C CNN
-	1    2500 7050
+L SOT-89-3regul U4
+U 1 1 5881E916
+P 2500 7150
+F 0 "U4" H 2300 7350 40  0000 C CNN
+F 1 "SOT-89-3regul" H 2350 7350 40  0000 L CNN
+F 2 "TO_SOT_Packages_SMD:SOT89-3_Housing" H 2500 7250 30  0000 C CIN
+F 3 "" H 2500 7150 60  0000 C CNN
+	1    2500 7150
 	1    0    0    -1
 $EndComp

Commit message: rev4.0設計開始
Parts:
- removed JP1: JUMPER3, Connect:GS3, symbol JUMPER3
- added C9: 0.1u, RP_KiCAD_Libs:C1608_WP, symbol C
- added D3: DIODE, RP_KiCAD_Libs:C1608_WP, symbol DIODE
- added D4: LED, RP_KiCAD_Libs:C1608_WP, symbol LED
- added P4: CONN_01X03, RP_KiCAD_Connector:XA_3LC, symbol CONN_01X03
- added P7: CONN_01X02, Pin_Headers:Pin_Header_Straight_1x02, symbol CONN_01X02
- added PC1: TLP117, RP_KiCAD_Libs:SOIC-5_3.9x4.9mm_Pitch1.27mm, symbol TLP117
- added Q1, Q2: MOSFET_N, TO_SOT_Packages_SMD:SOT-23_Handsoldering, symbol MOSFET_N
- added R8, R9: 1k, RP_KiCAD_Libs:C1608_WP, symbol R
- D1, D2: footprint LEDs:LED_0805 -> RP_KiCAD_Libs:C1608_WP
Connections:
- net labels added: PWM_A, PWM_B, VALVE
- wire segments 19 -> 39
Other:
- moved on the sheet: C6
