File: KiCAD_Projects/Amp_ISO/Amp_ISO.sch (KiCad schematic (older format))
At the start: 0 parts

Commit message: MDver4.0だいたいできた｡絶縁アンプ基板作った｡
Parts:
- added C1, C2: 0.1u, RP_KiCAD_Libs:C1608_WP, symbol C
- added D1, D2: LED, RP_KiCAD_Libs:C1608_WP, symbol LED
- added P1, P3, P4: CONN_01X01, Connect:PINTST, symbol CONN_01X01
- added P2: CONN_01X03, RP_KiCAD_Connector:XA_3LC, symbol CONN_01X03
- added PC1: TLP117, RP_KiCAD_Libs:SOIC-5_3.9x4.9mm_Pitch1.27mm, symbol TLP117
- added Q1: MOSFET_N, TO_SOT_Packages_SMD:SOT-23_Handsoldering, symbol MOSFET_N
- added R1, R2, R3, R4: R, RP_KiCAD_Libs:C1608_WP, symbol R
Connections:
- new net: PC1.3 (K), R4.1
- new net: Q1.D, R4.2
- new net: D1.2 (K), R2.1
- new net: D2.2 (K), R3.1
- new net 5V_LOGIC: C1.1, D1.1 (A), P3.1 (P1), PC1.1 (A)
- new net 5V_POWER: C2.1, D2.1 (A), P2.2 (P2), PC1.6 (VCC)
- new net GND_LOGIC: C1.2, P4.1 (P1), Q1.S, R1.2, R2.2
- new net GND_POWER: C2.2, P2.3 (P3), PC1.4 (GND), R3.2
- new net SIGNAL_LOGIC: P1.1 (P1), Q1.G, R1.1
- new net SIGNAL_POWER: P2.1 (P1), PC1.5 (VO)
Changed lines of the file:
@@
 LIBS:conn
 LIBS:device
+LIBS:opto
+LIBS:regul
+LIBS:stm32
+LIBS:user
 LIBS:power
-LIBS:regul
-LIBS:user
+LIBS:Amp_ISO-cache
 EELAYER 25 0
 EELAYER END
@@
 Comment4 ""
 $EndDescr
+$Comp
+L TLP117 PC1
+U 1 1 589990AC
+P 5900 2700
+F 0 "PC1" H 5900 2450 60  0000 C CNN
+F 1 "TLP117" H 5900 2950 60  0000 C CNN
+F 2 "RP_KiCAD_Libs:SOIC-5_3.9x4.9mm_Pitch1.27mm" H 5900 2700 60  0001 C CNN
+F 3 "" H 5900 2700 60  0001 C CNN
+	1    5900 2700
+	1    0    0    -1
+$EndComp
+$Comp
+L MOSFET_N Q1
+U 1 1 589990E9
+P 4900 3050
+F 0 "Q1" H 4910 3220 60  0000 R CNN
+F 1 "MOSFET_N" H 4910 2900 60  0000 R CNN
+F 2 "TO_SOT_Packages_SMD:SOT-23_Handsoldering" H 4900 3050 60  0001 C CNN
+F 3 "" H 4900 3050 60  0000 C CNN
+	1    4900 3050
+	1    0    0    -1
+$EndComp
+$Comp
+L R R4
+U 1 1 58999140
+P 5250 2850
+F 0 "R4" V 5330 2850 40  0000 C CNN
+F 1 "R" V 5257 2851 40  0000 C CNN
+F 2 "RP_KiCAD_Libs:C1608_WP" V 5180 2850 30  0001 C CNN
+F 3 "" H 5250 2850 30  0000 C CNN
+	1    5250 2850
+	0    1    1    0
+$EndComp
+Wire Wire Line
+	5000 2850 5100 2850
+Wire Wire Line
+	5400 2850 5500 2850
+Wire Wire Line
+	5500 2550 4450 2550
+Wire Wire Line
+	5000 3250 5000 3450
+Wire Wire Line
+	5000 3450 4100 3450
+Wire Wire Line
+	4700 3050 4450 3050
+Wire Wire Line
+	4450 2750 4450 3100
+Wire Wire Line
+	4450 2750 4050 2750
+$Comp
+L R R1
+U 1 1 589991EB
+P 4450 3250
+F 0 "R1" V 4530 3250 40  0000 C CNN
+F 1 "R" V 4457 3251 40  0000 C CNN
+F 2 "RP_KiCAD_Libs:C1608_WP" V 4380 3250 30  0001 C CNN
+F 3 "" H 4450 3250 30  0000 C CNN
+	1    4450 3250
+	1    0    0    -1
+$EndComp
+Connection ~ 4450 3050
+Wire Wire Line
+	4450 3400 4450 3450
+Connection ~ 4450 3450
+Text Label 2800 2800 0    60   ~ 0
+SIGNAL_LOGIC
+Text Label 2800 3200 0    60   ~ 0
+GND_LOGIC
+Text Label 2800 3000 0    60   ~ 0
+5V_LOGIC
+Text Label 4050 2750 2    60   ~ 0
+SIGNAL_LOGIC
+Text Label 4450 2550 2    60   ~ 0
+5V_LOGIC
+Text Label 4100 3450 2    60   ~ 0
+GND_LOGIC
+Text Label 3850 1750 2    60   ~ 0
+5V_LOGIC
+Text Label 3850 2150 2    60   ~ 0
+GND_LOGIC
+$Comp
+L C C1
+U 1 1 589995EE
+P 3850 1950
+F 0 "C1" H 3850 2050 40  0000 L CNN
+F 1 "0.1u" H 3856 1865 40  0000 L CNN
+F 2 "RP_KiCAD_Libs:C1608_WP" H 3888 1800 30  0001 C CNN
+F 3 "" H 3850 1950 60  0000 C CNN
+	1    3850 1950
+	1    0    0    -1
+$EndComp
+$Comp
+L LED D1
+U 1 1 589996D6
+P 4600 1400
+F 0 "D1" H 4600 1500 50  0000 C CNN
+F 1 "LED" H 4600 1300 50  0000 C CNN
+F 2 "RP_KiCAD_Libs:C1608_WP" H 4600 1400 60  0001 C CNN
+F 3 "" H 4600 1400 60  0000 C CNN
+	1    4600 1400
+	0    1    1    0
+$EndComp
+$Comp
+L R R2
+U 1 1 5899970B
+P 4600 1850
+F 0 "R2" V 4680 1850 40  0000 C CNN
+F 1 "R" V 4607 1851 40  0000 C CNN
+F 2 "RP_KiCAD_Libs:C1608_WP" V 4530 1850 30  0001 C CNN
+F 3 "" H 4600 1850 30  0000 C CNN
+	1    4600 1850
+	1    0    0    -1
+$EndComp
+$Comp
+L LED D2
+U 1 1 589997C0
+P 5000 1400
+F 0 "D2" H 5000 1500 50  0000 C CNN
+F 1 "LED" H 5000 1300 50  0000 C CNN
+F 2 "RP_KiCAD_Libs:C1608_WP" H 5000 1400 60  0001 C CNN
+F 3 "" H 5000 1400 60  0000 C CNN
+	1    5000 1400
+	0    1    1    0
+$EndComp
+$Comp
+L R R3
+U 1 1 589997C6
+P 5000 1850
+F 0 "R3" V 5080 1850 40  0000 C CNN
+F 1 "R" V 5007 1851 40  0000 C CNN
+F 2 "RP_KiCAD_Libs:C1608_WP" V 4930 1850 30  0001 C CNN
+F 3 "" H 5000 1850 30  0000 C CNN
+	1    5000 1850
+	1    0    0    -1
+$EndComp
+Wire Wire Line
+	4600 1600 4600 1700
+Wire Wire Line
+	5000 1600 5000 1700
+Text Label 4600 2000 2    60   ~ 0
+GND_LOGIC
+Text Label 4600 1200 2    60   ~ 0
+5V_LOGIC
+Text Label 6300 2850 0    60   ~ 0
+GND_POWER
+Text Label 6300 2550 0    60   ~ 0
+5V_POWER
+Text Label 6300 2700 0    60   ~ 0
+SIGNAL_POWER
+Text Label 5000 1200 0    60   ~ 0
+5V_POWER
+Text Label 5000 2000 0    60   ~ 0
+GND_POWER
+Text Label 5900 1350 0    60   ~ 0
+5V_POWER
+Text Label 5900 1750 0    60   ~ 0
+GND_POWER
+$Comp
+L C C2
+U 1 1 58999C02
+P 5900 1550
+F 0 "C2" H 5900 1650 40  0000 L CNN
+F 1 "0.1u" H 5906 1465 40  0000 L CNN
+F 2 "RP_KiCAD_Libs:C1608_WP" H 5938 1400 30  0001 C CNN
+F 3 "" H 5900 1550 60  0000 C CNN
+	1    5900 1550
+	1    0    0    -1
+$EndComp
+$Comp
+L CONN_01X03 P2
+U 1 1 58999E0F
+P 8000 2650
+F 0 "P2" H 8000 2850 50  0000 C CNN
+F 1 "CONN_01X03" V 8100 2650 50  0000 C CNN
+F 2 "RP_KiCAD_Connector:XA_3LC" H 8000 2650 50  0001 C CNN
+F 3 "" H 8000 2650 50  0000 C CNN
+	1    8000 2650
+	1    0    0    -1
+$EndComp
+Text Label 7800 2650 2    60   ~ 0
+5V_POWER
+Text Label 7800 2550 2    60   ~ 0
+SIGNAL_POWER
+Text Label 7800 2750 2    60   ~ 0
+GND_POWER
+$Comp
+L CONN_01X01 P1
+U 1 1 5899A2DA
+P 2600 2800
+F 0 "P1" H 2600 2900 50  0000 C CNN
+F 1 "CONN_01X01" V 2700 2800 50  0000 C CNN
+F 2 "Connect:PINTST" H 2600 2800 50  0001 C CNN
+F 3 "" H 2600 2800 50  0000 C CNN
+	1    2600 2800
+	-1   0    0    1
+$EndComp
+$Comp
+L CONN_01X01 P3
+U 1 1 5899A405
+P 2600 3000
+F 0 "P3" H 2600 3100 50  0000 C CNN
+F 1 "CONN_01X01" V 2700 3000 50  0000 C CNN
+F 2 "Connect:PINTST" H 2600 3000 50  0001 C CNN
+F 3 "" H 2600 3000 50  0000 C CNN
+	1    2600 3000
+	-1   0    0    1
+$EndComp
+$Comp
+L CONN_01X01 P4
+U 1 1 5899A444
+P 2600 3200
+F 0 "P4" H 2600 3300 50  0000 C CNN
+F 1 "CONN_01X01" V 2700 3200 50  0000 C CNN
+F 2 "Connect:PINTST" H 2600 3200 50  0001 C CNN
+F 3 "" H 2600 3200 50  0000 C CNN
+	1    2600 3200
+	-1   0    0    1
+$EndComp
 $EndSCHEMATC

Commit message: 4.0発注かけた｡テレメトリとコンパネ作る
Parts:
- P1, P3, P4: footprint Connect:PINTST -> Measurement_Points:Measurement_Point_Square-SMD-Pad_Small
Connections:
- net GND_POWER: now also P2.1 (P1); no longer P2.3 (P3)
- net SIGNAL_POWER: now also P2.3 (P3); no longer P2.1 (P1)
Changed lines of the file:
@@
 F 3 "" H 8000 2650 50  0000 C CNN
 	1    8000 2650
-	1    0    0    -1
+	1    0    0    1
 $EndComp
 Text Label 7800 2650 2    60   ~ 0
@@
 F 0 "P1" H 2600 2900 50  0000 C CNN
 F 1 "CONN_01X01" V 2700 2800 50  0000 C CNN
-F 2 "Connect:PINTST" H 2600 2800 50  0001 C CNN
+F 2 "Measurement_Points:Measurement_Point_Square-SMD-Pad_Small" H 2600 2800 50  0001 C CNN
 F 3 "" H 2600 2800 50  0000 C CNN
 	1    2600 2800
@@
 F 0 "P3" H 2600 3100 50  0000 C CNN
 F 1 "CONN_01X01" V 2700 3000 50  0000 C CNN
-F 2 "Connect:PINTST" H 2600 3000 50  0001 C CNN
+F 2 "Measurement_Points:Measurement_Point_Square-SMD-Pad_Small" H 2600 3000 50  0001 C CNN
 F 3 "" H 2600 3000 50  0000 C CNN
 	1    2600 3000
@@
 F 0 "P4" H 2600 3300 50  0000 C CNN
 F 1 "CONN_01X01" V 2700 3200 50  0000 C CNN
-F 2 "Connect:PINTST" H 2600 3200 50  0001 C CNN
+F 2 "Measurement_Points:Measurement_Point_Square-SMD-Pad_Small" H 2600 3200 50  0001 C CNN
 F 3 "" H 2600 3200 50  0000 C CNN
 	1    2600 3200
