File: KiCAD_Projects/ISO_DCDC_CAN/ISO_DCDC_CAN.sch (KiCad schematic (older format))
At the start: 116 parts, among them IC1 PC817, IC2 PC817, IC3 PC817, IC4 PC817, IC5 PC817, P1 CONN_01X01, P10 CONN_01X02, P11 CONN_01X02, P12 CONN_01X01, P13 CONN_01X04, P14 CONN_01X02, P15 CONN_01X02, P16 TST, P17 CONN_01X06, P19 CONN_01X01, P2 CONN_01X01, P20 CONN_01X01, P21 CONN_01X02, P22 CONN_01X01, P23 CONN_01X01, P25 CONN_01X01, P26 CONN_01X01, P3 CONN_01X01, P4 CONN_01X02, P5 CONN_01X02, P6 CONN_01X04, P7 CONN_01X04, P8 CONN_01X01, P9 CONN_01X01, Q1 MOSFET_N, U1 V23076-D3001-D142, U2 V23076-D3001-D142, U3 V23076-D3001-D142, U4 NCP1117ST285T3G, U5 STM32F103_48, U6 ADM3054, X1 CRYSTAL

Commit message: 4.0発注かけた｡テレメトリとコンパネ作る
Parts:
- C24, C25, C26, C27: renamed from C?; footprint (none) -> RP_KiCAD_Libs:C1608_WP
- R28, R29: renamed from R?; footprint (none) -> RP_KiCAD_Libs:C1608_WP
- U7, U8: renamed from U?; footprint (none) -> RP_KiCAD_Libs:ACS785xCB

Commit message: まともに新電源基板設計始めた
Parts:
- removed C24, C25: 0.1u, RP_KiCAD_Libs:C1608_WP, symbol C
- removed C26, C27: 10n, RP_KiCAD_Libs:C1608_WP, symbol C
- removed JP1, JP2: JUMPER, Pin_Headers:Pin_Header_Straight_1x02, symbol JUMPER
- removed R28: 4.7k, RP_KiCAD_Libs:C1608_WP, symbol R
- removed R5: 2.2k, RP_KiCAD_Libs:C1608_WP, symbol R
- removed U7, U8: ACS758, RP_KiCAD_Libs:ACS785xCB, symbol ACS758
- added D14: LED, LEDs:LED_0603, symbol LED
- added D15: DIODE, Diodes_SMD:POWER_DI5, symbol DIODE
- added P18, P24, P27: CONN_01X01, Connect:1pin, symbol CONN_01X01
- added R30: 2.2k, RP_KiCAD_Libs:C1608_WP, symbol R
- added U7: V23076-D3001-D142, Relays_ThroughHole:V23076-A3001-D142, symbol V23076-D3001-D142
- R29: value 4.7k -> 2.2k
Connections:
- net labels added: CS_A1, CS_A2, CS_B1, CS_B2
- net labels removed: CS_A, CS_B, POWER+_A
- wire segments 146 -> 157
Other:
- note added: "F_GND"
- moved on the sheet: C1, C10, C11, C12, C13, C14, C15, C16, C17, C18, C19, C2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
