File: KiCAD_Projects/3WS_MD_ver4.1/3WS_MD_ver4.1.kicad_pcb (KiCad board)
At the start: 2 copper layers, 76 x 76.2 mm, 175 parts, among them P1 CONN_01X02, P10 CONN_01X04, P11 TST, P12 CONN_02X08, P13 CONN_01X06, P14 CONN_01X02, P15 CONN_01X02, P16 CONN_01X04, P17 CONN_01X04, P2 CONN_01X02, P20 CONN_01X03, P3 CONN_01X04, P4 CONN_02X06, P5 TST, P6 CONN_01X04, P7 CONN_01X02, P8 CONN_01X04, P9 TST, Q1 MOSFET_N, Q2 MOSFET_N, Q3 MOSFET_N, Q4 MOSFET_N, Q5 MOSFET_N, Q6 MOSFET_N, Q7 MOSFET_N, Q8 MOSFET_N, SW1 SW_PUSH, SW2 SW_PUSH, SW3 SW_PUSH, U1 STM32F103_48, U10 NCP1117ST33T3G, U11 TBD62083A, U2 SI8234, U3 SI8234, U4 LM7812, U5 SI8234, U6 SI8234, U7 7805, U8 MAX3051, U9 SW_ROTARY_16, X2 CRYSTAL

Commit message: ver5.0設計中
Parts:
- removed the REF** at (20.5, 16.5)
Routing:
- net /OUT_A: track 15.6 -> 62.4 mm, vias 0 -> 18
- net /OUT_AN: track 13.1 -> 56.2 mm, vias 0 -> 18
Changed lines of the file:
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@@
     (links 379)
     (no_connects 0)
-    (area -0.050001 -1.300001 76.050001 75.050001)
+    (area -2.6192 -9.350001 77.200002 79.175)
     (thickness 1.6)
     (drawings 44)
-    (tracks 1654)
+    (tracks 1738)
     (zones 0)
-    (modules 175)
+    (modules 174)
     (nets 131)
   )
@@
   )
   (setup
-    (last_trace_width 0.5)
+    (last_trace_width 0.25)
     (user_trace_width 0.3)
     (user_trace_width 0.5)
@@
     )
   )
-  (module Diodes_SMD:TUMD2 (layer B.Cu)
-    (at 20.5 16.5)
-    (descr "ROHM - TUMD2")
-    (tags TUMD2)
-    (attr smd)
-    (fp_text reference REF** (at 0 1.85) (layer B.SilkS)
-      (effects (font (size 1 1) (thickness 0.15)) (justify mirror))
-    )
-    (fp_text value TUMD2 (at 0 -2.1) (layer B.Fab)
-      (effects (font (size 1 1) (thickness 0.15)) (justify mirror))
-    )
-    (fp_line (start -2.2 1) (end 1.85 1) (layer B.CrtYd) (width 0.05))
-    (fp_line (start 1.85 1) (end 1.85 -1) (layer B.CrtYd) (width 0.05))
-    (fp_line (start 1.85 -1) (end -2.2 -1) (layer B.CrtYd) (width 0.05))
-    (fp_line (start -2.2 -1) (end -2.2 1) (layer B.CrtYd) (width 0.05))
-    (fp_line (start 1.578 -0.762) (end -1.978 -0.762) (layer B.SilkS) (width 0.15))
-    (fp_line (start -1.978 -0.762) (end -1.978 0.762) (layer B.SilkS) (width 0.15))
-    (fp_line (start -1.978 0.762) (end 1.578 0.762) (layer B.SilkS) (width 0.15))
-    (fp_line (start 1.578 0.762) (end 1.578 -0.762) (layer B.SilkS) (width 0.15))
-    (pad 2 smd rect (at 1.05 0 180) (size 0.8 1.1) (layers B.Cu B.Paste B.Mask))
-    (pad 1 smd rect (at -0.85 0 180) (size 2 1.1) (layers B.Cu B.Paste B.Mask))
-    (model Diodes_SMD.3dshapes/TUMD2.wrl
-      (at (xyz 0 0 0))
-      (scale (xyz 4 4 4))
-      (rotate (xyz 0 0 180))
-    )
-  )
   (gr_text OUT_B (at 64 34.5) (layer F.SilkS)
     (effects (font (size 2 2) (thickness 0.3)))
@@
   (segment (start 26.445 33.3) (end 26.445 31.155) (width 0.5) (layer B.Cu) (net 9))
   (segment (start 26.445 31.155) (end 26.6 31) (width 0.5) (layer B.Cu) (net 9))
+  (segment (start 18.5 16) (end 18 16) (width 0.25) (layer F.Cu) (net 10))
+  (segment (start 18 16) (end 14.5 19.5) (width 0.25) (layer F.Cu) (net 10))
+  (via (at 14.5 19.5) (size 1.5) (drill 0.75) (layers F.Cu B.Cu) (net 10))
+  (segment (start 14.5 19.5) (end 16 19.5) (width 0.25) (layer B.Cu) (net 10))
+  (via (at 16 19.5) (size 1.5) (drill 0.75) (layers F.Cu B.Cu) (net 10))
+  (segment (start 16 19.5) (end 17.5 19.5) (width 0.25) (layer F.Cu) (net 10))
+  (via (at 17.5 19.5) (size 1.5) (drill 0.75) (layers F.Cu B.Cu) (net 10))
+  (segment (start 17.5 19.5) (end 19 19.5) (width 0.25) (layer B.Cu) (net 10))
+  (via (at 19 19.5) (size 1.5) (drill 0.75) (layers F.Cu B.Cu) (net 10))
+  (segment (start 19 19.5) (end 20.5 19.5) (width 0.25) (layer F.Cu) (net 10))
+  (via (at 20.5 19.5) (size 1.5) (drill 0.75) (layers F.Cu B.Cu) (net 10))
+  (segment (start 20.5 19.5) (end 22 19.5) (width 0.25) (layer B.Cu) (net 10))
+  (via (at 22 19.5) (size 1.5) (drill 0.75) (layers F.Cu B.Cu) (net 10))
+  (segment (start 22 19.5) (end 18.5 16) (width 0.25) (layer F.Cu) (net 10))
+  (segment (start 20.5 16.5) (end 22 16.5) (width 0.25) (layer B.Cu) (net 10))
+  (via (at 20.5 16.5) (size 1.5) (drill 0.75) (layers F.Cu B.Cu) (net 10))
+  (segment (start 19 16.5) (end 20.5 16.5) (width 0.25) (layer F.Cu) (net 10))
+  (segment (start 22 16.5) (end 22 18) (width 0.25) (layer F.Cu) (net 10))
+  (segment (start 20.5 18) (end 19 18) (width 0.25) (layer F.Cu) (net 10))
+  (via (at 20.5 18) (size 1.5) (drill 0.75) (layers F.Cu B.Cu) (net 10))
+  (segment (start 22 18) (end 20.5 18) (width 0.25) (layer B.Cu) (net 10))
+  (via (at 22 18) (size 1.5) (drill 0.75) (layers F.Cu B.Cu) (net 10))
+  (via (at 22 16.5) (size 1.5) (drill 0.75) (layers F.Cu B.Cu) (net 10))
+  (via (at 19 18) (size 1.5) (drill 0.75) (layers F.Cu B.Cu) (net 10))
+  (segment (start 19 18) (end 17.5 18) (width 0.25) (layer B.Cu) (net 10))
+  (via (at 17.5 18) (size 1.5) (drill 0.75) (layers F.Cu B.Cu) (net 10))
+  (segment (start 17.5 18) (end 16 18) (width 0.25) (layer F.Cu) (net 10))
+  (via (at 16 18) (size 1.5) (drill 0.75) (layers F.Cu B.Cu) (net 10))
+  (segment (start 16 18) (end 14.5 18) (width 0.25) (layer B.Cu) (net 10))
+  (via (at 14.5 18) (size 1.5) (drill 0.75) (layers F.Cu B.Cu) (net 10))
+  (segment (start 14.5 18) (end 18.5 16) (width 0.25) (layer F.Cu) (net 10))
+  (segment (start 18.5 16) (end 15 16) (width 0.25) (layer F.Cu) (net 10))
+  (segment (start 15 16) (end 14.5 16.5) (width 0.25) (layer F.Cu) (net 10))
+  (via (at 14.5 16.5) (size 1.5) (drill 0.75) (layers F.Cu B.Cu) (net 10))
+  (segment (start 14.5 16.5) (end 16 16.5) (width 0.25) (layer B.Cu) (net 10))
+  (via (at 16 16.5) (size 1.5) (drill 0.75) (layers F.Cu B.Cu) (net 10))
+  (segment (start 16 16.5) (end 17.5 16.5) (width 0.25) (layer F.Cu) (net 10))
+  (via (at 17.5 16.5) (size 1.5) (drill 0.75) (layers F.Cu B.Cu) (net 10))
+  (segment (start 17.5 16.5) (end 19 16.5) (width 0.25) (layer B.Cu) (net 10))
+  (via (at 19 16.5) (size 1.5) (drill 0.75) (layers F.Cu B.Cu) (net 10))
   (segment (start 19.46 21.5) (end 21.7 23.74) (width 0.5) (layer B.Cu) (net 10))
   (segment (start 21.7 23.74) (end 21.7 24) (width 0.5) (layer B.Cu) (net 10))
@@
   (segment (start 20.7 43.8) (end 23.689087 43.8) (width 0.25) (layer F.Cu) (net 26))
   (segment (start 20.25 44.25) (end 20.7 43.8) (width 0.25) (layer F.Cu) (net 26))
+  (segment (start 30.5 16) (end 34 16) (width 0.25) (layer F.Cu) (net 27) (status C00000))
+  (segment (start 34 16) (end 34.5 16.5) (width 0.25) (layer F.Cu) (net 27) (status C00000))
+  (via (at 34.5 16.5) (size 1.5) (drill 0.75) (layers F.Cu B.Cu) (net 27) (status C00000))
+  (segment (start 34.5 16.5) (end 34.5 18) (width 0.25) (layer B.Cu) (net 27) (status 400000))
+  (via (at 34.5 18) (size 1.5) (drill 0.75) (layers F.Cu B.Cu) (net 27) (status 800000))
+  (segment (start 34.5 18) (end 34.5 19.5) (width 0.25) (layer F.Cu) (net 27) (status C00000))
+  (via (at 34.5 19.5) (size 1.5) (drill 0.75) (layers F.Cu B.Cu) (net 27) (status C00000))
+  (segment (start 30.5 16) (end 30.5 17.5) (width 0.25) (layer F.Cu) (net 27) (status C00000))
+  (segment (start 30.5 17.5) (end 30 18) (width 0.25) (layer F.Cu) (net 27) (status C00000))
+  (via (at 30 18) (size 1.5) (drill 0.75) (layers F.Cu B.Cu) (net 27) (status C00000))
+  (segment (start 30 18) (end 30 16.5) (width 0.25) (layer B.Cu) (net 27) (status 400000))
+  (via (at 30 16.5) (size 1.5) (drill 0.75) (layers F.Cu B.Cu) (net 27) (status 800000))
+  (segment (start 30 16.5) (end 30.5 16) (width 0.25) (layer F.Cu) (net 27) (status C00000))
+  (segment (start 33 18) (end 33 19.5) (width 0.25) (layer B.Cu) (net 27) (status 800000))
+  (via (at 33 19.5) (size 1.5) (drill 0.75) (layers F.Cu B.Cu) (net 27) (status C00000))
+  (segment (start 33 19.5) (end 30.5 16) (width 0.25) (layer F.Cu) (net 27) (status C00000))
+  (via (at 30 19.5) (size 1.5) (drill 0.75) (layers F.Cu B.Cu) (net 27) (status C00000))
+  (segment (start 30 19.5) (end 31.5 19.5) (width 0.25) (layer B.Cu) (net 27) (status C00000))
+  (via (at 31.5 19.5) (size 1.5) (drill 0.75) (layers F.Cu B.Cu) (net 27) (status C00000))
+  (segment (start 31.5 19.5) (end 31.5 18) (width 0.25) (layer F.Cu) (net 27) (status C00000))
+  (via (at 31.5 18) (size 1.5) (drill 0.75) (layers F.Cu B.Cu) (net 27) (status C00000))
+  (segment (start 31.5 18) (end 31.5 16.5) (width 0.25) (layer B.Cu) (net 27) (status 400000))
+  (via (at 31.5 16.5) (size 1.5) (drill 0.75) (layers F.Cu B.Cu) (net 27) (status 800000))
+  (segment (start 31.5 16.5) (end 33 16.5) (width 0.25) (layer F.Cu) (net 27) (status C00000))
+  (via (at 33 16.5) (size 1.5) (drill 0.75) (layers F.Cu B.Cu) (net 27) (status C00000))
+  (segment (start 33 16.5) (end 33 18) (width 0.25) (layer B.Cu) (net 27))
+  (via (at 33 18) (size 1.5) (drill 0.75) (layers F.Cu B.Cu) (net 27))
+  (segment (start 33 18) (end 30.5 16) (width 0.25) (layer F.Cu) (net 27) (status 800000))
+  (segment (start 30.5 16) (end 29 16) (width 0.25) (layer F.Cu) (net 27) (status C00000))
+  (segment (start 29 16) (end 28.5 16.5) (width 0.25) (layer F.Cu) (net 27) (status C00000))
+  (via (at 28.5 16.5) (size 1.5) (drill 0.75) (layers F.Cu B.Cu) (net 27) (status C00000))
+  (segment (start 28.5 16.5) (end 28.5 18) (width 0.25) (layer B.Cu) (net 27) (status 400000))
+  (via (at 28.5 18) (size 1.5) (drill 0.75) (layers F.Cu B.Cu) (net 27) (status 800000))
+  (segment (start 28.5 18) (end 30.5 16) (width 0.25) (layer F.Cu) (net 27) (status C00000))
+  (segment (start 30.5 16) (end 27.5 16) (width 0.25) (layer F.Cu) (net 27) (status C00000))
+  (segment (start 27.5 16) (end 27 16.5) (width 0.25) (layer F.Cu) (net 27) (status C00000))
+  (via (at 27 16.5) (size 1.5) (drill 0.75) (layers F.Cu B.Cu) (net 27) (status C00000))
+  (segment (start 27 16.5) (end 27 18) (width 0.25) (layer B.Cu) (net 27) (status 400000))
+  (via (at 27 18) (size 1.5) (drill 0.75) (layers F.Cu B.Cu) (net 27) (status 800000))
+  (segment (start 27 18) (end 27 19.5) (width 0.25) (layer F.Cu) (net 27) (status C00000))
+  (via (at 27 19.5) (size 1.5) (drill 0.75) (layers F.Cu B.Cu) (net 27) (status C00000))
+  (segment (start 27 19.5) (end 28.5 19.5) (width 0.25) (layer B.Cu) (net 27) (status 400000))
+  (via (at 28.5 19.5) (size 1.5) (drill 0.75) (layers F.Cu B.Cu) (net 27) (status 800000))
+  (segment (start 28.5 19.5) (end 30.5 16) (width 0.25) (layer F.Cu) (net 27) (status C00000))
   (segment (start 35.4 31) (end 35 30.6) (width 0.5) (layer B.Cu) (net 27))
   (segment (start 35 30.6) (end 35 23) (width 0.5) (layer B.Cu) (net 27))
