File: KiCAD_Projects/DCDC_converter/DCDC_converter.sch (KiCad schematic (older format))
At the start: 2 parts

Commit message: BLMD設計終わり
Parts:
- added C1, C2: C, RP_KiCAD_Libs:C3216, symbol C
- added C3, C4: 470u, Capacitors_ThroughHole:C_Radial_D18_L36_P7.5, symbol C
- added D1, D2: DIODE, RP_KiCAD_Libs:C3216, symbol DIODE
- added FB1, FB2: FILTER, RP_KiCAD_Libs:C1608_NP, symbol FILTER
- added L1: INDUCTOR, Inductors:SELF-WE-PD-XXL, symbol INDUCTOR
- added Q1, Q2: MOSFET_N, TO_SOT_Packages_THT:TO-247_Horizontal_Neutral123_largePads, symbol MOSFET_N
- added R1, R2, R3, R4: R, RP_KiCAD_Libs:C1608_NP, symbol R
- added R5: 100k, RP_KiCAD_Libs:C1608_NP, symbol R
- added RV1: POT, Discret:RV2, symbol POT
- added U1: SI8234, Housings_SOIC:SOIC-16_3.9x9.9mm_Pitch1.27mm, symbol SI8234
- P1: renamed from P?; footprint (none) -> RP_KiCAD_Connector:DEANS_T
- gave numbers to parts that had none: 1
Connections:
- net EN: now also U1.5 (DISABLE)
- net GND: now also C2.2, C3.2, C4.2, Q2.S, R2.2, R4.2, R5.2, RV1.3, U1.4 (GNDI), U1.9 (GNCB)
- net PWM: now also U1.1 (PWM)
- net VBATT_IN: now also R1.2, R2.1
- net VOUT_IN: now also R3.2, R4.1
- new net: C1.2, L1.1, Q1.S, Q2.D, U1.14 (GNDA)
- new net: FB2.2, Q2.G
- new net: FB2.1, U1.10 (VOB)
- new net: C2.1, D2.1 (K), U1.11 (VDDB)
- new net: FB1.1, U1.15 (VOA)
- new net: C1.1, D1.1 (K), U1.16 (VDDA)
- new net: R5.1, RV1.2, U1.6 (DT)
- new net: FB1.2, Q1.G
- new net +3.3V: U1.3 (VDDI), U1.8 (VDDI)
- new net DCDC_IN: C4.1, L1.2, R1.1
- new net DCDC_OUT: C3.1, Q1.D, R3.1
- new net GD_12V: D1.2 (A), D2.2 (A)
- no-connect marks 0 -> 5
