File: KiCAD_Projects/Valve_to_isorated_AMP/Valve_to_isorated_AMP.kicad_pcb (KiCad board)
At the start: 2 copper layers, 0 parts

Commit message: BLMD設計終わり
Other:
- rule pad_to_mask_clearance: 0 -> 0.2
Changed lines of the file:
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@@
-(kicad_pcb (version 4) (host pcbnew 4.0.5)
+(kicad_pcb (version 4) (host pcbnew 4.0.2-stable)
   (general
     (links 0)
@@
   (setup
     (last_trace_width 0.25)
+    (user_trace_width 0.5)
+    (user_trace_width 1)
     (trace_clearance 0.2)
-    (zone_clearance 0.508)
+    (zone_clearance 0.4)
     (zone_45_only no)
     (trace_min 0.2)
     (segment_width 0.2)
-    (edge_width 0.1)
+    (edge_width 0.15)
     (via_size 0.6)
     (via_drill 0.4)
     (via_min_size 0.4)
     (via_min_drill 0.3)
+    (user_via 1.2 0.8)
     (uvia_size 0.3)
     (uvia_drill 0.1)
@@
     (mod_text_size 1 1)
     (mod_text_width 0.15)
-    (pad_size 1.5 1.5)
-    (pad_drill 0.6)
-    (pad_to_mask_clearance 0)
+    (pad_size 1.524 1.524)
+    (pad_drill 0.762)
+    (pad_to_mask_clearance 0.2)
     (aux_axis_origin 0 0)
-    (visible_elements FFFFFF7F)
+    (visible_elements 7FFFFFFF)
     (pcbplotparams
       (layerselection 0x00030_80000001)
