File: KiCAD_Projects/BLDC_MD/BLDC_MD.kicad_pcb (KiCad board)
At the start: 2 copper layers, 0 parts

Commit message: ver5.0と5.0Exの設計終わり｡CAN node ver1.2の設計終わり｡BLMD基板設計開始｡ISO_DCDCver1.1設計開始｡
Parts:
- added C1: C, RP_KiCAD_Libs:C1608_WP, F.Cu at (58.3, 80.2)
- added C10: 100n, RP_KiCAD_Libs:C1608_WP, F.Cu at (61.3, 61.8)
- added C11: 1u, RP_KiCAD_Libs:C1608_WP, F.Cu at (86.0, 79.0)
- added C12: 1u, RP_KiCAD_Libs:C1608_WP, F.Cu at (102.5, 60.5)
- added C13: 1u, RP_KiCAD_Libs:C1608_WP, F.Cu at (111.9, 49.5)
- added C14: 4.7u, RP_KiCAD_Libs:C3216, F.Cu at (88.1, 60.2)
- added C15: 4.7n, RP_KiCAD_Libs:C3216, F.Cu at (93.6, 59.3)
- added C16: 4.7n, RP_KiCAD_Libs:C3216, F.Cu at (62.4, 56.3)
- added C17: 100u, RP_KiCAD_Libs:C1608_WP, F.Cu at (96.9, 53.9)
- added C18: 4.7u, RP_KiCAD_Libs:C3216, F.Cu at (55.0, 75.0)
- added C2: C, RP_KiCAD_Libs:C1608_WP, F.Cu at (51.5, 80.2)
- added C3: C, RP_KiCAD_Libs:C1608_WP, F.Cu at (54.9, 80.2)
- added C4: C, RP_KiCAD_Libs:C1608_WP, F.Cu at (66.9, 61.8)
- added C5: 4.7u, RP_KiCAD_Libs:C3216, F.Cu at (87.5, 68.7)
- added C6: 4.7u, RP_KiCAD_Libs:C3216, F.Cu at (80.7, 73.5)
- added C7: 4.7u, RP_KiCAD_Libs:C3216, F.Cu at (67.9, 56.3)
- added C8: 4.7u, RP_KiCAD_Libs:C3216, F.Cu at (106.5, 44.0)
- added C9: 15n, RP_KiCAD_Libs:C1608_WP, F.Cu at (107.0, 59.2)
- added D1: DIODE, RP_KiCAD_Libs:C3216, F.Cu at (55.5, 56.3)
- added FB1: FILTER, RP_KiCAD_Libs:C1608_WP, B.Cu at (31.0, 19.0)
- added FB2: FILTER, RP_KiCAD_Libs:C1608_WP, B.Cu at (30.0, 38.0)
- added FB3: FILTER, RP_KiCAD_Libs:C1608_WP, B.Cu at (44.0, 19.0)
- added FB4: FILTER, RP_KiCAD_Libs:C1608_WP, B.Cu at (43.0, 38.0)
- added FB5: FILTER, RP_KiCAD_Libs:C1608_WP, B.Cu at (57.0, 18.0)
- added FB6: FILTER, RP_KiCAD_Libs:C1608_WP, B.Cu at (56.0, 38.0)
- added GD1: DRV8302, Housings_SSOP:VSO-56_11.1x21.5mm_Pitch0.75mm, F.Cu at (39.0, 56.0)
- added L1: 22u, Inductors:SELF-WE-PD3S, F.Cu at (92.8, 43.8)
- added L2: 3.3u, Inductors:NR4018_HandSoldering, F.Cu at (80.0, 57.0)
- added L3: 3.3u, Inductors:NR4018_HandSoldering, F.Cu at (70.0, 75.0)
- added P1: CONN_01X02, RP_KiCAD_Connector:DEANS_T_F, F.Cu at (10.0, 20.0)
- added P2: CONN_01X02, RP_KiCAD_Connector:DEANS_T_M, F.Cu at (10.0, 10.0)
- added Q1: MOSFET_N, TO_SOT_Packages_SMD:D2-PAK_compact, B.Cu at (25.0, 15.0)
- added Q2: MOSFET_N, TO_SOT_Packages_SMD:D2-PAK_compact, B.Cu at (25.0, 32.0)
- added Q3: MOSFET_N, TO_SOT_Packages_SMD:D2-PAK_compact, B.Cu at (38.0, 15.0)
- added Q4: MOSFET_N, TO_SOT_Packages_SMD:D2-PAK_compact, B.Cu at (38.0, 32.0)
- added Q5: MOSFET_N, TO_SOT_Packages_SMD:D2-PAK_compact, B.Cu at (51.0, 15.0)
- added Q6: MOSFET_N, TO_SOT_Packages_SMD:D2-PAK_compact, B.Cu at (51.0, 32.0)
- added R1: 1M, RP_KiCAD_Libs:C1608_WP, F.Cu at (108.3, 49.5)
- added R10: 10, RP_KiCAD_Libs:C1608_WP, B.Cu at (30.0, 42.0)
- added R11: 10, RP_KiCAD_Libs:C1608_WP, B.Cu at (44.0, 23.0)
- added R12: 10, RP_KiCAD_Libs:C1608_WP, B.Cu at (43.0, 42.0)
- added R13: 10, RP_KiCAD_Libs:C1608_WP, B.Cu at (57.0, 22.0)
- added R14: 10, RP_KiCAD_Libs:C1608_WP, B.Cu at (56.0, 42.0)
- added R15: 1m, RP_KiCAD_Libs:C3225, B.Cu at (23.0, 39.0)
- added R16: 1m, RP_KiCAD_Libs:C3225, B.Cu at (36.0, 39.0)
- added R17: 1m, RP_KiCAD_Libs:C3225, B.Cu at (49.0, 39.0)
- added R2: 100, RP_KiCAD_Libs:C1608_WP, F.Cu at (98.0, 58.7)
- added R3: 100, RP_KiCAD_Libs:C1608_WP, F.Cu at (92.5, 64.8)
- added R4: 100, RP_KiCAD_Libs:C1608_WP, F.Cu at (85.0, 74.2)
- added R5: 100, RP_KiCAD_Libs:C1608_WP, F.Cu at (102.5, 55.6)
- added R6: 10k, RP_KiCAD_Libs:C1608_WP, B.Cu at (25.0, 35.0)
- added R7: 10k, RP_KiCAD_Libs:C1608_WP, B.Cu at (38.0, 35.0)
- added R8: 10k, RP_KiCAD_Libs:C1608_WP, B.Cu at (51.0, 35.0)
- added R9: 10, RP_KiCAD_Libs:C1608_WP, B.Cu at (31.0, 23.0)
- added U1: STM32F446RCTx, Housings_DFN_QFN:QFN-64-1EP_9x9mm_Pitch0.5mm, F.Cu at (28.0, 102.0)
- added X1: CRYSTAL, Crystals:ABM3_2pads, F.Cu at (21.0, 66.0)
Other:
- board outline added: 100 x 100 mm

Commit message: セルチェッカー作った｡電源基板ver1.1作った｡ぶっさしMDいじった｡DCDCいじりだした｡
Parts:
- C11, C12, C13, R2, R3, R4, R5: moved to B.Cu
- C15, C16: footprint RP_KiCAD_Libs:C3216 -> RP_KiCAD_Libs:C1608_WP; moved to B.Cu
- moved C13 75.4 mm to (36.5, 51.0), turned to 180 degrees
- moved C12 70.1 mm to (33.0, 51.0), turned to 180 degrees
- moved C11 63.0 mm to (29.5, 51.0), turned to 180 degrees
- moved R5 62.5 mm to (40.5, 48.0), turned to 270 degrees
- moved R2 56.5 mm to (42.5, 48.0), turned to 270 degrees
- moved R4 53.4 mm to (38.5, 48.0), turned to 270 degrees
- moved R3 50.9 mm to (44.5, 48.0), turned to 270 degrees
- moved C15 50.8 mm to (43.5, 51.0)
- moved D1 40.4 mm to (15.5, 51.0)
- moved U1 25.2 mm to (34.0, 77.5)
- moved C16 23.0 mm to (40.0, 51.0)
- moved C7 8.74 mm to (71.0, 64.5)
- moved R6 6.50 mm to (19.0, 32.5)
- moved R7 6.50 mm to (32.0, 32.5)
- moved R8 6.50 mm to (45.0, 32.5)
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Routing:
- net BRIDGE_A_SRL: track 0.00 -> 93.5 mm
- net BRIDGE_C_SRH: track 0.00 -> 78.9 mm, vias 0 -> 1
- net BRIDGE_A_SRH: track 0.00 -> 78.4 mm, vias 0 -> 1
- net BRIDGE_C_OUT: track 0.00 -> 58.3 mm, vias 0 -> 2
- net BRIDGE_A_OUT: track 0.00 -> 56.7 mm, vias 0 -> 2
- net BRIDGE_B_OUT: track 0.00 -> 49.8 mm, vias 0 -> 2
- net BRIDGE_B_SRH: track 0.00 -> 36.2 mm, vias 0 -> 1
- net BRIDGE_C_HG: track 0.00 -> 35.7 mm, vias 0 -> 1
- net BRIDGE_A_HG: track 0.00 -> 32.1 mm, vias 0 -> 1
- net BRIDGE_B_HG: track 0.00 -> 27.0 mm, vias 0 -> 1
- net BRIDGE_C_LG: track 0.00 -> 15.5 mm, vias 0 -> 1
- net BRIDGE_A_LG: track 0.00 -> 11.4 mm, vias 0 -> 1
- net Net-(FB6-Pad2): track 0.00 -> 7.45 mm
- net Net-(FB4-Pad2): track 0.00 -> 7.45 mm
- net Net-(FB2-Pad2): track 0.00 -> 7.45 mm
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
Commit message: BLMD設計終わり
Parts:
- removed GD1: DRV8302, Housings_SSOP:VSO-56_11.1x21.5mm_Pitch0.75mm
- removed L1: 22u, Inductors:SELF-WE-PD3S
- removed L2, L3: 3.3u, Inductors:NR4018_HandSoldering
- added C19: 4.7u, RP_KiCAD_Libs:C3216, F.Cu at (73.0, 23.5)
- added C20: 470u, Capacitors_SMD:c_elec_10x10.5, F.Cu at (21.5, 13.0)
- added C21: 470u, Capacitors_SMD:c_elec_10x10.5, F.Cu at (21.5, 28.0)
- added C22: 100u, Capacitors_ThroughHole:C_Radial_D6.3_L11.2_P2.5, F.Cu at (66.5, 15.0)
- added C23: 100u, Capacitors_ThroughHole:C_Radial_D6.3_L11.2_P2.5, F.Cu at (37.5, 75.0)
- added C24: 4.7u, RP_KiCAD_Libs:C3216, F.Cu at (45.0, 72.5)
- added C25: 4.7u, RP_KiCAD_Libs:C3216, F.Cu at (45.0, 76.5)
- added C26: 4.7u, RP_KiCAD_Libs:C3216, B.Cu at (42.0, 67.5)
- added C27: 4.7u, RP_KiCAD_Libs:C3216, B.Cu at (51.0, 67.5)
- added C28: 0.1u, RP_KiCAD_Libs:C1608_WP, F.Cu at (72.5, 44.5)
- added C29: 0.1u, RP_KiCAD_Libs:C1608_WP, F.Cu at (28.0, 48.0)
- added C30: 0.1u, RP_KiCAD_Libs:C1608_WP, F.Cu at (34.5, 54.5)
- added C31: 0.1u, RP_KiCAD_Libs:C1608_WP, B.Cu at (37.5, 65.0)
- added C32: 0.1u, RP_KiCAD_Libs:C1608_WP, F.Cu at (21.5, 54.5)
- added D10: LED, LEDs:LED_0805, F.Cu at (12.5, 45.0)
- added D11: LED, LEDs:LED_0805, F.Cu at (12.5, 48.0)
- added D2: DIODE, RP_KiCAD_Libs:C1608_WP, F.Cu at (45.5, 31.0)
- added D3: DIODE, RP_KiCAD_Libs:C1608_WP, F.Cu at (51.0, 31.0)
- added D4: DIODE, RP_KiCAD_Libs:C1608_WP, F.Cu at (57.5, 31.0)
- added D5: DIODE, RP_KiCAD_Libs:C1608_WP, F.Cu at (27.0, 31.0)
- added D6: DIODE, RP_KiCAD_Libs:C1608_WP, F.Cu at (33.5, 31.0)
- added D7: DIODE, RP_KiCAD_Libs:C3216, F.Cu at (65.0, 10.5)
- added D8: DIODE, RP_KiCAD_Libs:C3216, F.Cu at (38.5, 70.0)
- added D9: LED, LEDs:LED_0805, F.Cu at (12.5, 51.0)
- added ISO1: Si866x, Housings_SOIC:SOIC-16_3.9x9.9mm_Pitch1.27mm, F.Cu at (68.0, 39.0)
- added P10: CONN_01X01, Connect:1pin, F.Cu at (31.0, 18.0)
- added P11: CONN_01X02, Pin_Headers:Pin_Header_Straight_1x02, F.Cu at (8.50, 75.5)
- added P3: CONN_01X04, RP_KiCAD_Connector:XA_4LC, F.Cu at (13.0, 69.0)
- added P4: CONN_01X04, RP_KiCAD_Connector:XA_4LC, F.Cu at (25.5, 69.0)
- added P5: CONN_01X04, RP_KiCAD_Connector:XA_4LC, F.Cu at (55.0, 69.0)
- added P6: CONN_01X02, RP_KiCAD_Connector:DEANS_T_F, F.Cu at (6.50, 4.50)
- added P7: CONN_01X02, RP_KiCAD_Connector:DEANS_T_M, F.Cu at (6.50, 13.0)
- added P8: CONN_01X01, Connect:1pin, F.Cu at (43.0, 18.0)
- added P9: CONN_01X01, Connect:1pin, F.Cu at (55.0, 18.0)
- added R18: 10, RP_KiCAD_Libs:C1608_WP, F.Cu at (57.5, 29.0)
- added R19: 10, RP_KiCAD_Libs:C1608_WP, F.Cu at (27.0, 29.0)
- added R20: 10, RP_KiCAD_Libs:C1608_WP, F.Cu at (33.5, 29.0)
- added R21: 100, RP_KiCAD_Libs:C1608_WP, B.Cu at (39.5, 13.0)
- added R22: 100, RP_KiCAD_Libs:C1608_WP, B.Cu at (51.5, 13.0)
- added R23: 100, RP_KiCAD_Libs:C1608_WP, B.Cu at (27.5, 13.0)
- added R24: 10k, RP_KiCAD_Libs:C1608_WP, B.Cu at (62.5, 62.5)
- added R25: 4.7k, RP_KiCAD_Libs:C1608_WP, B.Cu at (62.5, 66.0)
- added R26: R, RP_KiCAD_Libs:C1608_WP, F.Cu at (65.0, 24.5)
- added R27: R, RP_KiCAD_Libs:C1608_WP, F.Cu at (63.5, 24.5)
- added R28: R, RP_KiCAD_Libs:C1608_WP, F.Cu at (66.5, 24.5)
- added R29: 10k, RP_KiCAD_Libs:C1608_WP, B.Cu at (60.0, 62.5)
- added R30: 4.7k, RP_KiCAD_Libs:C1608_WP, B.Cu at (60.0, 66.0)
- added R31: 120, RP_KiCAD_Libs:C1608_WP, B.Cu at (12.0, 71.0)
- added R32: 100, RP_KiCAD_Libs:C1608_WP, F.Cu at (16.5, 50.5)
- added R33: 100, RP_KiCAD_Libs:C1608_WP, F.Cu at (16.5, 45.5)
- added R34: 100, RP_KiCAD_Libs:C1608_WP, F.Cu at (16.5, 48.0)
- added SW1: SW_PUSH, Buttons_Switches_SMD:RP_SMD_Button, F.Cu at (4.50, 69.5)
- added SW2: SW_PUSH, Buttons_Switches_SMD:RP_SMD_Button, F.Cu at (4.50, 45.0)
- added SW3: SW_PUSH, Buttons_Switches_SMD:RP_SMD_Button, F.Cu at (4.50, 50.0)
- added U10: MAX3051, Housings_SOIC:SOIC-8_3.9x4.9mm_Pitch1.27mm, B.Cu at (32.5, 65.0)
- added U11: LM7805CT, TO_SOT_Packages_SMD:TO-252-2Lead, B.Cu at (38.5, 74.5)
- added U12: SW_ROTARY_16, Buttons_Switches_ThroughHole:rotary_0F, F.Cu at (5.00, 62.5)
- added U2: NCP1117ST33T3G, TO_SOT_Packages_SMD:SOT89-3_Housing, B.Cu at (46.5, 67.5)
- added U3: ACS758, RP_KiCAD_Libs:ACS785xCB, F.Cu at (9.00, 42.0)
- added U4: SI8234, Housings_SOIC:SOIC-16_3.9x9.9mm_Pitch1.27mm, F.Cu at (44.0, 39.0)
- added U5: SI8234, Housings_SOIC:SOIC-16_3.9x9.9mm_Pitch1.27mm, F.Cu at (56.0, 39.0)
- added U6: SI8234, Housings_SOIC:SOIC-16_3.9x9.9mm_Pitch1.27mm, F.Cu at (32.0, 39.0)
- added U7: LM324, Housings_SSOP:SSOP-14_5.3x6.2mm_Pitch0.65mm, F.Cu at (68.0, 30.0)
- added U8: LM7812ACT, TO_SOT_Packages_SMD:TO-252-2Lead, B.Cu at (65.5, 11.0)
- added U9: LM7805CT, TO_SOT_Packages_SMD:SOT89-3_Housing, B.Cu at (71.4, 21.6)
- C1, C2: value C -> 22p
- C10: value 100n -> 1u; footprint RP_KiCAD_Libs:C1608_WP -> RP_KiCAD_Libs:C3216
- C11, C12: footprint RP_KiCAD_Libs:C1608_WP -> RP_KiCAD_Libs:C3216; moved to F.Cu
- C13: value 1u -> 4.7u; footprint RP_KiCAD_Libs:C1608_WP -> RP_KiCAD_Libs:C3216; moved to F.Cu
- C15, C16: value 4.7n -> 0.1u
- C17: value 100u -> 0.1u; moved to B.Cu
- C3, C4: value C -> 0.1u
- C5: value 4.7u -> 0.1u; footprint RP_KiCAD_Libs:C3216 -> RP_KiCAD_Libs:C1608_WP
- C6: value 4.7u -> 470n; footprint RP_KiCAD_Libs:C3216 -> RP_KiCAD_Libs:C1608_WP; moved to B.Cu
- C7, C8: value 4.7u -> 1u
- C9: value 15n -> 1u; footprint RP_KiCAD_Libs:C1608_WP -> RP_KiCAD_Libs:C3216
- D1: footprint RP_KiCAD_Libs:C3216 -> RP_KiCAD_Libs:C1608_WP
- P1: value CONN_01X02 -> CONN_01X06; footprint RP_KiCAD_Connector:DEANS_T_F -> RP_KiCAD_Connector:ZH_6T
- P2: value CONN_01X02 -> CONN_01X06; footprint RP_KiCAD_Connector:DEANS_T_M -> RP_KiCAD_Connector:ZH_6T
- R1: value 1M -> 1k; moved to B.Cu
- R10, R9: value 10 -> R; moved to F.Cu
- R11: value 10 -> 4.7k
- R12, R13, R14: value 10 -> 10k
- R15, R16, R17: value 1m -> 10; footprint RP_KiCAD_Libs:C3225 -> RP_KiCAD_Libs:C1608_WP; moved to F.Cu
- R2: value 100 -> 1k
- R3, R4, R5: value 100 -> 10k
- R8: value 10k -> R; moved to F.Cu
- U1: value STM32F446RCTx -> STM32F103_48; footprint Housings_DFN_QFN:QFN-64-1EP_9x9mm_Pitch0.5mm -> Housings_QFP:LQFP-48_7x7mm_Pitch0.5mm
- moved C17 83.1 mm to (26.0, 10.5), turned to 90 degrees
- moved C6 76.4 mm to (10.0, 44.5), turned to 90 degrees
- moved C8 60.4 mm to (47.0, 33.5)
- moved C9 59.9 mm to (53.0, 33.5)
- moved C18 58.3 mm to (73.0, 19.5)
- moved C14 53.8 mm to (73.0, 8.50)
- moved C13 53.1 mm to (73.0, 12.5), turned to 0 degrees
- moved C5 51.5 mm to (42.0, 44.5), turned to 270 degrees
- moved R1 51.0 mm to (62.5, 72.0), turned to 90 degrees
- moved C1 45.4 mm to (17.0, 61.5), turned to 135 degrees
- moved C7 43.1 mm to (41.0, 33.5)
- moved C16 41.7 mm to (50.0, 10.5), turned to 90 degrees
- moved C15 40.9 mm to (38.0, 10.5), turned to 270 degrees
- moved C4 40.8 mm to (30.0, 44.5), turned to 270 degrees
- moved R6 39.7 mm to (4.50, 69.5), turned to 0 degrees
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Connections:
- C10 pad 2: Net-(C10-Pad2) -> GNDPWR
- C11 pad 1: BRIDGE_A_OUT -> Net-(C11-Pad1)
- C11 pad 2: Net-(C11-Pad2) -> /OUT_W
- C12 pad 1: BRIDGE_B_OUT -> Net-(C12-Pad1)
- C12 pad 2: Net-(C12-Pad2) -> GNDPWR
- C13 pad 1: BRIDGE_C_OUT -> Net-(C13-Pad1)
- C13 pad 2: Net-(C13-Pad2) -> GNDPWR
- C14 pad 1: BRIDGE_A_SRL -> /GD_12V
- C14 pad 2: V_SUPPLY -> GNDPWR
- C15 pad 1: SN2 -> +BATT
- C15 pad 2: SP2 -> Net-(C15-Pad2)
- C16 pad 1: SN1 -> Net-(C16-Pad1)
- C16 pad 2: SP1 -> +BATT
- C17 pad 1: +5V -> Net-(C17-Pad1)
- C17 pad 2: BRIDGE_A_SRL -> +BATT
- C18 pad 1: Net-(C18-Pad1) -> /GD_12V
- C18 pad 2: BRIDGE_A_SRL -> GNDPWR
- C3 pad 1: Net-(C3-Pad1) -> +3.3V
- C4 pad 1: Net-(C4-Pad1) -> +3.3V
- C4 pad 2: Net-(C4-Pad2) -> GND
- C5 pad 1: V_SUPPLY -> +3.3V
- C5 pad 2: Net-(C5-Pad2) -> GND
- C6 pad 1: V_SUPPLY -> /I_SENSE
- C6 pad 2: Net-(C5-Pad2) -> GND
- C7 pad 1: V_SUPPLY -> Net-(C7-Pad1)
- C7 pad 2: Net-(C5-Pad2) -> /OUT_U
- C8 pad 1: V_SUPPLY -> Net-(C8-Pad1)
- C8 pad 2: Net-(C5-Pad2) -> GNDPWR
- C9 pad 1: BRIDGE_A_SRL -> Net-(C9-Pad1)
- C9 pad 2: Net-(C9-Pad2) -> /OUT_V
- D1 pad 1: Net-(C10-Pad1) -> Net-(C7-Pad1)
- D1 pad 2: BRIDGE_A_SRL -> Net-(D1-Pad2)
- P1 pad 1: +BATT -> GND
- P1 pad 2: BRIDGE_A_SRL -> +3.3V
- P2 pad 1: +BATT -> GND
- P2 pad 2: BRIDGE_A_SRL -> /HALL_0
- Q1 pad S: BRIDGE_A_OUT -> /OUT_U
- Q2 pad D: BRIDGE_A_OUT -> /OUT_U
- Q2 pad S: BRIDGE_A_SRH -> GNDPWR
- Q3 pad S: BRIDGE_B_OUT -> /OUT_V
- Q4 pad D: BRIDGE_B_OUT -> /OUT_V
- Q4 pad S: BRIDGE_B_SRH -> GNDPWR
- Q5 pad S: BRIDGE_C_OUT -> /OUT_W
- Q6 pad D: BRIDGE_C_OUT -> /OUT_W
- Q6 pad S: BRIDGE_C_SRH -> GNDPWR
- R1 pad 1: BRIDGE_A_SRL -> +5V
- R1 pad 2: Net-(GD1-Pad49) -> /ENC_B
- R10 pad 1: Net-(FB2-Pad1) -> Net-(R10-Pad1)
- R10 pad 2: BRIDGE_A_LG -> GND
- R11 pad 1: Net-(FB3-Pad1) -> Net-(R11-Pad1)
- R11 pad 2: BRIDGE_B_HG -> /I_SENSE
- R12 pad 1: Net-(FB4-Pad1) -> GNDPWR
- R12 pad 2: BRIDGE_B_LG -> Net-(FB2-Pad1)
- R13 pad 1: Net-(FB5-Pad1) -> GNDPWR
- R13 pad 2: BRIDGE_C_HG -> Net-(FB4-Pad1)
- R14 pad 1: Net-(FB6-Pad1) -> GNDPWR
- R14 pad 2: BRIDGE_C_LG -> Net-(FB6-Pad1)
- R15 pad 1: BRIDGE_A_SRH -> /GD_12V
- R15 pad 2: BRIDGE_A_SRL -> Net-(D1-Pad2)
- R16 pad 1: BRIDGE_B_SRH -> /GD_12V
- R16 pad 2: BRIDGE_A_SRL -> Net-(D2-Pad2)
- R17 pad 1: BRIDGE_C_SRH -> /GD_12V
- R17 pad 2: BRIDGE_A_SRL -> Net-(D3-Pad2)
- R2 pad 1: BRIDGE_C_SRH -> +5V
- R2 pad 2: SN2 -> /ENC_A
- R3 pad 1: BRIDGE_A_SRL -> +5V
- R3 pad 2: SP2 -> /HALL_0
- R4 pad 1: BRIDGE_A_SRH -> +5V
- R4 pad 2: SN1 -> /HALL_1
- R5 pad 1: BRIDGE_A_SRL -> +5V
- R5 pad 2: SP1 -> /HALL_2
- R6 pad 1: Net-(FB2-Pad2) -> +3.3V
- R6 pad 2: BRIDGE_A_SRH -> /NRST
- R7 pad 1: Net-(FB4-Pad2) -> /BOOT0
- R7 pad 2: BRIDGE_B_SRH -> GND
- R8 pad 1: Net-(FB6-Pad2) -> Net-(R8-Pad1)
- R8 pad 2: BRIDGE_C_SRH -> GND
- R9 pad 1: Net-(FB1-Pad1) -> Net-(R9-Pad1)
- R9 pad 2: BRIDGE_A_HG -> GND
- U1 pad 10: (no net) -> Net-(R29-Pad2)
- U1 pad 11: (no net) -> Net-(R24-Pad2)
- U1 pad 12: GND -> /I_SENSE
- U1 pad 13: +3.3V -> /EN_V
- U1 pad 14: (no net) -> /EN_U
- U1 pad 15: (no net) -> /EN_W
- U1 pad 16: (no net) -> /PWM_V
- U1 pad 17: (no net) -> /PWM_U
- U1 pad 18: GND -> /PWM_W
- U1 pad 19: +3.3V -> (no net)
- U1 pad 2: (no net) -> /SEL_8
- U1 pad 23: (no net) -> GND
- U1 pad 24: (no net) -> +3.3V
- U1 pad 25: (no net) -> /COMP_U
- U1 pad 26: (no net) -> /COMP_V
- U1 pad 27: (no net) -> /COMP_W
- U1 pad 3: (no net) -> /SEL_2
- U1 pad 30: Net-(C3-Pad1) -> /USART_TX
- U1 pad 31: GND -> /USART_RX
- U1 pad 32: +3.3V -> /CAN_RX
- U1 pad 33: (no net) -> /CAN_TX
- U1 pad 34: (no net) -> /SWDIO
- U1 pad 35: (no net) -> GND
- U1 pad 36: (no net) -> +3.3V
- U1 pad 37: (no net) -> /SWCLK
- U1 pad 38: (no net) -> /HALL_0
- U1 pad 39: (no net) -> /HALL_1
- U1 pad 4: (no net) -> /SEL_1
- U1 pad 40: (no net) -> /HALL_2
- U1 pad 41: (no net) -> /LED_B
- U1 pad 42: (no net) -> /LED_A
- U1 pad 43: (no net) -> /SW1
- U1 pad 44: (no net) -> /BOOT0
- U1 pad 45: (no net) -> /SW2
- U1 pad 46: (no net) -> /SEL_4
- U1 pad 5: Net-(C2-Pad2) -> Net-(C1-Pad2)
- U1 pad 6: Net-(C1-Pad2) -> Net-(C2-Pad2)
- U1 pad 7: (no net) -> /NRST
- U1 pad 8: (no net) -> GND
- U1 pad 9: (no net) -> +3.3V
Routing:
- net +3.3V: track 0.00 -> 199.4 mm, vias 0 -> 13
- net GND: track 0.00 -> 186.2 mm, vias 0 -> 12
- net GNDPWR: track 0.00 -> 149.4 mm, vias 0 -> 5
- net /OUT_W: track 0.00 -> 103.2 mm, vias 0 -> 3
- net BRIDGE_A_SRL: track 93.5 -> 0.00 mm
- net +5V: track 0.00 -> 88.1 mm, vias 0 -> 2
- net /OUT_U: track 0.00 -> 81.5 mm, vias 0 -> 3
- net /GD_12V: track 0.00 -> 79.8 mm, vias 0 -> 8
- net BRIDGE_C_SRH: track 78.9 -> 0.00 mm, vias 1 -> 0
- net BRIDGE_A_SRH: track 78.4 -> 0.00 mm, vias 1 -> 0
- net /OUT_V: track 0.00 -> 69.4 mm, vias 0 -> 3
- net BRIDGE_C_OUT: track 58.3 -> 0.00 mm, vias 2 -> 0
- net +BATT: track 0.00 -> 57.2 mm, vias 0 -> 1
- net BRIDGE_A_OUT: track 56.7 -> 0.00 mm, vias 2 -> 0
- net BRIDGE_B_OUT: track 49.8 -> 0.00 mm, vias 2 -> 0
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- added copper zone on B.Cu, net +BATT
- added copper zone on F.Cu, net +BATT
- added copper zone on B.Cu, net /OUT_U
- added copper zone on B.Cu, net /OUT_V
- added copper zone on B.Cu, net /OUT_W
- added copper zone on B.Cu, net GND
- added copper zone on F.Cu, net GND
- added copper zone on B.Cu, net GNDPWR
- added copper zone on F.Cu, net GNDPWR
- added copper zone on B.Cu, net Net-(P6-Pad1)
- added copper zone on F.Cu, net Net-(P6-Pad1)
Other:
- board size 100 x 100 mm -> 76 x 78 mm
- net class Default: via_dia 0.6 -> 0.5; via_drill 0.4 -> 0.3

Commit message: 基板発注かけた
Parts:
- added D12: LED, LEDs:LED_0805, F.Cu at (16.5, 66.5)
- added D13: LED, LEDs:LED_0805, F.Cu at (65.0, 5.00)
- added P12: CONN_01X01, Connect:PINTST, F.Cu at (25.5, 47.5)
- added P13: CONN_01X01, Connect:PINTST, F.Cu at (21.0, 48.0)
- added P14: CONN_01X01, Connect:PINTST, F.Cu at (19.0, 48.0)
- added P15: CONN_01X01, Connect:PINTST, F.Cu at (67.0, 52.0)
- added P16: CONN_01X01, Connect:PINTST, F.Cu at (67.5, 50.0)
- added P17: CONN_01X01, Connect:PINTST, F.Cu at (68.0, 48.0)
- added P18: CONN_01X01, Connect:PINTST, F.Cu at (50.5, 44.5)
- added P19: CONN_01X01, Connect:PINTST, F.Cu at (26.5, 44.5)
- added P20: CONN_01X01, Connect:PINTST, F.Cu at (38.5, 44.5)
- added R35: 1k, RP_KiCAD_Libs:C1608_WP, F.Cu at (13.0, 66.5)
- added R36: 1k, RP_KiCAD_Libs:C1608_WP, F.Cu at (67.5, 5.00)
- moved R3 0.71 mm to (22.5, 45.5)
- moved R4 0.71 mm to (20.5, 45.5)
- moved R5 0.71 mm to (18.5, 45.5)
Routing:
- net GNDPWR: track 149.4 -> 157.9 mm
- net /HALL_2: track 12.5 -> 17.4 mm
- net /GD_12V: track 79.8 -> 84.2 mm
- net +12V: track 25.8 -> 29.1 mm
- net /HALL_1: track 11.4 -> 14.7 mm, vias 0 -> 1
- net GND: track 186.2 -> 189.1 mm
- net Net-(D13-Pad2): track 0.00 -> 2.56 mm
- net /NRST: track 27.3 -> 29.3 mm
- net Net-(D12-Pad2): track 0.00 -> 1.55 mm
- net /PWM_V: track 35.4 -> 36.5 mm
- net /PWM_W: track 26.3 -> 27.5 mm
- net /PWM_U: track 23.5 -> 24.6 mm
- net /COMP_U: track 46.0 -> 46.6 mm
Other:
- board text added: "0"
- board text added: "1"
- board text added: "2"
- board text added: "U"
- board text added: "V"
- board text added: "W"
