File: KiCAD_Projects/ISO_DCDC_ver1.1/ISO_DCDC_ver1.1.sch (KiCad schematic (older format))
At the start: 75 parts, among them IC3 PC817, IC4 PC817, IC5 PC817, P1 CONN_01X01, P10 CONN_01X02, P11 CONN_01X02, P12 CONN_01X01, P13 CONN_01X04, P15 CONN_01X02, P16 TST, P19 CONN_01X01, P2 CONN_01X01, P20 CONN_01X01, P21 CONN_01X02, P22 CONN_01X01, P23 CONN_01X01, P25 CONN_01X01, P26 CONN_01X01, P3 CONN_01X01, P4 CONN_01X02, P5 CONN_01X02, P8 CONN_01X01, P9 CONN_01X01, Q1 MOSFET_N, U1 V23076-D3001-D142, U2 V23076-D3001-D142, U3 V23076-D3001-D142

Commit message: セルチェッカー作った｡電源基板ver1.1作った｡ぶっさしMDいじった｡DCDCいじりだした｡
Parts:
- removed D4: LED, LEDs:LED-3MM, symbol LED
- removed R7: 1k, RP_KiCAD_Libs:C1608_WP, symbol R
- added D4: DIODE, RP_KiCAD_Libs:C3216, symbol DIODE
- added P14, P6, P7: CONN_01X02, RP_KiCAD_Connector:XA_2T, symbol CONN_01X02
- added R15: 1k, RP_KiCAD_Libs:C1608_NP, symbol R
- C11, C2, C5, C8, R1, R10, R11, R14, R17, R18, R20, R21, R22, R23, R3, R4, R5, R6, R8, R9: footprint RP_KiCAD_Libs:C1608_WP -> RP_KiCAD_Libs:C1608_NP
Connections:
- net 12V_CAN is gone; now on net 12V: D5.1 (A)
- net 12V_CAN_GND is gone; now on net GND: R8.2
- net 12V: now also R14.2
- net 12V_RasPi: now also P11.2 (P2), P6.2 (P2), P7.2 (P2)
- net 12V_RasPi_GND: now also C1.2, DCDC4.3 (-Vout), IC3.2, P6.1 (P1), P7.1 (P1)
- net GND: no longer C1.2, DCDC4.3 (-Vout), IC3.2, P11.2 (P2)
- net GNDPWR: now also P14.1 (P1)
- net at C3.1, C4.1, C6.1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: now also D4.1 (K)
- net at IC5.4, R14.1: now also R15.2; no longer P13.4 (P4)
- new net: P13.4 (P4), R15.1
- new net: D4.2 (A), P14.2 (P2)
Other:
- moved on the sheet: P13

Commit message: コンパネver1.1作った｡本番仕様サジ電源基板つくった
Parts:
- removed D6: LED, LEDs:LED-3MM, symbol LED
- removed P9: CONN_01X01, Connect:1pin, symbol CONN_01X01
- removed R12, R2: 8.2, Resistors_SMD:R_2512, symbol R
- removed R5: 2.2k, RP_KiCAD_Libs:C1608_NP, symbol R
- removed U2: V23076-D3001-D142, Relays_ThroughHole:V23076-A3001-D142, symbol V23076-D3001-D142
- R13, R19: footprint RP_KiCAD_Libs:0204_2f5 -> RP_KiCAD_Libs:0204_2f7
Connections:
- net 15V: now also R19.2; no longer IC4.4
- net at C3.1, C4.1, C6.1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: now also P20.1 (P1)
- net at Q1.G, R11.1: now also IC3.3; no longer R19.2
- net at R19.1: now also IC4.4; no longer IC3.3
- net at D10.1 (A), P22.1 (P1), U1.5 (NO): now also P2.1 (P1)
Other:
- moved on the sheet: P2, P20, P3, R19
Changed lines of the file:
@@
-$EndComp
-$Comp
-L R R2
-U 1 1 57D737B9
-P 2850 3700
-F 0 "R2" V 2930 3700 40  0000 C CNN
-F 1 "8.2" V 2857 3701 40  0000 C CNN
-F 2 "Resistors_SMD:R_2512" V 2780 3700 30  0001 C CNN
-F 3 "" H 2850 3700 30  0000 C CNN
-	1    2850 3700
-	0    1    1    0
-$EndComp
-$Comp
-L R R12
-U 1 1 57D73CF6
-P 2850 3850
-F 0 "R12" V 2930 3850 40  0000 C CNN
-F 1 "8.2" V 2857 3851 40  0000 C CNN
-F 2 "Resistors_SMD:R_2512" V 2780 3850 30  0001 C CNN
-F 3 "" H 2850 3850 30  0000 C CNN
-	1    2850 3850
-	0    1    1    0
 $EndComp
 $Comp
@@
 L CONN_01X01 P20
 U 1 1 57DA5871
-P 2350 3900
-F 0 "P20" H 2350 4000 50  0000 C CNN
-F 1 "CONN_01X01" V 2450 3900 50  0000 C CNN
-F 2 "Connect:1pin" H 2350 3900 50  0001 C CNN
-F 3 "" H 2350 3900 50  0000 C CNN
-	1    2350 3900
-	0    1    1    0
+P 2450 3700
+F 0 "P20" H 2450 3800 50  0000 C CNN
+F 1 "CONN_01X01" V 2550 3700 50  0000 C CNN
+F 2 "Connect:1pin" H 2450 3700 50  0001 C CNN
+F 3 "" H 2450 3700 50  0000 C CNN
+	1    2450 3700
+	-1   0    0    1
 $EndComp
 Text Label 5400 2550 0    60   ~ 0
 15V
-Text Label 6300 6500 2    60   ~ 0
+Text Label 6000 6500 2    60   ~ 0
 15V
 Text Label 5300 9700 1    60   ~ 0
@@
 L R R19
 U 1 1 57DC0B9F
-P 5400 7100
-F 0 "R19" V 5480 7100 40  0000 C CNN
-F 1 "R" V 5407 7101 40  0000 C CNN
-F 2 "RP_KiCAD_Libs:0204_2f5" V 5330 7100 30  0001 C CNN
-F 3 "" H 5400 7100 30  0000 C CNN
-	1    5400 7100
+P 6150 6500
+F 0 "R19" V 6230 6500 40  0000 C CNN
+F 1 "R" V 6157 6501 40  0000 C CNN
+F 2 "RP_KiCAD_Libs:0204_2f7" V 6080 6500 30  0001 C CNN
+F 3 "" H 6150 6500 30  0000 C CNN
+	1    6150 6500
 	0    1    1    0
 $EndComp
@@
 P 1400 7700
 F 0 "#PWR017" H 1400 7750 40  0001 C CNN
-F 1 "GNDPWR" H 1400 7620 40  0000 C CNN
+F 1 "GNDPWR" H 1400 7650 40  0000 C CNN
 F 2 "" H 1400 7700 60  0001 C CNN
 F 3 "" H 1400 7700 60  0001 C CNN
@@
 $EndComp
 $Comp
-L V23076-D3001-D142 U2
-U 1 1 5806E0D8
-P 2300 8900
-F 0 "U2" H 2350 9150 60  0000 C CNN
-F 1 "V23076-D3001-D142" H 2300 8650 60  0000 C CNN
-F 2 "Relays_ThroughHole:V23076-A3001-D142" H 2300 8900 60  0001 C CNN
-F 3 "" H 2300 8900 60  0000 C CNN
-	1    2300 8900
-	-1   0    0    1
-$EndComp
-$Comp
-L GNDPWR #PWR021
-U 1 1 5806E0DE
-P 1400 9300
-F 0 "#PWR021" H 1400 9350 40  0001 C CNN
-F 1 "GNDPWR" H 1400 9220 40  0000 C CNN
-F 2 "" H 1400 9300 60  0001 C CNN
-F 3 "" H 1400 9300 60  0001 C CNN
-	1    1400 9300
-	0    -1   -1   0
-$EndComp
-$Comp
-L LED D6
-U 1 1 5806E0F1
-P 1800 9250
-F 0 "D6" H 1800 9350 50  0000 C CNN
-F 1 "LED" H 1800 9150 50  0000 C CNN
-F 2 "LEDs:LED-3MM" H 1800 9250 60  0001 C CNN
-F 3 "" H 1800 9250 60  0000 C CNN
-	1    1800 9250
-	0    1    1    0
-$EndComp
-$Comp
-L R R5
-U 1 1 5806E0F7
-P 1800 9600
-F 0 "R5" V 1880 9600 40  0000 C CNN
-F 1 "2.2k" V 1807 9601 40  0000 C CNN
-F 2 "RP_KiCAD_Libs:C1608_NP" V 1730 9600 30  0001 C CNN
-F 3 "" H 1800 9600 30  0000 C CNN
-	1    1800 9600
-	1    0    0    -1
-$EndComp
-$Comp
-L GNDPWR #PWR022
-U 1 1 5806E0FE
-P 1800 9850
-F 0 "#PWR022" H 1800 9900 40  0001 C CNN
-F 1 "GNDPWR" H 1800 9770 40  0000 C CNN
-F 2 "" H 1800 9850 60  0001 C CNN
-F 3 "" H 1800 9850 60  0001 C CNN
-	1    1800 9850
-	1    0    0    -1
-$EndComp
-Text Label 2700 8800 0    60   ~ 0
-POWER_EN_HIGH
-Text Label 2700 9000 0    60   ~ 0
-POWER_EN_LOW
-$Comp
 L CONN_01X01 P2
 U 1 1 5806E107
-P 1200 9050
-F 0 "P2" H 1200 9150 50  0000 C CNN
-F 1 "CONN_01X01" V 1300 9050 50  0000 C CNN
-F 2 "Connect:1pin" H 1200 9050 50  0001 C CNN
-F 3 "" H 1200 9050 50  0000 C CNN
-	1    1200 9050
+P 650 7450
+F 0 "P2" H 650 7550 50  0000 C CNN
+F 1 "CONN_01X01" V 750 7450 50  0000 C CNN
+F 2 "Connect:1pin" H 650 7450 50  0001 C CNN
+F 3 "" H 650 7450 50  0000 C CNN
+	1    650  7450
 	-1   0    0    1
 $EndComp
@@
 L CONN_01X01 P3
 U 1 1 5806E10D
-P 1200 9300
-F 0 "P3" H 1200 9400 50  0000 C CNN
-F 1 "CONN_01X01" V 1300 9300 50  0000 C CNN
-F 2 "Connect:1pin" H 1200 9300 50  0001 C CNN
-F 3 "" H 1200 9300 50  0000 C CNN
-	1    1200 9300
-	-1   0    0    1
-$EndComp
-$Comp
-L GNDPWR #PWR023
+P 650 7700
+F 0 "P3" H 650 7800 50  0000 C CNN
+F 1 "CONN_01X01" V 750 7700 50  0000 C CNN
+F 2 "Connect:1pin" H 650 7700 50  0001 C CNN
+F 3 "" H 650 7700 50  0000 C CNN
+	1    650  7700
+	-1   0    0    1
+$EndComp
+$Comp
+L GNDPWR #PWR021
 U 1 1 5807533D
 P 4200 9150
-F 0 "#PWR023" H 4200 9200 40  0001 C CNN
+F 0 "#PWR021" H 4200 9200 40  0001 C CNN
 F 1 "GNDPWR" H 4200 9070 40  0000 C CNN
 F 2 "" H 4200 9150 60  0001 C CNN
 F 3 "" H 4200 9150 60  0001 C CNN
 	1    4200 9150
-	0    -1   -1   0
-$EndComp
-$Comp
-L CONN_01X01 P9
-U 1 1 58075343
-P 1500 8550
-F 0 "P9" H 1500 8650 50  0000 C CNN
-F 1 "CONN_01X01" V 1600 8550 50  0000 C CNN
-F 2 "Connect:1pin" H 1500 8550 50  0001 C CNN
-F 3 "" H 1500 8550 50  0000 C CNN
-	1    1500 8550
 	0    -1   -1   0
 $EndComp
@@
 POWER_EN_HIGH
 $Comp
-L GNDPWR #PWR024
+L GNDPWR #PWR022
 U 1 1 5808D408
 P 6350 7600
-F 0 "#PWR024" H 6350 7650 40  0001 C CNN
+F 0 "#PWR022" H 6350 7650 40  0001 C CNN
 F 1 "GNDPWR" H 6350 7520 40  0000 C CNN
 F 2 "" H 6350 7600 60  0001 C CNN
@@
 Wire Notes Line
 	2550 3550 2550 1550
-Wire Wire Line
-	2350 3700 2700 3700
-Connection ~ 2650 3700
-Wire Wire Line
-	2700 3850 2650 3850
 Connection ~ 3050 3700
-Wire Wire Line
-	3000 3850 3050 3850
 Wire Wire Line
 	1750 6550 1750 6650
@@
 Connection ~ 4600 7400
 Wire Wire Line
-	4900 7100 5250 7100
+	4900 7100 5550 7100
 Connection ~ 5100 7100
 Wire Wire Line
@@
 	3050 3700 3050 4350
 Wire Wire Line
-	2650 3850 2650 3700
-Wire Wire Line
 	1700 5750 1800 5750
 Wire Wire Line
-	1850 8750 1750 8750
-Wire Wire Line
-	1750 8750 1750 8950
-Wire Wire Line
-	1750 8950 1850 8950
-Wire Wire Line
-	1500 8850 1850 8850
-Connection ~ 1750 8850
-Wire Wire Line
-	1400 9050 1850 9050
-Wire Wire Line
-	1500 8750 1500 8850
-Wire Wire Line
-	1800 9750 1800 9850
-Connection ~ 1800 9050
-Wire Wire Line
 	7300 6500 7400 6500
 Wire Wire Line
@@
 	7300 7250 7550 7250
 Wire Wire Line
-	5800 7100 5550 7100
-Wire Wire Line
-	6000 6700 6300 6700
-Wire Wire Line
-	6000 4950 6300 4950
-Wire Wire Line
-	6300 5150 5800 5150
-Wire Wire Line
-	5800 5150 5800 7100
-Wire Wire Line
-	3000 3700 3200 3700
+	5700 6700 6300 6700
+Wire Wire Line
+	5700 4950 6300 4950
+Wire Wire Line
+	6300 5150 5550 5150
+Wire Wire Line
+	5550 5150 5550 7100
+Wire Wire Line
+	2650 3700 3200 3700
 Wire Wire Line
 	7000 6700 7100 6700
@@
 	4300 3500 4600 3500
 $Comp
-L GNDPWR #PWR025
+L GNDPWR #PWR023
 U 1 1 5824D96D
 P 4450 3550
-F 0 "#PWR025" H 4450 3600 40  0001 C CNN
+F 0 "#PWR023" H 4450 3600 40  0001 C CNN
 F 1 "GNDPWR" H 4450 3470 40  0000 C CNN
 F 2 "" H 4450 3550 60  0001 C CNN
@@
 F 0 "R13" V 6280 7400 40  0000 C CNN
 F 1 "R" V 6207 7401 40  0000 C CNN
-F 2 "RP_KiCAD_Libs:0204_2f5" V 6130 7400 30  0001 C CNN
+F 2 "RP_KiCAD_Libs:0204_2f7" V 6130 7400 30  0001 C CNN
 F 3 "" H 6200 7400 30  0000 C CNN
 	1    6200 7400
@@
 $EndComp
 $Comp
-L GND #PWR026
+L GND #PWR024
 U 1 1 58C7FC3A
 P 7450 3900
-F 0 "#PWR026" H 7450 3900 30  0001 C CNN
+F 0 "#PWR024" H 7450 3900 30  0001 C CNN
 F 1 "GND" H 7450 3830 30  0001 C CNN
 F 2 "" H 7450 3900 60  0001 C CNN
@@
 $EndComp
 $Comp
-L GND #PWR027
+L GND #PWR025
 U 1 1 58C80D75
 P 9150 2750
-F 0 "#PWR027" H 9150 2750 30  0001 C CNN
+F 0 "#PWR025" H 9150 2750 30  0001 C CNN
 F 1 "GND" H 9150 2680 30  0001 C CNN
 F 2 "" H 9150 2750 60  0001 C CNN
@@
 $EndComp
 $Comp
-L GND #PWR028
+L GND #PWR026
 U 1 1 58C80F52
 P 9750 2750
-F 0 "#PWR028" H 9750 2750 30  0001 C CNN
+F 0 "#PWR026" H 9750 2750 30  0001 C CNN
 F 1 "GND" H 9750 2680 30  0001 C CNN
 F 2 "" H 9750 2750 60  0001 C CNN
@@
 12V
 Wire Wire Line
-	6000 4950 6000 6700
-$Comp
-L GND #PWR029
+	5700 4950 5700 6700
+$Comp
+L GND #PWR027
 U 1 1 58C832A5
 P 7100 6700
-F 0 "#PWR029" H 7100 6700 30  0001 C CNN
+F 0 "#PWR027" H 7100 6700 30  0001 C CNN
 F 1 "GND" H 7100 6630 30  0001 C CNN
 F 2 "" H 7100 6700 60  0001 C CNN
@@
 $EndComp
 $Comp
-L GND #PWR030
+L GND #PWR028
 U 1 1 58C83789
 P 7150 7600
-F 0 "#PWR030" H 7150 7600 30  0001 C CNN
+F 0 "#PWR028" H 7150 7600 30  0001 C CNN
 F 1 "GND" H 7150 7530 30  0001 C CNN
 F 2 "" H 7150 7600 60  0001 C CNN
@@
 $EndComp
 $Comp
-L GND #PWR031
+L GND #PWR029
 U 1 1 58C83F47
 P 7850 6950
-F 0 "#PWR031" H 7850 6950 30  0001 C CNN
+F 0 "#PWR029" H 7850 6950 30  0001 C CNN
 F 1 "GND" H 7850 6880 30  0001 C CNN
 F 2 "" H 7850 6950 60  0001 C CNN
@@
 $EndComp
 $Comp
-L GNDPWR #PWR032
+L GNDPWR #PWR030
 U 1 1 58C95A54
 P 5650 10500
-F 0 "#PWR032" H 5650 10550 40  0001 C CNN
+F 0 "#PWR030" H 5650 10550 40  0001 C CNN
 F 1 "GNDPWR" H 5650 10420 40  0000 C CNN
 F 2 "" H 5650 10500 60  0001 C CNN
@@
 	5800 3700 5800 4100
 $Comp
-L GND #PWR033
+L GND #PWR031
 U 1 1 58C9F653
 P 9050 8900
-F 0 "#PWR033" H 9050 8900 30  0001 C CNN
+F 0 "#PWR031" H 9050 8900 30  0001 C CNN
 F 1 "GND" H 9050 8830 30  0001 C CNN
 F 2 "" H 9050 8900 60  0001 C CNN
@@
 $EndComp
 $Comp
-L GNDPWR #PWR034
+L GNDPWR #PWR032
 U 1 1 58CAB745
 P 2550 4450
-F 0 "#PWR034" H 2550 4500 40  0001 C CNN
+F 0 "#PWR032" H 2550 4500 40  0001 C CNN
 F 1 "GNDPWR" H 2550 4370 40  0000 C CNN
 F 2 "" H 2550 4450 60  0001 C CNN
@@
 Wire Wire Line
 	3050 4350 3000 4350
-Connection ~ 3050 3850
 Wire Wire Line
 	2600 4350 2550 4350
+$Comp
+L GNDPWR #PWR033
+U 1 1 58DA68D2
+P 850 7700
+F 0 "#PWR033" H 850 7750 40  0001 C CNN
+F 1 "GNDPWR" H 850 7650 40  0000 C CNN
+F 2 "" H 850 7700 60  0001 C CNN
+F 3 "" H 850 7700 60  0001 C CNN
+	1    850  7700
+	0    -1   -1   0
+$EndComp
+Wire Wire Line
+	850  7450 950  7450
+Wire Wire Line
+	950  7450 950  7350
+Wire Wire Line
+	950  7350 1500 7350
+Wire Wire Line
+	1500 7350 1500 7450
+Connection ~ 1500 7450
 $EndSCHEMATC
