File: KiCAD_Projects/BLDC_MD_ver1.1/_saved_BLDC_MD_ver1.1.sch (KiCad schematic (older format))
At the start: 152 parts, among them P1 CONN_01X06, P10 CONN_01X01, P11 CONN_01X02, P12 CONN_01X01, P13 CONN_01X01, P14 CONN_01X01, P15 CONN_01X01, P16 CONN_01X01, P17 CONN_01X01, P18 CONN_01X01, P19 CONN_01X01, P2 CONN_01X06, P20 CONN_01X01, P21 CONN_01X04, P22 CONN_01X04, P23 CONN_01X01, P24 CONN_01X02, P25 CONN_01X01, P3 CONN_01X04, P4 CONN_01X04, P5 CONN_01X04, P6 CONN_01X02, P7 CONN_01X02, P8 CONN_01X01, P9 CONN_01X01, Q1 MOSFET_N, Q10 MOSFET_N, Q2 MOSFET_N, Q3 MOSFET_N, Q4 MOSFET_N, Q5 MOSFET_N, Q6 MOSFET_N, Q7 MOSFET_N, Q8 MOSFET_N, Q9 MOSFET_N, SW1 SW_PUSH, SW2 SW_PUSH, SW3 SW_PUSH, U1 STM32F103_48, U10 MAX3051, U11 LM7805CT, U13 V23076-D3001-D142, U2 NCP1117ST33T3G, U3 ACS758, U4 SI8234, U5 SI8234, U6 SI8234, U7 LM324, U8 LM7812ACT, U9 LM7805CT, X1 CRYSTAL

Commit message: BLMDver1.1設計大体終わり｡
Parts:
- added C23: C, Capacitors_ThroughHole:C_Radial_D5_L11_P2.5, symbol C
- added R44: R, RP_KiCAD_Libs:C3216, symbol R
- added SW4, SW5, SW6, SW7: SWITCH_INV, symbol SWITCH_INV
- C33: footprint RP_KiCAD_Libs:C1608_WP -> Capacitors_ThroughHole:C_Radial_D8_L11.5_P3.5
- C34: footprint RP_KiCAD_Libs:C1608_WP -> Capacitors_ThroughHole:C_Radial_D5_L11_P2.5
- P21: footprint RP_KiCAD_Connector:XA_4T -> RP_KiCAD_Connector:XA_4LC
- P24: footprint RP_KiCAD_Connector:XA_2T -> RP_KiCAD_Connector:XA_2LC
Connections:
- net labels added: TOGGLE_0, TOGGLE_1, TOGGLE_2, TOGGLE_3
- wire segments 179 -> 180
Changed lines of the file:
@@
 Text Label 3850 4300 3    60   ~ 0
 COMP_W
+Text Label 3950 4300 3    60   ~ 0
+HALL_0
 Text Label 4050 4300 3    60   ~ 0
-HALL_0
+HALL_1
 Text Label 4150 4300 3    60   ~ 0
-HALL_1
-Text Label 4250 4300 3    60   ~ 0
 HALL_2
 Text Label 2000 3500 2    60   ~ 0
@@
 F 0 "C34" H 15350 11400 40  0000 L CNN
 F 1 "C" H 15356 11215 40  0000 L CNN
-F 2 "RP_KiCAD_Libs:C1608_WP" H 15388 11150 30  0001 C CNN
+F 2 "Capacitors_ThroughHole:C_Radial_D5_L11_P2.5" H 15388 11150 30  0001 C CNN
 F 3 "" H 15350 11300 60  0000 C CNN
 	1    15350 11300
@@
 F 0 "C33" H 13700 11300 40  0000 L CNN
 F 1 "C" H 13706 11115 40  0000 L CNN
-F 2 "RP_KiCAD_Libs:C1608_WP" H 13738 11050 30  0001 C CNN
+F 2 "Capacitors_ThroughHole:C_Radial_D8_L11.5_P3.5" H 13738 11050 30  0001 C CNN
 F 3 "" H 13700 11200 60  0000 C CNN
 	1    13700 11200
@@
 F 0 "P24" H 15750 10800 50  0000 C CNN
 F 1 "CONN_01X02" V 15850 10650 50  0000 C CNN
-F 2 "RP_KiCAD_Connector:XA_2T" H 15750 10650 50  0001 C CNN
+F 2 "RP_KiCAD_Connector:XA_2LC" H 15750 10650 50  0001 C CNN
 F 3 "" H 15750 10650 50  0000 C CNN
 	1    15750 10650
-	1    0    0    1
+	1    0    0    -1
 $EndComp
 $Comp
@@
 Connection ~ 15200 8300
 Wire Wire Line
-	15200 8300 15200 9250
+	15200 7950 15200 9250
 $Comp
 L DIODE D17
@@
 F 0 "P21" H 12150 9700 50  0000 C CNN
 F 1 "CONN_01X04" V 12250 9450 50  0000 C CNN
-F 2 "RP_KiCAD_Connector:XA_4T" H 12150 9450 50  0001 C CNN
+F 2 "RP_KiCAD_Connector:XA_4LC" H 12150 9450 50  0001 C CNN
 F 3 "" H 12150 9450 50  0000 C CNN
 	1    12150 9450
@@
 Text Label 12100 11350 0    60   ~ 0
 EMG_OUT
+$Comp
+L C C23
+U 1 1 58F7BBF7
+P 15200 11300
+F 0 "C23" H 15200 11400 40  0000 L CNN
+F 1 "C" H 15206 11215 40  0000 L CNN
+F 2 "Capacitors_ThroughHole:C_Radial_D5_L11_P2.5" H 15238 11150 30  0001 C CNN
+F 3 "" H 15200 11300 60  0000 C CNN
+	1    15200 11300
+	1    0    0    -1
+$EndComp
+Connection ~ 15200 11100
+Connection ~ 15200 11500
+$Comp
+L R R44
+U 1 1 58F7DAE2
+P 14450 7950
+F 0 "R44" V 14530 7950 40  0000 C CNN
+F 1 "R" V 14457 7951 40  0000 C CNN
+F 2 "RP_KiCAD_Libs:C3216" V 14380 7950 30  0001 C CNN
+F 3 "" H 14450 7950 30  0000 C CNN
+	1    14450 7950
+	0    1    1    0
+$EndComp
+$Comp
+L GND #PWR0126
+U 1 1 58F7F10B
+P 14300 7950
+F 0 "#PWR0126" H 14300 7950 30  0001 C CNN
+F 1 "GND" H 14300 7880 30  0001 C CNN
+F 2 "" H 14300 7950 60  0001 C CNN
+F 3 "" H 14300 7950 60  0001 C CNN
+	1    14300 7950
+	0    1    1    0
+$EndComp
+Wire Wire Line
+	14600 7950 15200 7950
+$Comp
+L SWITCH_INV SW4
+U 1 1 58E4A923
+P 8000 4900
+F 0 "SW4" H 7800 5050 50  0000 C CNN
+F 1 "SWITCH_INV" H 7850 4750 50  0000 C CNN
+F 2 "" H 8000 4900 60  0000 C CNN
+F 3 "" H 8000 4900 60  0000 C CNN
+	1    8000 4900
+	1    0    0    -1
+$EndComp
+$Comp
+L SWITCH_INV SW5
+U 1 1 58E4B7B2
+P 8000 5300
+F 0 "SW5" H 7800 5450 50  0000 C CNN
+F 1 "SWITCH_INV" H 7850 5150 50  0000 C CNN
+F 2 "" H 8000 5300 60  0000 C CNN
+F 3 "" H 8000 5300 60  0000 C CNN
+	1    8000 5300
+	1    0    0    -1
+$EndComp
+$Comp
+L SWITCH_INV SW6
+U 1 1 58E4BE0C
+P 8000 5650
+F 0 "SW6" H 7800 5800 50  0000 C CNN
+F 1 "SWITCH_INV" H 7850 5500 50  0000 C CNN
+F 2 "" H 8000 5650 60  0000 C CNN
+F 3 "" H 8000 5650 60  0000 C CNN
+	1    8000 5650
+	1    0    0    -1
+$EndComp
+$Comp
+L SWITCH_INV SW7
+U 1 1 58E4C002
+P 8000 6000
+F 0 "SW7" H 7800 6150 50  0000 C CNN
+F 1 "SWITCH_INV" H 7850 5850 50  0000 C CNN
+F 2 "" H 8000 6000 60  0000 C CNN
+F 3 "" H 8000 6000 60  0000 C CNN
+	1    8000 6000
+	1    0    0    -1
+$EndComp
+$Comp
+L GND #PWR0127
+U 1 1 58E4C15C
+P 8500 6100
+F 0 "#PWR0127" H 8500 6100 30  0001 C CNN
+F 1 "GND" H 8500 6030 30  0001 C CNN
+F 2 "" H 8500 6100 60  0001 C CNN
+F 3 "" H 8500 6100 60  0001 C CNN
+	1    8500 6100
+	0    -1   -1   0
+$EndComp
+$Comp
+L GND #PWR0128
+U 1 1 58E4CADD
+P 8500 5750
+F 0 "#PWR0128" H 8500 5750 30  0001 C CNN
+F 1 "GND" H 8500 5680 30  0001 C CNN
+F 2 "" H 8500 5750 60  0001 C CNN
+F 3 "" H 8500 5750 60  0001 C CNN
+	1    8500 5750
+	0    -1   -1   0
+$EndComp
+$Comp
+L GND #PWR0129
+U 1 1 58E4CCCB
+P 8500 5400
+F 0 "#PWR0129" H 8500 5400 30  0001 C CNN
+F 1 "GND" H 8500 5330 30  0001 C CNN
+F 2 "" H 8500 5400 60  0001 C CNN
+F 3 "" H 8500 5400 60  0001 C CNN
+	1    8500 5400
+	0    -1   -1   0
+$EndComp
+$Comp
+L GND #PWR0130
+U 1 1 58E4E5FE
+P 8500 5000
+F 0 "#PWR0130" H 8500 5000 30  0001 C CNN
+F 1 "GND" H 8500 4930 30  0001 C CNN
+F 2 "" H 8500 5000 60  0001 C CNN
+F 3 "" H 8500 5000 60  0001 C CNN
+	1    8500 5000
+	0    -1   -1   0
+$EndComp
+Text Label 7500 4900 2    60   ~ 0
+TOGGLE_0
+Text Label 7500 5300 2    60   ~ 0
+TOGGLE_1
+Text Label 7500 5650 2    60   ~ 0
+TOGGLE_2
+Text Label 7500 6000 2    60   ~ 0
+TOGGLE_3
+Text Label 4350 1000 1    60   ~ 0
+TOGGLE_0
+Text Label 4250 1000 1    60   ~ 0
+TOGGLE_1
+Text Label 4150 1000 1    60   ~ 0
+TOGGLE_2
+Text Label 3550 1000 1    60   ~ 0
+TOGGLE_3
 $EndSCHEMATC
