File: KiCAD_Projects/CanDCMD_ver1.0/CanDCMD_ver1.0.kicad_pcb (KiCad board)
At the start: 2 copper layers, 73 x 79 mm, 150 parts, among them P1 CONN_01X02, P10 CONN_01X02, P12 CONN_01X02, P13 CONN_01X06, P16 CONN_01X04, P17 CONN_01X04, P2 CONN_01X02, P3 CONN_01X04, P4 CONN_01X04, P6 CONN_01X04, P7 CONN_01X02, P8 CONN_01X04, Q1 MOSFET_N, Q2 MOSFET_N, Q3 MOSFET_N, Q4 MOSFET_N, Q5 MOSFET_N, Q6 MOSFET_N, Q7 MOSFET_N, Q8 MOSFET_N, SW1 SW_PUSH, SW2 SW_PUSH, SW3 SW_PUSH, U1 STM32F103_48, U10 NCP1117ST33T3G, U11 LM1084IS-3.3/NOPB, U2 SI8234, U3 SI8234, U4 LM7812, U5 SI8234, U6 SI8234, U7 7805, U8 MAX3051, U9 SW_ROTARY_16, X2 CRYSTAL

Commit message: 発注した｡古い基板プロジェクトの移動
Parts:
- R21, R22, R23, R24, R25, R26, R27, R28: value 10 -> 1
Routing:
- net +BATT: track 175.2 -> 191.6 mm, vias 76 -> 85
- net (no net): track 9.00 -> 0.00 mm, vias 11 -> 4
Changed lines of the file:
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@@
     (links 342)
     (no_connects 0)
-    (area -0.075001 -0.075001 73.075001 79.075001)
+    (area -4.575 -1.200001 74.82442 80.200002)
     (thickness 1.6)
     (drawings 33)
-    (tracks 1634)
+    (tracks 1640)
     (zones 0)
     (modules 150)
@@
       (effects (font (size 1.2065 1.2065) (thickness 0.1016)) (justify left bottom))
     )
-    (fp_text value FILTER (at 2 -2 90) (layer F.SilkS)
+    (fp_text value FILTER (at -1 2.5 90) (layer F.SilkS)
       (effects (font (size 1.2065 1.2065) (thickness 0.1016)) (justify left bottom))
     )
@@
       (effects (font (size 1.2065 1.2065) (thickness 0.1016)) (justify left bottom))
     )
-    (fp_text value FILTER (at 2 -2 90) (layer F.SilkS)
+    (fp_text value FILTER (at -4.5 2 90) (layer F.SilkS)
       (effects (font (size 1.2065 1.2065) (thickness 0.1016)) (justify left bottom))
     )
@@
       (effects (font (size 1.2065 1.2065) (thickness 0.1016)) (justify left bottom))
     )
-    (fp_text value FILTER (at 2 -2 270) (layer F.SilkS)
+    (fp_text value FILTER (at -1.5 2.5 270) (layer F.SilkS)
       (effects (font (size 1.2065 1.2065) (thickness 0.1016)) (justify left bottom))
     )
@@
       (effects (font (size 1.2065 1.2065) (thickness 0.1016)) (justify left bottom))
     )
-    (fp_text value FILTER (at 2 -2 90) (layer F.SilkS)
+    (fp_text value FILTER (at -4.5 2.5 90) (layer F.SilkS)
       (effects (font (size 1.2065 1.2065) (thickness 0.1016)) (justify left bottom))
     )
@@
       (effects (font (size 1.2065 1.2065) (thickness 0.1016)) (justify left bottom))
     )
-    (fp_text value 10 (at -1 -0.5 180) (layer F.SilkS)
+    (fp_text value 1 (at -0.5 -0.5 180) (layer F.SilkS)
       (effects (font (size 1.2065 1.2065) (thickness 0.1016)) (justify left bottom))
     )
@@
       (effects (font (size 1.2065 1.2065) (thickness 0.1016)) (justify left bottom))
     )
-    (fp_text value 10 (at -1 -0.5 180) (layer F.SilkS)
+    (fp_text value 1 (at -0.5 -0.5 180) (layer F.SilkS)
       (effects (font (size 1.2065 1.2065) (thickness 0.1016)) (justify left bottom))
     )
@@
       (effects (font (size 1.2065 1.2065) (thickness 0.1016)) (justify left bottom))
     )
-    (fp_text value 10 (at -1 -0.5) (layer F.SilkS)
+    (fp_text value 1 (at -0.5 -0.5) (layer F.SilkS)
       (effects (font (size 1.2065 1.2065) (thickness 0.1016)) (justify left bottom))
     )
@@
       (effects (font (size 1.2065 1.2065) (thickness 0.1016)) (justify left bottom))
     )
-    (fp_text value 10 (at -1 -0.5) (layer F.SilkS)
+    (fp_text value 1 (at -0.5 -0.5) (layer F.SilkS)
       (effects (font (size 1.2065 1.2065) (thickness 0.1016)) (justify left bottom))
     )
@@
       (effects (font (size 1.2065 1.2065) (thickness 0.1016)) (justify left bottom))
     )
-    (fp_text value 10 (at -1 -0.5) (layer F.SilkS)
+    (fp_text value 1 (at -0.5 -0.5) (layer F.SilkS)
       (effects (font (size 1.2065 1.2065) (thickness 0.1016)) (justify left bottom))
     )
@@
       (effects (font (size 1.2065 1.2065) (thickness 0.1016)) (justify left bottom))
     )
-    (fp_text value 10 (at -1 -0.5) (layer F.SilkS)
+    (fp_text value 1 (at -0.5 -0.5) (layer F.SilkS)
       (effects (font (size 1.2065 1.2065) (thickness 0.1016)) (justify left bottom))
     )
@@
       (effects (font (size 1.2065 1.2065) (thickness 0.1016)) (justify left bottom))
     )
-    (fp_text value 10 (at -1 -0.5) (layer F.SilkS)
+    (fp_text value 1 (at -0.5 -0.5) (layer F.SilkS)
       (effects (font (size 1.2065 1.2065) (thickness 0.1016)) (justify left bottom))
     )
@@
       (effects (font (size 1.2065 1.2065) (thickness 0.1016)) (justify left bottom))
     )
-    (fp_text value 10 (at -1 -0.5) (layer F.SilkS)
+    (fp_text value 1 (at -0.5 -0.5) (layer F.SilkS)
       (effects (font (size 1.2065 1.2065) (thickness 0.1016)) (justify left bottom))
     )
@@
   (via (at 70 3) (size 4) (drill 3) (layers F.Cu B.Cu) (net 0))
   (via (at 3 3) (size 4) (drill 3) (layers F.Cu B.Cu) (net 0))
-  (segment (start 9 16) (end 9 17.5) (width 0.5) (layer F.Cu) (net 0))
-  (via (at 9 17.5) (size 1.5) (drill 0.75) (layers F.Cu B.Cu) (net 0))
-  (segment (start 9 17.5) (end 9 19) (width 0.5) (layer B.Cu) (net 0))
-  (via (at 9 19) (size 1.5) (drill 0.75) (layers F.Cu B.Cu) (net 0))
-  (segment (start 9 19) (end 9 20.5) (width 0.5) (layer F.Cu) (net 0))
-  (via (at 9 20.5) (size 1.5) (drill 0.75) (layers F.Cu B.Cu) (net 0))
-  (segment (start 9 20.5) (end 9 22) (width 0.5) (layer B.Cu) (net 0))
-  (via (at 9 22) (size 1.5) (drill 0.75) (layers F.Cu B.Cu) (net 0))
-  (segment (start 9 22) (end 9 23.5) (width 0.5) (layer F.Cu) (net 0))
-  (via (at 9 23.5) (size 1.5) (drill 0.75) (layers F.Cu B.Cu) (net 0))
-  (via (at 9 16) (size 1.5) (drill 0.75) (layers F.Cu B.Cu) (net 0))
-  (segment (start 9 16) (end 10.5 16) (width 0.5) (layer B.Cu) (net 0))
-  (via (at 10.5 16) (size 1.5) (drill 0.75) (layers F.Cu B.Cu) (net 0))
-  (segment (start 62.5 43.6) (end 62.6 43.5) (width 0.25) (layer B.Cu) (net 1) (status C00000))
-  (segment (start 62.6 43.5) (end 71.5 43.5) (width 0.25) (layer B.Cu) (net 1) (status 400000))
+  (segment (start 62.5 43.6) (end 62.6 43.5) (width 0.25) (layer B.Cu) (net 1))
+  (segment (start 62.6 43.5) (end 71.5 43.5) (width 0.25) (layer B.Cu) (net 1))
   (via (at 71.5 43.5) (size 0.5) (drill 0.3) (layers F.Cu B.Cu) (net 1))
-  (segment (start 61.5 43.5) (end 62.5 43.5) (width 0.25) (layer B.Cu) (net 1) (status 800000))
-  (segment (start 62.5 43.5) (end 62.5 43.6) (width 0.25) (layer B.Cu) (net 1) (status C00000))
+  (segment (start 61.5 43.5) (end 62.5 43.5) (width 0.25) (layer B.Cu) (net 1))
+  (segment (start 62.5 43.5) (end 62.5 43.6) (width 0.25) (layer B.Cu) (net 1))
   (segment (start 60 43.5) (end 61.5 43.5) (width 0.25) (layer B.Cu) (net 1))
   (via (at 61.5 43.5) (size 0.5) (drill 0.3) (layers F.Cu B.Cu) (net 1))
@@
   (segment (start 39.46 18) (end 39.46 16.54) (width 0.5) (layer B.Cu) (net 13))
   (segment (start 41 35.1) (end 40.6 35.5) (width 0.5) (layer F.Cu) (net 13))
+  (segment (start 9 23.5) (end 9 25) (width 0.25) (layer B.Cu) (net 14))
+  (via (at 9 17.5) (size 1.5) (drill 0.75) (layers F.Cu B.Cu) (net 14))
+  (segment (start 9 17.5) (end 9 19) (width 0.25) (layer B.Cu) (net 14))
+  (via (at 9 19) (size 1.5) (drill 0.75) (layers F.Cu B.Cu) (net 14))
+  (segment (start 9 19) (end 9 20.5) (width 0.25) (layer F.Cu) (net 14))
+  (via (at 9 20.5) (size 1.5) (drill 0.75) (layers F.Cu B.Cu) (net 14))
+  (segment (start 9 20.5) (end 9 22) (width 0.25) (layer B.Cu) (net 14))
+  (via (at 9 22) (size 1.5) (drill 0.75) (layers F.Cu B.Cu) (net 14))
+  (segment (start 9 22) (end 9 23.5) (width 0.25) (layer F.Cu) (net 14))
+  (via (at 9 23.5) (size 1.5) (drill 0.75) (layers F.Cu B.Cu) (net 14))
+  (segment (start 9 16) (end 9 17.5) (width 0.25) (layer F.Cu) (net 14))
+  (via (at 10.5 25) (size 1.5) (drill 0.75) (layers F.Cu B.Cu) (net 14))
+  (segment (start 9 25) (end 10.5 25) (width 0.25) (layer F.Cu) (net 14))
+  (via (at 9 25) (size 1.5) (drill 0.75) (layers F.Cu B.Cu) (net 14))
+  (segment (start 9.8 12) (end 9.8 15.2) (width 0.25) (layer F.Cu) (net 14))
+  (segment (start 9.8 15.2) (end 9 16) (width 0.25) (layer F.Cu) (net 14))
+  (via (at 9 16) (size 1.5) (drill 0.75) (layers F.Cu B.Cu) (net 14))
+  (segment (start 9 16) (end 10.5 16) (width 0.25) (layer B.Cu) (net 14))
+  (via (at 10.5 16) (size 1.5) (drill 0.75) (layers F.Cu B.Cu) (net 14))
   (segment (start 9 5.5) (end 9 7) (width 0.5) (layer F.Cu) (net 14))
   (via (at 9 7) (size 1.5) (drill 0.75) (layers F.Cu B.Cu) (net 14))
@@
   (segment (start 62.825 34.825) (end 62.825 35.85) (width 0.5) (layer F.Cu) (net 92))
   (segment (start 62 34) (end 62.825 34.825) (width 0.5) (layer F.Cu) (net 92))
-  (segment (start 49.631371 61.520458) (end 49 60.889087) (width 0.25) (layer F.Cu) (net 93) (status 400000))
+  (segment (start 49.631371 61.520458) (end 49 60.889087) (width 0.25) (layer F.Cu) (net 93))
   (segment (start 49 60.889087) (end 49 58.5) (width 0.25) (layer F.Cu) (net 93))
   (segment (start 49 58.5) (end 49.5 58) (width 0.25) (layer F.Cu) (net 93))
@@
   (segment (start 65 46.25) (end 65.365 45.885) (width 0.3) (layer F.Cu) (net 93))
   (segment (start 65.365 45.15) (end 65.365 45.885) (width 0.3) (layer F.Cu) (net 93))
-  (segment (start 47.368629 61.520458) (end 48 60.889087) (width 0.25) (layer F.Cu) (net 94) (status 400000))
+  (segment (start 47.368629 61.520458) (end 48 60.889087) (width 0.25) (layer F.Cu) (net 94))
   (segment (start 48 60.889087) (end 48 60.5) (width 0.25) (layer F.Cu) (net 94))
   (via (at 48 60.5) (size 0.5) (drill 0.3) (layers F.Cu B.Cu) (net 94))
