File: KiCAD_Projects/ISO_DCDC_ver1.2/ISO_DCDC_ver1.2.kicad_pcb (KiCad board)
At the start: 2 copper layers, 90 x 77 mm, 51 parts, among them IC4 PC817, IC5 PC817, P1 CONN_01X01, P10 CONN_01X02, P12 CONN_01X01, P13 CONN_01X04, P14 CONN_01X02, P15 CONN_01X02, P2 CONN_01X01, P21 CONN_01X02, P22 CONN_01X01, P23 CONN_01X01, P25 CONN_01X01, P26 CONN_01X01, P3 CONN_01X01, P4 CONN_01X02, P5 CONN_01X02, P6 CONN_01X02, P8 CONN_01X01, Q1 MOSFET_N, U1 V23076-D3001-D142, U2 7805, U3 V23076-D3001-D142

Commit message: 発注した｡
Parts:
- P4, P5: footprint RP_KiCAD_Connector:XA_2LC -> RP_KiCAD_Connector:XA_2T
- moved R11 56.3 mm to (20.0, 16.5), turned to 90 degrees
- moved R19 55.3 mm to (-0.50, -6.00)
- moved D4 53.4 mm to (36.0, 54.5)
- moved Q1 51.3 mm to (22.5, 19.0), turned to 0 degrees
- moved P6 41.6 mm to (-14.5, 7.00)
- moved D13 37.9 mm to (26.0, -7.50)
- moved C1 35.7 mm to (41.5, 41.5), turned to 270 degrees
- moved C10 29.9 mm to (67.5, 41.0), turned to 180 degrees
- moved P14 28.9 mm to (-10.5, 17.5)
- moved D5 26.2 mm to (54.5, 34.5), turned to 90 degrees
- moved R15 22.7 mm to (56.0, 26.5)
- moved R22 22.7 mm to (56.0, 29.0)
- moved R14 21.8 mm to (56.5, 24.5)
- moved R8 19.1 mm to (56.5, 33.5), turned to 270 degrees
- moved P5 14.2 mm to (3.00, 19.0)
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Routing:
- net /POWER_EN_HIGH: track 0.00 -> 71.3 mm
- net /POWER_EN_LOW: track 0.00 -> 40.7 mm
- net /15V: track 0.00 -> 37.6 mm
- net /12V: track 0.00 -> 24.1 mm
- net GND: track 0.00 -> 21.0 mm
- net Net-(P21-Pad1): track 0.00 -> 11.7 mm
- net Net-(IC5-Pad4): track 0.00 -> 5.41 mm
- net GNDPWR: track 0.00 -> 4.69 mm
- net Net-(IC4-Pad1): track 0.00 -> 3.41 mm
- net Net-(P13-Pad4): track 0.00 -> 3.00 mm
- net Net-(P13-Pad3): track 0.00 -> 3.00 mm
- net Net-(D5-Pad2): track 0.00 -> 2.22 mm
- net Net-(IC4-Pad3): track 0.00 -> 2.10 mm
Other:
- board size 90 x 77 mm -> 90 x 74 mm
- board text removed: "EXTERNAL POWER IN"

Commit message: ISO_DCDC_ver1.2の設計終わり｡加工依頼用データだし｡
Parts:
- removed C1, C2: 1000u, Capacitors_ThroughHole:C_Radial_D8_L11.5_P3.5
- removed D13: LED, LEDs:LED-3MM
- removed P15: CONN_01X02, RP_KiCAD_Connector:XA_2T
- removed R9: 1k, RP_KiCAD_Libs:C1608_NP
- removed U2: 7805, TO_SOT_Packages_SMD:TO-252-2Lead_regu
- added D2: DIODE, RP_KiCAD_Libs:C3216, B.Cu at (20.0, 47.0)
- added P7: CONN_01X02, RP_KiCAD_Connector:XA_2T, F.Cu at (57.5, 31.5)
- added R2: R, Resistors_SMD:R_2812, B.Cu at (23.5, 26.5)
- added R3: R, Resistors_SMD:R_2812, B.Cu at (23.5, 17.0)
- added R4: R, Resistors_SMD:R_2812, B.Cu at (23.5, 45.5)
- added R5: R, Resistors_SMD:R_2812, B.Cu at (23.5, 36.0)
- C10: footprint Capacitors_ThroughHole:C_Radial_D8_L11.5_P3.5 -> Capacitors_ThroughHole:C_Radial_D10_L20_P5
- R13, R19: footprint RP_KiCAD_Libs:0204_2f7 -> RP_KiCAD_Libs:C1608_NP; moved to B.Cu
- moved P14 62.7 mm to (50.5, 3.00)
- moved P6 56.1 mm to (41.5, 3.00)
- moved D4 54.8 mm to (48.0, 1.00), turned to 0 degrees
- moved D1 51.2 mm to (30.0, 4.00), turned to 180 degrees
- moved P21 49.8 mm to (23.0, 1.50), turned to 90 degrees
- moved R1 49.0 mm to (23.0, 5.00)
- moved P10 34.4 mm to (57.5, 24.0)
- moved R19 30.4 mm to (29.0, 1.50), turned to 180 degrees
- moved D3 29.4 mm to (32.5, 15.5)
- moved C6 27.4 mm to (35.5, 29.0), turned to 0 degrees
- moved D5 21.7 mm to (46.0, 14.5), turned to 270 degrees
- moved C10 20.4 mm to (51.0, 29.0)
- moved R11 19.5 mm to (39.5, 16.5), turned to 270 degrees
- moved P13 19.5 mm to (51.5, 16.5)
- moved R8 19.5 mm to (48.0, 16.0), turned to 90 degrees
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Connections:
- C6 pad 1: Net-(C1-Pad1) -> /15V
- D1 pad 1: /15V -> /POWER_EN_LOW
- D4 pad 1: Net-(C1-Pad1) -> /15V
- D7 pad 1: /15V -> Net-(D7-Pad1)
- D7 pad 2: /POWER_EN_LOW -> Net-(D7-Pad2)
- DCDC3 pad 6: Net-(C1-Pad1) -> /15V
- P6 pad 2: Net-(C1-Pad1) -> /15V
- R1 pad 2: GNDPWR -> /15V
- U1 pad 1: /POWER_EN_LOW -> Net-(D2-Pad2)
- U1 pad 2: /POWER_EN_HIGH -> Net-(D2-Pad1)
- U3 pad 1: /POWER_EN_LOW -> Net-(D7-Pad2)
- U3 pad 2: /POWER_EN_HIGH -> Net-(D7-Pad1)
Routing:
- net GNDPWR: track 4.69 -> 194.1 mm
- net GND: track 21.0 -> 75.0 mm
- net /12V: track 24.1 -> 77.9 mm
- net /15V: track 37.6 -> 89.8 mm
- net /POWER_EN_LOW: track 40.7 -> 66.5 mm
- net Net-(IC4-Pad4): track 0.00 -> 17.6 mm, vias 0 -> 2
- net Net-(D3-Pad1): track 0.00 -> 15.8 mm
- net Net-(D7-Pad1): track 0.00 -> 13.2 mm
- net Net-(D2-Pad2): track 0.00 -> 11.3 mm
- net Net-(IC5-Pad1): track 0.00 -> 10.5 mm, vias 0 -> 2
- net +BATT: track 0.00 -> 9.95 mm
- net /POWER_EN_HIGH: track 71.3 -> 61.5 mm
- net Net-(D7-Pad2): track 0.00 -> 8.56 mm
- net Net-(IC4-Pad3): track 2.10 -> 10.0 mm
- net Net-(P21-Pad1): track 11.7 -> 19.5 mm
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- added copper zone on B.Cu, net GND
Other:
- board size 90 x 74 mm -> 60 x 60 mm

Commit message: 電源基板ver1.2加工した｡次ver1.3作るべきかも
Parts:
- removed D4: DIODE, RP_KiCAD_Libs:C3216
- removed P14: CONN_01X02, RP_KiCAD_Connector:XA_2T
- IC4, IC5: footprint Housings_SOIC:SOIJ-4_5.3x5.3mm_Pitch1.27mm -> Housings_DIP:DIP-4_W7.62mm_LongPads_Slim; moved to F.Cu
- moved D5 8.32 mm to (50.5, 21.5), turned to 0 degrees
- moved IC4 8.08 mm to (45.5, 19.5)
- moved R1 6.71 mm to (29.0, 8.00)
- moved IC5 4.53 mm to (38.0, 9.00)
- moved P21 3.00 mm to (23.0, 4.50), turned to 180 degrees
- moved R11 2.92 mm to (38.0, 14.0), turned to 90 degrees
- moved Q1 2.50 mm to (35.0, 20.5)
- moved D1 2.06 mm to (28.0, 4.50), turned to 0 degrees
- moved R19 1.00 mm to (29.0, 2.50)
- moved D10 0.71 mm to (7.50, 30.5)
- moved D8 0.71 mm to (7.50, 24.0)
- moved D9 0.71 mm to (7.50, 46.0)
- moved C10 0.50 mm to (50.5, 29.0)
- moved D12 0.50 mm to (10.0, 10.0)
- moved D2 0.50 mm to (20.0, 47.5)
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Connections:
- D1 pad 1: /POWER_EN_LOW -> /15V
- R1 pad 2: /15V -> /POWER_EN_LOW
Routing:
- net GNDPWR: track 194.1 -> 163.3 mm
- net /12V: track 77.9 -> 107.3 mm
- net GND: track 75.0 -> 59.4 mm
- net Net-(IC4-Pad1): track 1.91 -> 14.3 mm
- net Net-(IC4-Pad4): track 17.6 -> 26.4 mm
- net Net-(D5-Pad2): track 2.02 -> 9.49 mm
- net /POWER_EN_LOW: track 66.5 -> 59.8 mm
- net Net-(D1-Pad2): track 3.87 -> 8.37 mm
- net Net-(IC4-Pad3): track 10.0 -> 7.15 mm
- net Net-(D4-Pad2): track 2.37 -> 0.00 mm
- net /15V: track 89.8 -> 88.0 mm
- net Net-(IC5-Pad1): track 10.5 -> 9.04 mm
- net Net-(D3-Pad1): track 15.8 -> 16.9 mm
- net Net-(P21-Pad1): track 19.5 -> 18.6 mm
- net +BATT: track 9.95 -> 9.25 mm
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