File: KiCAD_Projects/ISO_DCDC_ver1.2/ISO_DCDC_ver1.2.sch (KiCad schematic (older format))
At the start: 51 parts, among them IC4 PC817, IC5 PC817, P1 CONN_01X01, P10 CONN_01X02, P12 CONN_01X01, P13 CONN_01X04, P14 CONN_01X02, P15 CONN_01X02, P2 CONN_01X01, P21 CONN_01X02, P22 CONN_01X01, P23 CONN_01X01, P25 CONN_01X01, P26 CONN_01X01, P3 CONN_01X01, P4 CONN_01X02, P5 CONN_01X02, P6 CONN_01X02, P8 CONN_01X01, Q1 MOSFET_N, U1 V23076-D3001-D142, U2 7805, U3 V23076-D3001-D142

Commit message: 発注した｡
Parts:
- P4, P5: footprint RP_KiCAD_Connector:XA_2LC -> RP_KiCAD_Connector:XA_2T
Changed lines of the file:
@@
 F 0 "P5" H 4400 5900 50  0000 C CNN
 F 1 "CONN_01X02" V 4500 5750 50  0000 C CNN
-F 2 "RP_KiCAD_Connector:XA_2LC" H 4400 5750 50  0001 C CNN
+F 2 "RP_KiCAD_Connector:XA_2T" H 4400 5750 50  0001 C CNN
 F 3 "" H 4400 5750 50  0000 C CNN
 	1    4400 5750
@@
 F 0 "P4" H 4400 5400 50  0000 C CNN
 F 1 "CONN_01X02" V 4500 5250 50  0000 C CNN
-F 2 "RP_KiCAD_Connector:XA_2LC" H 4400 5250 50  0001 C CNN
+F 2 "RP_KiCAD_Connector:XA_2T" H 4400 5250 50  0001 C CNN
 F 3 "" H 4400 5250 50  0000 C CNN
 	1    4400 5250

Commit message: ISO_DCDC_ver1.2の設計終わり｡加工依頼用データだし｡
Parts:
- removed C1, C2: 1000u, Capacitors_ThroughHole:C_Radial_D8_L11.5_P3.5, symbol C
- removed D13: LED, LEDs:LED-3MM, symbol LED
- removed P15: CONN_01X02, RP_KiCAD_Connector:XA_2T, symbol CONN_01X02
- removed R9: 1k, RP_KiCAD_Libs:C1608_NP, symbol R
- removed U2: 7805, TO_SOT_Packages_SMD:TO-252-2Lead_regu, symbol 7805
- added D2: DIODE, RP_KiCAD_Libs:C3216, symbol DIODE
- added P7: CONN_01X02, RP_KiCAD_Connector:XA_2T, symbol CONN_01X02
- added R2, R3, R4, R5: R, Resistors_SMD:R_2812, symbol R
- C10: footprint Capacitors_ThroughHole:C_Radial_D8_L11.5_P3.5 -> Capacitors_ThroughHole:C_Radial_D10_L20_P5
- R13, R19: footprint RP_KiCAD_Libs:0204_2f7 -> RP_KiCAD_Libs:C1608_NP
Connections:
- net 12V: now also P7.2 (P2)
- net 15V: now also C6.1, D4.1 (K), DCDC3.6 (+Vin), P6.2 (P2), R1.2; no longer D1.1 (A), D7.1 (K)
- net GND: now also P7.1 (P1)
- net GNDPWR: no longer R1.2
- net POWER_EN_HIGH: now also R3.1, R5.1; no longer U1.2 (A2), U3.2 (A2)
- net POWER_EN_LOW: now also D1.1 (A), R2.1, R4.1; no longer D7.2 (A), U1.1 (A1), U3.1 (A1)
- new net: D7.2 (A), R3.2, U3.1 (A1)
- new net: D7.1 (K), R2.2, U3.2 (A2)
- new net: D2.2 (A), R5.2, U1.1 (A1)
- new net: D2.1 (K), R4.2, U1.2 (A2)
Other:
- moved on the sheet: C10, C6, D10, D12, D3, D4, D5, D7, D8, D9, DCDC3, IC4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

Commit message: 電源基板ver1.2加工した｡次ver1.3作るべきかも
Parts:
- removed D4: DIODE, RP_KiCAD_Libs:C3216, symbol DIODE
- removed P14: CONN_01X02, RP_KiCAD_Connector:XA_2T, symbol CONN_01X02
- IC4, IC5: footprint Housings_SOIC:SOIJ-4_5.3x5.3mm_Pitch1.27mm -> Housings_DIP:DIP-4_W7.62mm_LongPads_Slim
Connections:
- net 15V: now also D1.1 (A); no longer R1.2
- net POWER_EN_LOW: now also R1.2; no longer D1.1 (A)
Changed lines of the file:
@@
 F 0 "IC4" H 8987 6278 40  0000 C CNN
 F 1 "PC817" H 9350 5915 40  0000 C CNN
-F 2 "Housings_SOIC:SOIJ-4_5.3x5.3mm_Pitch1.27mm" H 9036 5925 29  0000 C CNN
+F 2 "Housings_DIP:DIP-4_W7.62mm_LongPads_Slim" H 9036 5925 29  0000 C CNN
 F 3 "" H 9200 6100 60  0000 C CNN
 	1    9200 6100
@@
 F 0 "IC5" H 9037 7178 40  0000 C CNN
 F 1 "PC817" H 9400 6815 40  0000 C CNN
-F 2 "Housings_SOIC:SOIJ-4_5.3x5.3mm_Pitch1.27mm" H 9086 6825 29  0000 C CNN
+F 2 "Housings_DIP:DIP-4_W7.62mm_LongPads_Slim" H 9086 6825 29  0000 C CNN
 F 3 "" H 9250 7000 60  0000 C CNN
 	1    9250 7000
@@
 Text Label 11600 7700 0    60   ~ 0
 12V
-$Comp
-L CONN_01X02 P14
-U 1 1 58CAAA00
-P 6950 3700
-F 0 "P14" H 6950 3850 50  0000 C CNN
-F 1 "CONN_01X02" V 7050 3700 50  0000 C CNN
-F 2 "RP_KiCAD_Connector:XA_2T" H 6950 3700 50  0001 C CNN
-F 3 "" H 6950 3700 50  0000 C CNN
-	1    6950 3700
-	-1   0    0    1
-$EndComp
+Wire Wire Line
+	7650 3650 7600 3650
 $Comp
 L GNDPWR #PWR024
-U 1 1 58CAB745
-P 7150 3750
-F 0 "#PWR024" H 7150 3800 40  0001 C CNN
-F 1 "GNDPWR" H 7150 3670 40  0000 C CNN
-F 2 "" H 7150 3750 60  0001 C CNN
-F 3 "" H 7150 3750 60  0001 C CNN
-	1    7150 3750
-	0    -1   -1   0
-$EndComp
-$Comp
-L DIODE D4
-U 1 1 58CABAEE
-P 7400 3650
-F 0 "D4" H 7400 3750 40  0000 C CNN
-F 1 "DIODE" H 7400 3550 40  0000 C CNN
-F 2 "RP_KiCAD_Libs:C3216" H 7400 3650 60  0001 C CNN
-F 3 "" H 7400 3650 60  0000 C CNN
-	1    7400 3650
-	1    0    0    -1
-$EndComp
-Wire Wire Line
-	7650 3650 7600 3650
-Wire Wire Line
-	7200 3650 7150 3650
-$Comp
-L GNDPWR #PWR025
 U 1 1 58DA68D2
 P 2150 7200
-F 0 "#PWR025" H 2150 7250 40  0001 C CNN
+F 0 "#PWR024" H 2150 7250 40  0001 C CNN
 F 1 "GNDPWR" H 2150 7150 40  0000 C CNN
 F 2 "" H 2150 7200 60  0001 C CNN
@@
 $EndComp
 $Comp
-L GND #PWR026
+L GND #PWR025
 U 1 1 5909E685
 P 12000 3600
-F 0 "#PWR026" H 12000 3600 30  0001 C CNN
+F 0 "#PWR025" H 12000 3600 30  0001 C CNN
 F 1 "GND" H 12000 3530 30  0001 C CNN
 F 2 "" H 12000 3600 60  0001 C CNN
@@
 	1    0    0    -1
 $EndComp
+Text Label 5350 9800 0    60   ~ 0
+POWER_EN_LOW
+Wire Wire Line
+	5350 9800 5350 9700
 Text Label 5350 9000 0    60   ~ 0
-POWER_EN_LOW
-Wire Wire Line
-	5350 9800 5350 9700
-Text Label 5350 9800 0    60   ~ 0
 15V
 $EndSCHEMATC
