File: KiCAD_Projects/KawaRoboMain/KawaRoboMain.kicad_pcb (KiCad board)
At the start: 2 copper layers, 0 parts

Commit message: Morex系ゴニョゴニョした
Parts:
- added C1: 0.1u, RP_KiCAD_Libs:C1608_WP, F.Cu at (37.5, 23.0)
- added C10: 0.1u, RP_KiCAD_Libs:C1608_WP, F.Cu at (16.5, 36.0)
- added C11: 4.7u, RP_KiCAD_Libs:C3216, F.Cu at (46.5, 16.0)
- added C12: 4.7u, RP_KiCAD_Libs:C3216, F.Cu at (48.5, 80.0)
- added C13: 4.7u, RP_KiCAD_Libs:C3216, F.Cu at (52.0, 24.0)
- added C14: 4.7u, RP_KiCAD_Libs:C3216, F.Cu at (46.5, 24.0)
- added C15: 4.7u, RP_KiCAD_Libs:C3216, F.Cu at (52.0, 32.0)
- added C16: 4.7u, RP_KiCAD_Libs:C3216, F.Cu at (52.0, 40.0)
- added C17: 4.7u, RP_KiCAD_Libs:C3216, F.Cu at (52.0, 48.0)
- added C18: 4.7u, RP_KiCAD_Libs:C3216, F.Cu at (52.0, 56.0)
- added C19: 4.7u, RP_KiCAD_Libs:C3216, F.Cu at (46.5, 32.0)
- added C2: 4.7u, RP_KiCAD_Libs:C3216, F.Cu at (26.5, 7.00)
- added C20: 4.7u, RP_KiCAD_Libs:C3216, F.Cu at (46.5, 40.0)
- added C21: 4.7u, RP_KiCAD_Libs:C3216, F.Cu at (46.5, 48.0)
- added C22: 4.7u, RP_KiCAD_Libs:C3216, F.Cu at (46.5, 56.0)
- added C23: 4.7u, RP_KiCAD_Libs:C3216, F.Cu at (52.0, 64.0)
- added C24: 4.7u, RP_KiCAD_Libs:C3216, F.Cu at (52.0, 72.0)
- added C25: 4.7u, RP_KiCAD_Libs:C3216, F.Cu at (46.5, 64.0)
- added C26: 4.7u, RP_KiCAD_Libs:C3216, F.Cu at (46.5, 72.0)
- added C27: 22p, RP_KiCAD_Libs:C1608_WP, F.Cu at (28.5, 91.0)
- added C28: 22p, RP_KiCAD_Libs:C1608_WP, F.Cu at (28.5, 78.0)
- added C29: 0.1u, RP_KiCAD_Libs:C1608_WP, F.Cu at (39.5, 79.5)
- added C3: 0.1u, RP_KiCAD_Libs:C1608_WP, F.Cu at (37.0, 58.0)
- added C30: 220u, Capacitors_ThroughHole:C_Radial_D10_L13_P5, F.Cu at (67.0, 84.0)
- added C31: 220u, Capacitors_ThroughHole:C_Radial_D10_L13_P5, F.Cu at (46.0, 7.00)
- added C32: 220u, Capacitors_ThroughHole:C_Radial_D10_L13_P5, F.Cu at (46.0, 84.0)
- added C33: 220u, Capacitors_ThroughHole:C_Radial_D10_L13_P5, F.Cu at (56.5, 84.0)
- added C34: 220u, Capacitors_ThroughHole:C_Radial_D10_L13_P5, F.Cu at (56.5, 7.00)
- added C35: 220u, Capacitors_ThroughHole:C_Radial_D10_L13_P5, F.Cu at (67.0, 7.00)
- added C36: 4.7u, RP_KiCAD_Libs:C3216, F.Cu at (32.0, 7.00)
- added C37: 4.7u, RP_KiCAD_Libs:C3216, F.Cu at (32.0, 17.0)
- added C38: 0.1u, RP_KiCAD_Libs:C1608_WP, F.Cu at (37.0, 41.5)
- added C39: 2.2u, RP_KiCAD_Libs:C2012, F.Cu at (-12.5, 15.5)
- added C4: 22p, RP_KiCAD_Libs:C1608_WP, F.Cu at (23.5, 21.5)
- added C40: 2.2u, RP_KiCAD_Libs:C2012, F.Cu at (-12.5, 7.50)
- added C41: 0.1u, RP_KiCAD_Libs:C1608_WP, F.Cu at (13.0, 52.0)
- added C42: 0.1u, RP_KiCAD_Libs:C1608_WP, F.Cu at (30.5, 74.0)
- added C43: 0.1u, RP_KiCAD_Libs:C1608_WP, F.Cu at (19.5, 69.0)
- added C5: 22p, RP_KiCAD_Libs:C1608_WP, F.Cu at (19.5, 21.5)
- added C6: 0.1u, RP_KiCAD_Libs:C1608_WP, F.Cu at (9.50, 14.5)
- added C7: 4.7u, RP_KiCAD_Libs:C3216, F.Cu at (26.5, 17.0)
- added C8: 0.1u, RP_KiCAD_Libs:C1608_WP, F.Cu at (26.5, 26.0)
- added C9: 0.1u, RP_KiCAD_Libs:C1608_WP, F.Cu at (26.5, 36.0)
- added D1: LED, LEDs:LED_0805, F.Cu at (26.5, 22.5)
- added D10: DIODE, RP_KiCAD_Libs:C2012, F.Cu at (43.0, 72.0)
- added D11: LED, LEDs:LED_0805, F.Cu at (32.5, 22.5)
- added D12: LED, LEDs:LED_0805, F.Cu at (29.5, 22.5)
- added D13: LED, LEDs:LED_0805, F.Cu at (27.3, 69.2)
- added D14: LED, LEDs:LED_0805, F.Cu at (27.3, 66.7)
- added D15: DIODE, Diodes_SMD:SOD-123, F.Cu at (38.5, 8.00)
- added D2: LED, LEDs:LED_0805, F.Cu at (35.5, 22.5)
- added D3: DIODE, RP_KiCAD_Libs:C2012, F.Cu at (43.0, 16.0)
- added D4: DIODE, RP_KiCAD_Libs:C2012, F.Cu at (43.0, 24.0)
- added D5: DIODE, RP_KiCAD_Libs:C2012, F.Cu at (43.0, 32.0)
- added D6: DIODE, RP_KiCAD_Libs:C2012, F.Cu at (43.0, 40.0)
- added D7: DIODE, RP_KiCAD_Libs:C2012, F.Cu at (43.0, 48.0)
- added D8: DIODE, RP_KiCAD_Libs:C2012, F.Cu at (43.0, 56.0)
- added D9: DIODE, RP_KiCAD_Libs:C2012, F.Cu at (43.0, 64.0)
- added IC1: ATMEGA328P-A, Housings_QFP:TQFP-32_7x7mm_Pitch0.8mm, F.Cu at (15.9, 81.3)
- added IC2: SP3485CN, Housings_SOIC:SOIC-8_3.9x4.9mm_Pitch1.27mm, F.Cu at (9.50, 18.0)
- added JP1: JUMPER, Connect:GS2, B.Cu at (36.0, 87.5)
- added JP2: JUMPER3, Connect:GS3, B.Cu at (13.5, 84.5)
- added JP3: JUMPER, Connect:GS2, B.Cu at (11.4, 94.6)
- added JP4: JUMPER3, Connect:GS3, B.Cu at (-12.0, 6.50)
- added ME1: AS504x, Housings_SSOP:SSOP-16_3.9x4.9mm_Pitch0.635mm, B.Cu at (-13.0, 11.0)
- added P1: CONN_01X06, RP_KiCAD_Connector:XA_6T, F.Cu at (3.00, 33.5)
- added P10: CONN_01X02, RP_KiCAD_Connector:XA_2T, F.Cu at (3.00, 2.50)
- added P11: CONN_01X12, Pin_Headers:Pin_Header_Straight_1x12, F.Cu at (23.5, 66.7)
- added P12: CONN_01X12, Pin_Headers:Pin_Header_Straight_1x12, F.Cu at (8.27, 94.6)
- added P13: CONN_01X04, Connectors_Molex:Molex_SPOX-5267_22-03-5045_04x2.54mm_Straight, F.Cu at (3.00, 18.0)
- added P14: CONN_01X06, RP_KiCAD_Connector:XA_6T, F.Cu at (3.00, 81.0)
- added P15: CONN_01X06, RP_KiCAD_Connector:XA_6T, F.Cu at (3.00, 63.5)
- added P16: CONN_01X02, Socket_Strips:Socket_Strip_Straight_1x02, F.Cu at (8.00, 52.0)
- added P17: CONN_01X04, RP_KiCAD_Connector:XA_4T, F.Cu at (3.00, 51.0)
- added P18: CONN_01X06, RP_KiCAD_Connector:ZH_6T, F.Cu at (-17.0, 7.25)
- added P19: CONN_01X06, RP_KiCAD_Connector:ZH_6T, F.Cu at (-8.00, 7.25)
- added P3: CONN_01X06, RP_KiCAD_Connector:ZH_6T, F.Cu at (34.0, 94.0)
- added P4: CONN_01X08, Socket_Strips:Socket_Strip_Straight_1x08, F.Cu at (33.0, 72.5)
- added P5: CONN_01X06, RP_KiCAD_Connector:ZH_6T, F.Cu at (26.5, 40.0)
- added P6: CONN_01X04, Socket_Strips:Socket_Strip_Straight_1x04, F.Cu at (19.0, 49.5)
- added P7: CONN_01X04, Socket_Strips:Socket_Strip_Straight_1x04, F.Cu at (21.0, 3.00)
- added P8: CONN_01X04, Socket_Strips:Socket_Strip_Straight_1x04, F.Cu at (32.0, 3.00)
- added P9: CONN_01X03, RP_KiCAD_Connector:XA_3T, F.Cu at (3.00, 23.5)
- added Q1: MOSFET_N, TO_SOT_Packages_SMD:SOT-428_GDS_compact, B.Cu at (67.5, 20.0)
- added Q10: MOSFET_N, TO_SOT_Packages_SMD:SOT-428_GDS_compact, B.Cu at (56.5, 52.0)
- added Q11: MOSFET_N, TO_SOT_Packages_SMD:SOT-428_GDS_compact, B.Cu at (67.5, 60.0)
- added Q12: MOSFET_N, TO_SOT_Packages_SMD:SOT-428_GDS_compact, B.Cu at (56.5, 60.0)
- added Q13: MOSFET_N, TO_SOT_Packages_SMD:SOT-428_GDS_compact, B.Cu at (67.5, 68.0)
- added Q14: MOSFET_N, TO_SOT_Packages_SMD:SOT-428_GDS_compact, B.Cu at (56.5, 68.0)
- added Q15: MOSFET_N, TO_SOT_Packages_SMD:SOT-428_GDS_compact, B.Cu at (67.5, 76.0)
- added Q16: MOSFET_N, TO_SOT_Packages_SMD:SOT-428_GDS_compact, B.Cu at (56.5, 76.0)
- added Q17: MOSFET_N, TO_SOT_Packages_SMD:SOT-23_Handsoldering, F.Cu at (9.50, 24.5)
- added Q2: MOSFET_N, TO_SOT_Packages_SMD:SOT-428_GDS_compact, B.Cu at (56.5, 20.0)
- added Q3: MOSFET_N, TO_SOT_Packages_SMD:SOT-428_GDS_compact, B.Cu at (67.5, 28.0)
- added Q4: MOSFET_N, TO_SOT_Packages_SMD:SOT-428_GDS_compact, B.Cu at (56.5, 28.0)
- added Q5: MOSFET_N, TO_SOT_Packages_SMD:SOT-428_GDS_compact, B.Cu at (67.5, 36.0)
- added Q6: MOSFET_N, TO_SOT_Packages_SMD:SOT-428_GDS_compact, B.Cu at (56.5, 36.0)
- added Q7: MOSFET_N, TO_SOT_Packages_SMD:SOT-428_GDS_compact, B.Cu at (67.5, 44.0)
- added Q8: MOSFET_N, TO_SOT_Packages_SMD:SOT-428_GDS_compact, B.Cu at (56.5, 44.0)
- added Q9: MOSFET_N, TO_SOT_Packages_SMD:SOT-428_GDS_compact, B.Cu at (67.5, 52.0)
- added R1: 10k, RP_KiCAD_Libs:C1608_WP, F.Cu at (37.5, 19.5)
- added R10: 100, RP_KiCAD_Libs:C1608_WP, B.Cu at (53.5, 36.5)
- added R11: 100, RP_KiCAD_Libs:C1608_WP, B.Cu at (64.5, 44.0)
- added R12: 100, RP_KiCAD_Libs:C1608_WP, B.Cu at (53.5, 44.5)
- added R13: 100, RP_KiCAD_Libs:C1608_WP, B.Cu at (64.5, 52.0)
- added R14: 100, RP_KiCAD_Libs:C1608_WP, B.Cu at (53.5, 52.5)
- added R15: 100, RP_KiCAD_Libs:C1608_WP, B.Cu at (64.5, 60.0)
- added R16: 100, RP_KiCAD_Libs:C1608_WP, B.Cu at (53.5, 60.5)
- added R17: 20k, RP_KiCAD_Libs:C1608_WP, F.Cu at (36.0, 80.0)
- added R18: 20k, RP_KiCAD_Libs:C1608_WP, F.Cu at (36.0, 77.5)
- added R19: R, RP_KiCAD_Libs:C1608_WP, F.Cu at (20.5, 90.5)
- added R2: 10k, RP_KiCAD_Libs:C1608_WP, F.Cu at (32.0, 36.0)
- added R20: 1k, RP_KiCAD_Libs:C1608_WP, F.Cu at (19.0, 43.0)
- added R21: 10k, RP_KiCAD_Libs:C1608_WP, F.Cu at (43.5, 79.5)
- added R22: 4.7k, RP_KiCAD_Libs:C1608_WP, F.Cu at (41.5, 79.5)
- added R23: 100, RP_KiCAD_Libs:C1608_WP, B.Cu at (64.5, 68.0)
- added R24: 100, RP_KiCAD_Libs:C1608_WP, B.Cu at (53.5, 68.5)
- added R25: 100, RP_KiCAD_Libs:C1608_WP, B.Cu at (64.5, 76.0)
- added R26: 100, RP_KiCAD_Libs:C1608_WP, B.Cu at (53.5, 76.5)
- added R27: 100, RP_KiCAD_Libs:C1608_WP, F.Cu at (30.5, 19.5)
- added R28: 100, RP_KiCAD_Libs:C1608_WP, F.Cu at (27.0, 19.5)
- added R29: 470, RP_KiCAD_Libs:C1608_WP, F.Cu at (27.3, 71.1)
- added R3: 100, RP_KiCAD_Libs:C1608_WP, F.Cu at (23.5, 19.5)
- added R30: 470, RP_KiCAD_Libs:C1608_WP, F.Cu at (27.3, 64.8)
- added R31: 1k, RP_KiCAD_Libs:C1608_WP, F.Cu at (32.0, 39.5)
- added R32: 10k, RP_KiCAD_Libs:C1608_WP, F.Cu at (21.0, 94.0)
- added R33: 1k, RP_KiCAD_Libs:C1608_WP, F.Cu at (8.50, 27.0)
- added R34: 10k, RP_KiCAD_Libs:C1608_WP, F.Cu at (13.0, 35.0)
- added R35: 10k, RP_KiCAD_Libs:C1608_WP, F.Cu at (13.0, 24.5)
- added R36: 1k, RP_KiCAD_Libs:C1608_WP, F.Cu at (8.00, 22.0)
- added R37: 1k, RP_KiCAD_Libs:C1608_WP, F.Cu at (11.5, 22.0)
- added R38: 470, RP_KiCAD_Libs:C1608_WP, F.Cu at (11.4, 73.7)
- added R39: 470, RP_KiCAD_Libs:C1608_WP, F.Cu at (11.4, 69.8)
- added R4: 100, RP_KiCAD_Libs:C1608_WP, F.Cu at (34.0, 19.5)
- added R40: 470, RP_KiCAD_Libs:C1608_WP, F.Cu at (11.4, 66.0)
- added R41: 1k, RP_KiCAD_Libs:C1608_WP, F.Cu at (11.4, 75.6)
- added R42: 1k, RP_KiCAD_Libs:C1608_WP, F.Cu at (11.4, 71.8)
- added R43: 1k, RP_KiCAD_Libs:C1608_WP, F.Cu at (11.4, 67.9)
- added R44: 120, RP_KiCAD_Libs:C1608_WP, F.Cu at (10.5, 51.0)
- added R45: R, RP_KiCAD_Libs:C1608_WP, B.Cu at (-13.0, 15.5)
- added R5: 100, RP_KiCAD_Libs:C1608_WP, B.Cu at (64.5, 19.5)
- added R6: 100, RP_KiCAD_Libs:C1608_WP, B.Cu at (53.5, 20.5)
- added R7: 100, RP_KiCAD_Libs:C1608_WP, B.Cu at (64.5, 27.5)
- added R8: 100, RP_KiCAD_Libs:C1608_WP, B.Cu at (53.5, 28.5)
- added R9: 100, RP_KiCAD_Libs:C1608_WP, B.Cu at (64.5, 36.0)
- added SW1: SW_PUSH, Buttons_Switches_SMD:SW_SPST_EVQPE1, F.Cu at (38.5, 14.5)
- added SW2: SW_PUSH, Buttons_Switches_SMD:SW_SPST_EVQPE1, F.Cu at (15.9, 94.0)
- added SW3: SWITCH_INV, Buttons_Switches_ThroughHole:SW_toggle_3P, F.Cu at (9.00, 6.00)
- added U1: STM32F103_48, Housings_QFP:LQFP-48_7x7mm_Pitch0.5mm, F.Cu at (21.4, 31.0)
- added U10: NCP5359, Housings_SOIC:SOIC-8_3.9x4.9mm_Pitch1.27mm, F.Cu at (48.5, 36.0)
- added U11: NCP5359, Housings_SOIC:SOIC-8_3.9x4.9mm_Pitch1.27mm, F.Cu at (48.5, 44.0)
- added U12: 74LS32, Housings_SOIC:SOIC-14_3.9x8.7mm_Pitch1.27mm, F.Cu at (35.0, 29.5)
- added U13: 74LS32, Housings_SOIC:SOIC-14_3.9x8.7mm_Pitch1.27mm, F.Cu at (35.0, 64.5)
- added U14: 74HC04, Housings_SOIC:SOIC-14_3.9x8.7mm_Pitch1.27mm, F.Cu at (35.0, 48.0)
- added U15: NCP1117ST12T3G, TO_SOT_Packages_SMD:SOT-223_reg, F.Cu at (35.5, 12.0)
- added U16: NCP1117ST33T3G, TO_SOT_Packages_SMD:SOT89-3_Housing, F.Cu at (-12.5, 11.5)
- added U2: NCP1117ST33T3G, TO_SOT_Packages_SMD:SOT-223_reg, F.Cu at (25.0, 12.0)
- added U3: NCP5359, Housings_SOIC:SOIC-8_3.9x4.9mm_Pitch1.27mm, F.Cu at (48.5, 52.0)
- added U4: MAX3051, Housings_SOIC:SOIC-8_3.9x4.9mm_Pitch1.27mm, F.Cu at (11.5, 56.5)
- added U5: NCP5359, Housings_SOIC:SOIC-8_3.9x4.9mm_Pitch1.27mm, F.Cu at (48.5, 60.0)
- added U6: NCP5359, Housings_SOIC:SOIC-8_3.9x4.9mm_Pitch1.27mm, F.Cu at (48.5, 68.0)
- added U7: NCP5359, Housings_SOIC:SOIC-8_3.9x4.9mm_Pitch1.27mm, F.Cu at (48.5, 76.0)
- added U8: NCP5359, Housings_SOIC:SOIC-8_3.9x4.9mm_Pitch1.27mm, F.Cu at (48.5, 20.0)
- added U9: NCP5359, Housings_SOIC:SOIC-8_3.9x4.9mm_Pitch1.27mm, F.Cu at (48.5, 28.0)
- added X1: CRYSTAL, Crystals:Crystal_HC50-U_Vertical, F.Cu at (28.0, 84.5)
- added X2: CRYSTAL, Crystals:ABM3_2pads, F.Cu at (21.5, 24.0)
Routing:
- net GND: track 0.00 -> 570.4 mm, vias 0 -> 20
- net +5V: track 0.00 -> 268.4 mm, vias 0 -> 11
- net +3.3V: track 0.00 -> 250.0 mm, vias 0 -> 16
- net +BATT: track 0.00 -> 237.4 mm, vias 0 -> 89
- net /GD_12V: track 0.00 -> 157.7 mm
- net GNDPWR: track 0.00 -> 121.0 mm, vias 0 -> 68
- net /Motor~SD: track 0.00 -> 102.1 mm, vias 0 -> 16
- net /AT_TX: track 0.00 -> 88.8 mm, vias 0 -> 4
- net /AT_RX: track 0.00 -> 78.6 mm, vias 0 -> 4
- net /OUT_2_A: track 0.00 -> 75.7 mm, vias 0 -> 42
- net /OUT_1_A: track 0.00 -> 72.3 mm, vias 0 -> 42
- net /OUT_0_B: track 0.00 -> 72.3 mm, vias 0 -> 42
- net /OUT_0_A: track 0.00 -> 72.1 mm, vias 0 -> 42
- net /OUT_1_B: track 0.00 -> 69.4 mm, vias 0 -> 42
- net +12V: track 0.00 -> 69.1 mm
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- added copper zone on B.Cu, net +BATT
- added copper zone on F.Cu, net +BATT
- added copper zone on B.Cu, net /OUT_0_A
- added copper zone on F.Cu, net /OUT_0_A
- added copper zone on B.Cu, net /OUT_0_B
- added copper zone on F.Cu, net /OUT_0_B
- added copper zone on B.Cu, net /OUT_1_A
- added copper zone on F.Cu, net /OUT_1_A
- added copper zone on B.Cu, net /OUT_1_B
- added copper zone on F.Cu, net /OUT_1_B
- added copper zone on B.Cu, net /OUT_2_A
- added copper zone on F.Cu, net /OUT_2_A
- added copper zone on B.Cu, net /OUT_2_B
- added copper zone on F.Cu, net /OUT_2_B
- added copper zone on B.Cu, net /OUT_3_A
- added copper zone on F.Cu, net /OUT_3_A
- added copper zone on B.Cu, net /OUT_3_B
- added copper zone on F.Cu, net /OUT_3_B
- added copper zone on B.Cu, net GNDPWR
- added copper zone on F.Cu, net GNDPWR
Other:
- board outline added: 100 x 100 mm
- board text added: "3.3V"
- board text added: "5V"
- board text added: "5V suppy"
- board text added: "ADD CNG"

Commit message: no message
Parts:
- removed C39, C40: 2.2u, RP_KiCAD_Libs:C2012
- removed ME1: AS504x, Housings_SSOP:SSOP-16_3.9x4.9mm_Pitch0.635mm
- removed P19: CONN_01X06, RP_KiCAD_Connector:ZH_6T
- removed U16: NCP1117ST33T3G, TO_SOT_Packages_SMD:SOT89-3_Housing
- added C44: 4.7u, RP_KiCAD_Libs:C3216, F.Cu at (20.0, 68.5)
- added D16: LED, LEDs:LED_0805, F.Cu at (10.0, 31.5)
- added JP5: JUMPER, Connect:GS2, F.Cu at (15.5, 20.5)
- added JP6: JUMPER3, Connect:GS3, B.Cu at (5.50, 26.5)
- added JP7: JUMPER3, Connect:GS3, B.Cu at (5.50, 36.0)
- added P2: CONN_01X04, RP_KiCAD_Connector:XA_4T, F.Cu at (3.00, 20.0)
- added P20: CONN_01X04, RP_KiCAD_Connector:XA_4T, F.Cu at (3.00, 32.5)
- added SW4: SW_PUSH, Buttons_Switches_SMD:RP_SMD_Button, F.Cu at (24.0, 56.0)
- added SW5: SW_PUSH, Buttons_Switches_SMD:RP_SMD_Button, F.Cu at (24.0, 60.5)
- added SW6: SW_PUSH, Buttons_Switches_SMD:RP_SMD_Button, F.Cu at (24.0, 47.0)
- added SW7: SW_PUSH, Buttons_Switches_SMD:RP_SMD_Button, F.Cu at (24.0, 51.5)
- JP4: value JUMPER3 -> JUMPER; footprint Connect:GS3 -> Connect:GS2
- P18: value CONN_01X06 -> CONN_01X04; footprint RP_KiCAD_Connector:ZH_6T -> Socket_Strips:Socket_Strip_Straight_1x04
- R1, R2: value 10k -> 1k
- R19: value R -> 1k
- R27, R28, R3, R4: value 100 -> 330
- R31: value 1k -> 470
- R45: value R -> 330; moved to F.Cu
- SW1, SW2: footprint Buttons_Switches_SMD:SW_SPST_EVQPE1 -> Buttons_Switches_SMD:RP_SMD_Button
- moved P18 60.2 mm to (8.00, 62.0), turned to 0 degrees
- moved JP4 38.8 mm to (20.0, 28.5), turned to 0 degrees
- moved R31 32.2 mm to (36.0, 71.5), turned to 180 degrees
- moved R45 31.0 mm to (13.5, 31.5)
- moved D1 18.4 mm to (13.5, 9.50)
- moved R3 15.9 mm to (16.0, 5.50)
- moved C41 15.0 mm to (9.00, 37.5), turned to 270 degrees
- moved U4 13.6 mm to (9.50, 43.0), turned to 270 degrees
- moved P9 13.5 mm to (3.00, 10.0)
- moved P1 11.5 mm to (3.00, 45.0)
- moved P17 10.5 mm to (13.5, 50.0)
- moved P13 7.63 mm to (9.50, 22.0)
- moved P16 6.50 mm to (8.00, 58.5)
- moved P6 5.70 mm to (14.5, 46.0), turned to 90 degrees
- moved R35 5.52 mm to (13.5, 30.0), turned to 180 degrees
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Connections:
- net /VALVE_2 renamed /AT_SW2
- net /VALVE_3 renamed /AT_SW1
- C12 pad 1: GNDPWR -> GND
- C13 pad 1: GNDPWR -> GND
- C15 pad 1: GNDPWR -> GND
- C16 pad 1: GNDPWR -> GND
- C17 pad 1: GNDPWR -> GND
- C18 pad 1: GNDPWR -> GND
- C23 pad 1: GNDPWR -> GND
- C24 pad 1: GNDPWR -> GND
- C30 pad 2: GNDPWR -> GND
- C31 pad 2: GNDPWR -> GND
- C32 pad 2: GNDPWR -> GND
- C33 pad 2: GNDPWR -> GND
- C34 pad 2: GNDPWR -> GND
- C35 pad 2: GNDPWR -> GND
- IC1 pad 19: (no net) -> /Motor~SD
- JP4 pad 1: /ENC_5V -> Net-(JP4-Pad1)
- JP4 pad 2: Net-(JP4-Pad2) -> GND
- P18 pad 1: /ENC_GND -> GND
- P18 pad 2: /ENC_5V -> +5V
- P18 pad 3: /ENC_~CS -> /I2C_SDA
- P18 pad 4: /ENC_SCK -> /I2C_SCL
- Q10 pad S: GNDPWR -> GND
- Q12 pad S: GNDPWR -> GND
- Q14 pad S: GNDPWR -> GND
- Q16 pad S: GNDPWR -> GND
- Q2 pad S: GNDPWR -> GND
- Q4 pad S: GNDPWR -> GND
- Q6 pad S: GNDPWR -> GND
- Q8 pad S: GNDPWR -> GND
- R45 pad 2: /ENC_Prog -> GND
- U1 pad 10: (no net) -> /PWM_T2C1
- U1 pad 11: (no net) -> /PWM_T2C2
- U1 pad 14: /STM_~SS0 -> /PWM_T3C1
- U1 pad 15: /STM_SCK -> /PWM_T3C2
- U1 pad 16: /STM_MISO -> Net-(JP4-Pad1)
- U1 pad 17: /STM_MOSI -> /STM_SW2
- U1 pad 18: (no net) -> /STM_SW1
- U1 pad 19: (no net) -> /SERVO_DIR
- U1 pad 20: /SERVO_DIR -> /STM_LED4
- U1 pad 25: (no net) -> /STM_~SS0
- U1 pad 26: (no net) -> /STM_SCK
- U1 pad 27: (no net) -> /STM_MISO
- U1 pad 28: (no net) -> /STM_MOSI
- U10 pad 6: GNDPWR -> GND
- U11 pad 6: GNDPWR -> GND
- U3 pad 6: GNDPWR -> GND
- U5 pad 6: GNDPWR -> GND
- U6 pad 6: GNDPWR -> GND
- U7 pad 6: GNDPWR -> GND
- U8 pad 6: GNDPWR -> GND
- U9 pad 6: GNDPWR -> GND
Routing:
- net GND: track 570.4 -> 922.6 mm, vias 20 -> 152
- net GNDPWR: track 121.0 -> 0.00 mm, vias 68 -> 0
- net /Motor~SD: track 102.1 -> 154.0 mm, vias 16 -> 22
- net /STM_SW2: track 0.00 -> 45.8 mm, vias 0 -> 4
- net /STM_SW1: track 0.00 -> 38.2 mm, vias 0 -> 4
- net +5V: track 268.4 -> 304.6 mm
- net /ENC_GND: track 25.5 -> 0.00 mm, vias 1 -> 0
- net /ENC_5V: track 21.4 -> 0.00 mm, vias 1 -> 0
- net /AT_SW1: track 8.93 -> 30.3 mm, vias 0 -> 1
- net /PWM_T2C2: track 0.00 -> 21.1 mm, vias 0 -> 1
- net /SBUS: track 6.87 -> 26.8 mm, vias 0 -> 1
- net /PWM_T2C1: track 0.00 -> 19.7 mm, vias 0 -> 1
- net /PWM_T3C2: track 0.00 -> 18.9 mm, vias 0 -> 1
- net /AT_SW2: track 7.62 -> 25.8 mm, vias 0 -> 1
- net /PWM_T3C1: track 0.00 -> 16.9 mm, vias 0 -> 1
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- added copper zone on B.Cu, net /LOGIC_BATT
- added copper zone on F.Cu, net /LOGIC_BATT
- added copper zone on B.Cu, net GND
- added copper zone on F.Cu, net GND
- removed copper zone on B.Cu, net GNDPWR
- removed copper zone on F.Cu, net GNDPWR
Other:
- board size 100 x 100 mm -> 77 x 96 mm
- board text added: "0A"
- board text added: "0B"
- board text added: "1"
- board text added: "12V"
- board text added: "1A"
- board text added: "1B"
- board text added: "2"
- board text added: "2017.08.08"
- board text added: "2A"
- board text added: "2B"
- board text added: "3"
- board text added: "3A"
- board text added: "3B"
- board text added: "AT_SW"
- board text added: "AnalogIn"
- board text added: "BATT"
- board text added: "CAN"
- board text added: "Encoder"
- board text added: "HC04"
- board text added: "I2C"
- board text added: "KawaRoboMainBoard ver1.0"
- board text added: "LED1"
- board text added: "LED2"
- board text added: "LGC BST"
- board text added: "MPU ADD"
- board text added: "MPU6050"
- board text added: "Mouse"
- board text added: "POWER"
- board text added: "PWM"
- board text added: "PWR"
- board text added: "RS485"
- board text added: "RST"
- board text added: "SBUS"
- board text added: "SDA SCL"
- board text added: "SPI"
- board text added: "ST-LINK"
- board text added: "STM_SPI"
- board text added: "STM_SW"
- board text added: "SW1"
- board text added: "SW2"
- board text added: "TRM"
- board text added: "UART"
- board text added: "USER_JP"
- board text removed: "ADD CNG"
