File: KiCAD_Projects/KawaRoboMain/KawaRoboMain.sch (KiCad schematic (older format))
At the start: 23 parts, among them P5 CONN_01X06, SW1 SW_PUSH, U1 STM32F103_48, U2 NCP1117ST33T3G, U4 NCP1117ST50T3G, X2 CRYSTAL

Commit message: Morex系ゴニョゴニョした
Parts:
- removed JP10: JUMPER3, Connect:GS3, symbol JUMPER3
- removed U4: NCP1117ST50T3G, TO_SOT_Packages_SMD:SOT-223_reg, symbol NCP1117ST50T3G
- added C11, C12, C13, C14, C15, C16, C17, C18, C19, C20, C21, C22, C23, C24, C25, C26, C36, C37: 4.7u, RP_KiCAD_Libs:C3216, symbol C
- added C27, C28: 22p, RP_KiCAD_Libs:C1608_WP, symbol C
- added C29, C38, C41, C42, C43: 0.1u, RP_KiCAD_Libs:C1608_WP, symbol C
- added C30, C31, C32, C33, C34, C35: 220u, Capacitors_ThroughHole:C_Radial_D10_L13_P5, symbol C
- added C39, C40: 2.2u, RP_KiCAD_Libs:C2012, symbol C
- added D10, D3, D4, D5, D6, D7, D8, D9: DIODE, RP_KiCAD_Libs:C2012, symbol DIODE
- added D11, D12, D13, D14: LED, LEDs:LED_0805, symbol LED
- added D15: DIODE, Diodes_SMD:SOD-123, symbol DIODE
- added IC1: ATMEGA328P-A, Housings_QFP:TQFP-32_7x7mm_Pitch0.8mm, symbol ATMEGA328P-A
- added IC2: SP3485CN, Housings_SOIC:SOIC-8_3.9x4.9mm_Pitch1.27mm, symbol SP3485CN
- added JP1, JP3: JUMPER, Connect:GS2, symbol JUMPER
- added JP2, JP4: JUMPER3, Connect:GS3, symbol JUMPER3
- added ME1: AS504x, Housings_SSOP:SSOP-16_3.9x4.9mm_Pitch0.635mm, symbol AS504x
- added P1, P14, P15: CONN_01X06, RP_KiCAD_Connector:XA_6T, symbol CONN_01X06
- added P10: CONN_01X02, RP_KiCAD_Connector:XA_2T, symbol CONN_01X02
- added P11, P12: CONN_01X12, Pin_Headers:Pin_Header_Straight_1x12, symbol CONN_01X12
- added P13: CONN_01X04, Connectors_Molex:Molex_SPOX-5267_22-03-5045_04x2.54mm_Straight, symbol CONN_01X04
- added P16: CONN_01X02, Socket_Strips:Socket_Strip_Straight_1x02, symbol CONN_01X02
- added P17: CONN_01X04, RP_KiCAD_Connector:XA_4T, symbol CONN_01X04
- added P18, P19, P3: CONN_01X06, RP_KiCAD_Connector:ZH_6T, symbol CONN_01X06
- added P4: CONN_01X08, Socket_Strips:Socket_Strip_Straight_1x08, symbol CONN_01X08
- added P6, P7, P8: CONN_01X04, Socket_Strips:Socket_Strip_Straight_1x04, symbol CONN_01X04
- added P9: CONN_01X03, RP_KiCAD_Connector:XA_3T, symbol CONN_01X03
- added Q1, Q10, Q11, Q12, Q13, Q14, Q15, Q16, Q2, Q3, Q4, Q5, Q6, Q7, Q8, Q9: MOSFET_N, TO_SOT_Packages_SMD:SOT-428_GDS_compact, symbol MOSFET_N
- added Q17: MOSFET_N, TO_SOT_Packages_SMD:SOT-23_Handsoldering, symbol MOSFET_N
- added R10, R11, R12, R13, R14, R15, R16, R23, R24, R25, R26, R27, R28, R5, R6, R7, R8, R9: 100, RP_KiCAD_Libs:C1608_WP, symbol R
- added R17, R18: 20k, RP_KiCAD_Libs:C1608_WP, symbol R
- added R19, R45: R, RP_KiCAD_Libs:C1608_WP, symbol R
- added R20, R31, R33, R36, R37, R41, R42, R43: 1k, RP_KiCAD_Libs:C1608_WP, symbol R
- added R21, R32, R34, R35: 10k, RP_KiCAD_Libs:C1608_WP, symbol R
- added R22: 4.7k, RP_KiCAD_Libs:C1608_WP, symbol R
- added R29, R30, R38, R39, R40: 470, RP_KiCAD_Libs:C1608_WP, symbol R
- added R44: 120, RP_KiCAD_Libs:C1608_WP, symbol R
- added SW2: SW_PUSH, Buttons_Switches_SMD:SW_SPST_EVQPE1, symbol SW_PUSH
- added SW3: SWITCH_INV, Buttons_Switches_ThroughHole:SW_toggle_3P, symbol SWITCH_INV
- added U10, U11, U3, U5, U6, U7, U8, U9: NCP5359, Housings_SOIC:SOIC-8_3.9x4.9mm_Pitch1.27mm, symbol NCP5359
- added U12, U13: 74LS32, Housings_SOIC:SOIC-14_3.9x8.7mm_Pitch1.27mm, symbol 74LS32
- added U14: 74HC04, Housings_SOIC:SOIC-14_3.9x8.7mm_Pitch1.27mm, symbol 74HC04
- added U15: NCP1117ST12T3G, TO_SOT_Packages_SMD:SOT-223_reg, symbol NCP1117ST12T3G
- added U16: NCP1117ST33T3G, TO_SOT_Packages_SMD:SOT89-3_Housing, symbol NCP1117ST33T3G
- added U4: MAX3051, Housings_SOIC:SOIC-8_3.9x4.9mm_Pitch1.27mm, symbol MAX3051
- added X1: CRYSTAL, Crystals:Crystal_HC50-U_Vertical, symbol CRYSTAL
- C2, C7: footprint RP_KiCAD_Libs:C2012 -> RP_KiCAD_Libs:C3216
- C3: value 4.7u -> 0.1u; footprint RP_KiCAD_Libs:C2012 -> RP_KiCAD_Libs:C1608_WP
Connections:
- net labels added: +BATT, AT_A2, AT_A3, AT_LED1, AT_LED2, AT_RST, AT_RX, AT_TX, DCDC_EN, ENC_5V, ENC_GND, ENC_MISO, ENC_Prog, ENC_SCK, ENC_~CS, GD_12V, GNDPWR, I2C_SCL, I2C_SDA, INT0, INT1, LOGIC_BATT, Motor0CW, Motor0PWM, Motor1CW, Motor1PWM, Motor2CW, Motor2PWM, Motor3CW, Motor3PWM, Motor~SD, OUT_0_A, OUT_0_B, OUT_1_A, OUT_1_B, OUT_2_A, OUT_2_B, OUT_3_A, OUT_3_B, PWM_0_A, PWM_0_B, PWM_1_A, PWM_1_B, PWM_2_A, PWM_2_B, PWM_3_A, PWM_3_B, RAW, SBUS, SERVO_DIR, SERVO_RX, SERVO_TX, SPI_MISO, SPI_MOSI, SPI_SCK, SPI_SS_ENC, SPI_SS_Mouse, SPI_SS_USB, STM_LED1, STM_LED2, STM_LED3, STM_MISO, STM_MOSI, STM_SCK, STM_~SS0, STM_~SS1, STM_~SS2, VALVE_0, VALVE_1, VALVE_2, VALVE_3, VCC, batt_voltage, ~SD~_0, ~SD~_1, ~SD~_2, ~SD~_3
- wire segments 14 -> 272
- no-connect marks 0 -> 10
Other:
- note removed: "LED"
- moved on the sheet: C2, C4, C5, C7, C9, D1, D2, P5, R1, R2, R3, R4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

Commit message: no message
Parts:
- removed C39, C40: 2.2u, RP_KiCAD_Libs:C2012, symbol C
- removed JP4: JUMPER3, Connect:GS3, symbol JUMPER3
- removed ME1: AS504x, Housings_SSOP:SSOP-16_3.9x4.9mm_Pitch0.635mm, symbol AS504x
- removed P18, P19: CONN_01X06, RP_KiCAD_Connector:ZH_6T, symbol CONN_01X06
- removed U16: NCP1117ST33T3G, TO_SOT_Packages_SMD:SOT89-3_Housing, symbol NCP1117ST33T3G
- added C44: 4.7u, RP_KiCAD_Libs:C3216, symbol C
- added D16: LED, LEDs:LED_0805, symbol LED
- added JP4, JP5: JUMPER, Connect:GS2, symbol JUMPER
- added JP6, JP7: JUMPER3, Connect:GS3, symbol JUMPER3
- added P18: CONN_01X04, Socket_Strips:Socket_Strip_Straight_1x04, symbol CONN_01X04
- added P2, P20: CONN_01X04, RP_KiCAD_Connector:XA_4T, symbol CONN_01X04
- added SW4, SW5, SW6, SW7: SW_PUSH, Buttons_Switches_SMD:RP_SMD_Button, symbol SW_PUSH
- R1, R2: value 10k -> 1k
- R19: value R -> 1k
- R27, R28, R3, R4: value 100 -> 330
- R31: value 1k -> 470
- R45: value R -> 330
- SW1, SW2: footprint Buttons_Switches_SMD:SW_SPST_EVQPE1 -> Buttons_Switches_SMD:RP_SMD_Button
Connections:
- net ENC_Prog is gone; now on net GND: R45.2
- net GNDPWR is gone; now on net GND: C12.1, C13.1, C15.1, C16.1, C17.1, C18.1, C23.1, C24.1, C30.2, C31.2, C32.2, C33.2, C34.2, C35.2, Q10.S, Q12.S, Q14.S, Q16.S, Q2.S, Q4.S, Q6.S, Q8.S, U10.6 (GND), U11.6 (GND), U3.6 (GND), U5.6 (GND), U6.6 (GND), U7.6 (GND), U8.6 (GND), U9.6 (GND)
- net STM_~SS2 is gone; now on net SERVO_DIR: U1.19 (PB1/ADC12_IN9)
- net +12V: now also JP6.3, JP7.3
- net +5V: now also C44.1, JP6.1, JP7.1, P18.2 (P2)
- net GND: now also C44.2, JP4.2, P18.1 (P1), P2.1 (P1), P20.1 (P1), SW4.1, SW5.1, SW6.1, SW7.1
- net I2C_SCL: now also P18.4 (P4)
- net I2C_SDA: now also P18.3 (P3)
- net Motor~SD: now also IC1.19 (ADC6)
- net SERVO_DIR: no longer U1.20 (PB2/BOOT1)
- net SERVO_TX: now also JP5.2
- net STM_MISO: now also U1.27 (PB14/SPI2_MISO); no longer U1.16 (PA6/SPI1_MISO)
- net STM_MOSI: now also U1.28 (PB15/SPI2_MOSI); no longer U1.17 (PA7/SPI1_MOSI)
- net STM_SCK: now also U1.26 (PB13/SPI2_SCK); no longer U1.15 (PA5/SPI1_SCK)
- net STM_~SS0: now also U1.25 (PB12/SPI2_NSS); no longer U1.14 (PA4/SPI1_NSS)
- net STM_~SS1: now also U1.29 (PA8); no longer U1.18 (PB0/ADC12_IN8)
- net PWM_T2C1: now reaches U1.10 (PA0/WKUP/ADC12_IN0)
- net PWM_T2C1: now also P2.3 (P3)
- net PWM_T2C2: now reaches U1.11 (PA1/ADC12_IN1)
- net PWM_T2C2: now also P2.4 (P4)
- net at IC2.6 (A), P13.2 (P2): now also JP5.1
- net at R45.1: now also D16.2 (K)
- net VALVE_2 renamed AT_SW2
- net AT_SW2: now also SW5.2
- net VALVE_3 renamed AT_SW1
- net AT_SW1: now also SW4.2
- new net: JP4.1, U1.16 (PA6/SPI1_MISO)
- new net: JP7.2, P20.2 (P2)
- new net: JP6.2, P2.2 (P2)
- new net PWM_T3C1: P20.3 (P3), U1.14 (PA4/SPI1_NSS)
- new net PWM_T3C2: P20.4 (P4), U1.15 (PA5/SPI1_SCK)
- new net STM_LED4: D16.1 (A), U1.20 (PB2/BOOT1)
- new net STM_SW1: SW6.2, U1.18 (PB0/ADC12_IN8)
- new net STM_SW2: SW7.2, U1.17 (PA7/SPI1_MOSI)
- no-connect marks 10 -> 7
Other:
- moved on the sheet: D13, D14, R29, R30
