File: KiCAD_Projects/AS5040/AS5040.kicad_pcb (KiCad board)
At the start: 2 copper layers, 45 x 20 mm, 16 parts, among them P1 CONN_01X06, P2 CONN_01X06, P3 CONN_01X06, P4 CONN_01X06, P5 CONN_01X06, P6 CONN_01X06, U1 NCP1117ST33T3G, U2 NCP1117ST33T3G

Commit message: no message
Parts:
- moved C3 1.00 mm to (36.0, 13.5)
- moved C4 1.00 mm to (36.0, 5.00)
- moved JP2 1.00 mm to (36.0, 13.5)
- moved ME2 1.00 mm to (36.0, 10.0)
- moved P4 1.00 mm to (26.0, 13.0)
- moved P5 1.00 mm to (30.0, 13.0)
- moved P6 1.00 mm to (41.0, 13.0)
- moved U2 1.00 mm to (36.0, 9.00)
Routing:
- net GND: track 67.2 -> 68.2 mm
- net +5V: track 59.9 -> 60.9 mm
Other:
- board size 45 x 20 mm -> 46 x 20 mm
