File: KiCAD_Projects/KawaRoboMain_ver1.1/KawaRoboMain_ver1.1.sch (KiCad schematic (older format))
At the start: 178 parts, among them IC1 ATMEGA328P-A, IC2 SP3485CN, P1 CONN_01X06, P10 CONN_01X02, P11 CONN_01X12, P12 CONN_01X12, P13 CONN_01X04, P14 CONN_01X06, P15 CONN_01X06, P16 CONN_01X02, P17 CONN_01X04, P18 CONN_01X04, P19 CONN_01X01, P2 CONN_01X04, P20 CONN_01X04, P21 CONN_01X01, P22 CONN_01X01, P3 CONN_01X06, P4 CONN_01X08, P5 CONN_01X06, P6 CONN_01X04, P7 CONN_01X04, P8 CONN_01X04, P9 CONN_01X03, Q1 MOSFET_N, Q10 MOSFET_N, Q11 MOSFET_N, Q12 MOSFET_N, Q13 MOSFET_N, Q14 MOSFET_N, Q15 MOSFET_N, Q16 MOSFET_N, Q17 MOSFET_N, Q2 MOSFET_N, Q3 MOSFET_N, Q4 MOSFET_N, Q5 MOSFET_N, Q6 MOSFET_N, Q7 MOSFET_N, Q8 MOSFET_N, Q9 MOSFET_N, SW1 SW_PUSH, SW2 SW_PUSH, SW3 SWITCH_INV, SW4 SW_PUSH, SW5 SW_PUSH, SW6 SW_PUSH, SW7 SW_PUSH, U1 STM32F103_48, U10 NCP5359, U11 NCP5359, U14 74HC04, U15 NCP1117ST12T3G, U16 74HC02, U17 74HC02, U2 NCP1117ST33T3G, U3 NCP5359, U4 MAX3051, U5 NCP5359, U6 NCP5359, U7 NCP5359, U8 NCP5359, U9 NCP5359, X1 CRYSTAL, X2 CRYSTAL

Commit message: かわロボ基2.0設計中
Parts:
- removed R13, R14, R15, R16, R23, R24, R25, R26: 100, RP_KiCAD_Libs:C1608_WP, symbol R
- removed R31: 470, RP_KiCAD_Libs:C1608_WP, symbol R
- added JP10, JP11, JP12, JP9: JUMPER, Connect:GS2, symbol JUMPER
- added JP8: JUMPER3, Connect:GS3, symbol JUMPER3
- C1, C10, C27, C28, C29, C3, C38, C4, C41, C42, C43, C5, C6, C8, C9, R1, R17, R18, R19, R2, R20, R21, R22, R27, R28, R29, R3, R30, R32, R33, R34, R35, R36, R37, R38, R39, R4, R40, R41, R42, R43, R44, R45: footprint RP_KiCAD_Libs:C1608_WP -> RP_KiCAD_Libs:C1608_WP_S
- C11, C12, C13, C14, C15, C16, C17, C18, C19, C2, C20, C21, C22, C23, C24, C25, C26, C36, C37, C40, C44, C45, C46, C7: footprint RP_KiCAD_Libs:C3216 -> RP_KiCAD_Libs:C3216_S
- IC2, U10, U11, U3, U4, U5, U6, U7, U8, U9: footprint Housings_SOIC:SOIC-8_3.9x4.9mm_Pitch1.27mm -> Housings_SOIC:SOIC-8_3.9x4.9mm_Pitch1.27mm_S
- P4: footprint Socket_Strips:Socket_Strip_Straight_1x08 -> Socket_Strips:Socket_Strip_Straight_1x08_MPU6050
- R10, R11, R12, R5, R6, R7, R8, R9: value 100 -> 1k; footprint RP_KiCAD_Libs:C1608_WP -> RP_KiCAD_Libs:C1608_WP_S
Connections:
- net VALVE_0 is gone; now on net Motor~SD: IC1.2 ((PCINT20/XCK/T0)PD4), P11.6 (P6)
- net +12V: now also P7.4 (P4), JP8.3; no longer P17.2 (P2), P7.1 (P1)
- net +5V: now also P8.4 (P4), JP8.1; no longer P8.1 (P1)
- net GND: now also P7.3 (P3), P8.3 (P3), R10.2, R11.2, R12.2, R5.2, R6.2, R7.2, R8.2, R9.2; no longer P7.2 (P2), P8.2 (P2)
- net I2C_SCL: now also JP9.2
- net I2C_SDA: now also JP10.2
- net Motor0CW: now also U14.1, U16.3; no longer U16.11, U16.2
- net Motor0PWM: now also U16.11, U16.2; no longer U14.1, U16.3
- net Motor1CW: now also U14.3, U16.9; no longer U16.5, U16.8
- net Motor1PWM: now also U16.5, U16.8; no longer U14.3, U16.9
- net Motor2CW: now also U14.5, U17.3; no longer U17.11, U17.2
- net Motor2PWM: now also U17.11, U17.2; no longer U14.5, U17.3
- net Motor3CW: now also U14.9, U17.6; no longer U17.5, U17.8
- net Motor3PWM: now also U17.5, U17.8; no longer U14.9, U17.6
- net Motor~SD: no longer IC1.19 (ADC6)
- net OUT_0_A: now also R9.1
- net OUT_0_B: now also R10.1
- net OUT_1_A: now also R11.1
- net OUT_1_B: now also R12.1
- net OUT_2_A: now also R5.1
- net OUT_2_B: now also R6.1
- net OUT_3_A: now also R7.1
- net OUT_3_B: now also R8.1
- net at Q1.G: now also U8.8 (DRV_HI); no longer R5.1
- net at Q2.G: now also U8.5 (DRV_LO); no longer R6.1
- net at Q3.G: now also U9.8 (DRV_HI); no longer R7.1
- net at Q4.G: now also U9.5 (DRV_LO); no longer R8.1
- net at Q5.G: now also U10.8 (DRV_HI); no longer R9.1
- net at Q6.G: now also U10.5 (DRV_LO); no longer R10.1
- net at Q7.G: now also U11.8 (DRV_HI); no longer R11.1
- net at Q8.G: now also U11.5 (DRV_LO); no longer R12.1
- net at Q9.G: now also U3.8 (DRV_HI)
- net at Q10.G: now also U3.5 (DRV_LO)
- net at Q11.G: now also U5.8 (DRV_HI)
- net at Q12.G: now also U5.5 (DRV_LO)
- net at Q13.G: now also U6.8 (DRV_HI)
- net at Q14.G: now also U6.5 (DRV_LO)
- net at Q15.G: now also U7.8 (DRV_HI)
- net at Q16.G: now also U7.5 (DRV_LO)
- net at P10.1 (P1), SW3.2: now also P7.2 (P2), P8.2 (P2); no longer P7.3 (P3), P8.3 (P3)
- net at R44.2, U4.6 (CANL): now also JP11.2; no longer P17.4 (P4)
- net at P16.2 (P2), U4.7 (CANH): now also JP12.2; no longer P17.3 (P3)
- removed net DCDC_EN: P7.4 (P4), P8.4 (P4)
- net VALVE_1 renamed BUZZER
- new net: JP8.2, P17.2 (P2)
- new net: JP10.1, JP12.1, P17.3 (P3)
- new net: JP11.1, JP9.1, P17.4 (P4)
- no-connect marks 7 -> 9
Other:
- moved on the sheet: P17
