File: KiCAD_Projects/_oldPCBs/MicroMouse_1.0/MicroMouse_1.0.sch (KiCad schematic (older format))
At the start: 36 parts, among them P5 CONN_01X06, SW1 SW_PUSH, U1 STM32F103_48, U4 NCP1117ST50T3G, X2 CRYSTAL

Commit message: ブラシレス作り始めた(n回目)
Changed lines of the file:
@@
 Text Label 14800 5950 2    60   ~ 0
 OUT_R2
-Text Label 6650 1450 0    60   ~ 0
+Text Label 5950 1050 0    60   ~ 0
 MotorEN
-Text Label 6650 1550 0    60   ~ 0
+Text Label 5950 1150 0    60   ~ 0
 PWM_L
-Text Label 6650 1650 0    60   ~ 0
+Text Label 5950 1250 0    60   ~ 0
 PWM_R
 Text Label 4000 4050 2    60   ~ 0
