File: KiCAD_Projects/CanBLDCMD_ver1.0/CanBLDCMD_ver1.0.sch (KiCad schematic (older format))
At the start: 111 parts, among them P1 CONN_01X04, P10 CONN_01X02, P3 CONN_01X04, P4 CONN_01X04, P5 CONN_01X02, P6 CONN_01X04, P7 CONN_01X06, P8 CONN_01X02, P9 CONN_01X02, Q1 MOSFET_N, Q2 MOSFET_N, Q3 MOSFET_N, Q4 MOSFET_N, Q5 MOSFET_N, Q6 MOSFET_N, SW1 SW_PUSH, SW2 SW_PUSH, SW3 SW_PUSH, U1 SW_ROTARY_16, U2 MAX3051, U3 STM32F103_48, U4 SI8275, U5 SI8275, U6 SI8275, U7 7805, U8 NCP1117ST33T3G, U9 LM1084IS-3.3/NOPB, X1 ceralock

Commit message: F103mini_rev2.0おわり｡BLDCの部品選定終わったけど電圧フィードバックで詰んだ
Parts:
- removed AMP1, AMP2, AMP3: TSC103, Housings_SOIC:SOIC-8_3.9x4.9mm_Pitch1.27mm, symbol TSC103
- removed C5: 0.1u, RP_KiCAD_Libs:C1608_WP, symbol C
- removed P1: CONN_01X04, RP_KiCAD_Connector:XA_4LC, symbol CONN_01X04
- removed P10, P9: CONN_01X02, RP_KiCAD_Connector:XT60, symbol CONN_01X02
- removed R16: 4.7k, RP_KiCAD_Libs:C1608_WP, symbol R
- removed R18, R19: 10k, RP_KiCAD_Libs:C1608_WP, symbol R
- removed U1: SW_ROTARY_16, Buttons_Switches_ThroughHole:rotary_0F, symbol SW_ROTARY_16
- added CS1, CS2, CS3: TS1102, TO_SOT_Packages_SMD:SOT-23-5, symbol TS1102
- added D16, D17, D18, D19, D20, D21, D22, D23, D8: LED, RP_KiCAD_Libs:C1608_WP, symbol LED
- added D24, D25, D26: DIODE, RP_KiCAD_Libs:C1608_WP, symbol DIODE-RESCUE-3WS_MD_rev2.1
- added JP1: JUMPER3, Connect:GS3, symbol JUMPER3
- added P1: CONN_01X06, RP_KiCAD_Connector:XA_6T, symbol CONN_01X06
- added R10, R17, R20, R21, R22, R23, R24, R25, R9: 1k, RP_KiCAD_Libs:C1608_WP, symbol R
- added W1, W10, W11, W12, W13, W14, W15, W2, W3, W4, W5, W6, W7, W8, W9: TEST_1P, Connect:PINTST, symbol TEST_1P
- P4: footprint RP_KiCAD_Connector:XA_4LC -> RP_KiCAD_Connector:XA_4T
- Q1, Q2, Q3, Q4, Q5, Q6: footprint TO_SOT_Packages_SMD:D2-PAK_compact -> TO_SOT_Packages_SMD:SOT-428_GDS_compact
- R15: value 4.7k -> 1k
Connections:
- net GNDPWR is gone; now on net GND: C13.2, C15.2, C17.2, C20.2, C21.2, C22.1, C23.1, C24.1, C26.2, C27.2, C28.2, C29.2, C30.2, C31.2, C32.2, C33.2, C34.2, DCDC1.3 (GND), P8.1 (P1), Q2.S, Q4.S, Q6.S, R38.2, U4.9 (GNCB), U5.9 (GNCB), U6.9 (GNCB), U9.1 (GND)
- net +3.3V: now also JP1.1
- net +5V: now also JP1.3; no longer R7.1, R8.1
- net +BATT: now also CS1.5 (RS+), CS2.5 (RS+), CS3.5 (RS+)
- net BattSense: now also U3.13 (PA3/USART2_RX)
- net CS_U: now also R8.1, U3.12 (PA2/USART2_TX), D25.1 (A)
- net CS_V: now also R15.1, U3.11 (PA1/ADC12_IN1), D26.1 (A)
- net CS_W: now also R7.1, U3.10 (PA0/WKUP/ADC12_IN0), D24.1 (A)
- net EN_U: now also U3.45 (PB8/TIM4_CH3), D17.1 (A), W3.1
- net EN_V: now also U3.43 (PB7/I2C_SDA), D20.1 (A), W6.1
- net EN_W: now also U3.42 (PB6/I2C_SCL), D23.1 (A), W9.1
- net GND: now also CS1.1 (GND), CS1.2 (GND), CS2.1 (GND), CS2.2 (GND), CS3.1 (GND), CS3.2 (GND), P1.6 (P6), R10.2, R17.2, R20.2, R21.2, R22.2, R23.2, R24.2, R25.2, R9.2
- net PWM_U_H: now also U3.31 (PA10/USART_RX), D8.1 (A), W1.1
- net PWM_U_L: now also U3.28 (PB15/SPI2_MOSI), D16.1 (A), W2.1
- net PWM_V_H: now also U3.30 (PA9/USART1_TX), D18.1 (A), W4.1
- net PWM_V_L: now also U3.27 (PB14/SPI2_MISO), D19.1 (A), W5.1
- net PWM_W_H: now also U3.29 (PA8), D21.1 (A), W7.1
- net PWM_W_L: now also U3.26 (PB13/SPI2_SCK), D22.1 (A), W8.1
- net PW_3.3V: now also D24.2 (K), D25.2 (K), D26.2 (K); no longer C27.1, C28.1, C29.1
- net Vsense_U: now also U3.18 (PB0/ADC12_IN8), W11.1
- net Vsense_V: now also U3.15 (PA5/SPI1_SCK), W12.1
- net Vsense_W: now also U3.14 (PA4/SPI1_NSS), W10.1
- net SPI_NSS: now reaches U3.38 (PA15/TDI)
- net SPI_NSS: now also P1.4 (P4)
- net SPI_SCK: now reaches U3.39 (PB3/TDO)
- net SPI_SCK: now also P1.3 (P3)
- net SPI_MISO: now reaches U3.40 (PB4/NTRST)
- net SPI_MISO: now also P1.2 (P2)
- net SPI_MOSI: now reaches U3.41 (PB5/I2C1_SMBAI)
- net SPI_MOSI: now also P1.1 (P1)
- net at Q3.D, R29.1, R32.1: now also CS2.4 (RS-)
- net at Q5.D, R30.1, R33.1: now also CS3.4 (RS-)
- net at Q1.D, R28.1, R31.1: now also CS1.4 (RS-)
- net ENC_A: no longer names the net of R15.2
- net ENC_A: now also C29.1, CS3.3 (OUT), W15.1
- net ENC_Aa: no longer names the net of R7.2
- net ENC_Aa: now also C27.1, CS1.3 (OUT), W13.1
- net ENC_Ab: no longer names the net of R8.2
- net ENC_Ab: now also C28.1, CS2.3 (OUT), W14.1
- new net: D8.2 (K), R9.1
- new net: D16.2 (K), R10.1
- new net: D17.2 (K), R17.1
- new net: D18.2 (K), R20.1
- new net: D19.2 (K), R21.1
- new net: D20.2 (K), R22.1
- new net: D21.2 (K), R23.1
- new net: D22.2 (K), R24.1
- new net: D23.2 (K), R25.1
- new net: JP1.2, P1.5 (P5)
Other:
- moved on the sheet: C27, C28, C29

Commit message: BLDCもだいたい設計終わった
Parts:
- removed C20, C26: 4.7u, RP_KiCAD_Libs:C3216, symbol C
- removed D4, D5: LED, RP_KiCAD_Libs:C1608_WP, symbol LED
- removed R12, R6: 100, RP_KiCAD_Libs:C1608_WP, symbol R
- removed U9: LM1084IS-3.3/NOPB, TO_SOT_Packages_SMD:SOT89-3_Housing, symbol LM1084IS-3.3/NOPB
- added C1: 4.7u, RP_KiCAD_Libs:C3216, symbol C
- added D27, D28, D29: LED, RP_KiCAD_Libs:C1608_WP, symbol LED
- added P2: CONN_01X06, RP_KiCAD_Connector:ZH_6T, symbol CONN_01X06
- added Q7, Q8, Q9: MOSFET_N, TO_SOT_Packages_SMD:SOT-23_Handsoldering, symbol MOSFET_N
- added R16, R18, R19: 1k, RP_KiCAD_Libs:C1608_WP, symbol R
- added R26, R39, R40: 100, RP_KiCAD_Libs:C1608_WP, symbol R
- P6: footprint RP_KiCAD_Connector:XA_4LC -> RP_KiCAD_Connector:XA_4T
Connections:
- net GD_12V is gone; now on net +12V: D10.1 (A), D11.1 (A), D12.1 (A), D13.1 (A), D14.1 (A), D9.1 (A)
- net PW_3.3V is gone; now on net +3.3V: D24.2 (K), D25.2 (K), D26.2 (K)
- net +3.3V: now also C1.1, D27.1 (A), D28.1 (A), D29.1 (A), R16.1, R18.1, R19.1
- net +5V: now also P2.1 (P1)
- net GND: now also P1.1 (P1), C1.2, P2.6 (P6), Q7.S, Q8.S, Q9.S; no longer P1.6 (P6)
- net SPI_MISO: now also P1.5 (P5); no longer P1.2 (P2)
- net SPI_MOSI: now also P1.6 (P6); no longer P1.1 (P1)
- net SPI_NSS: now also P1.3 (P3); no longer P1.4 (P4)
- net SPI_SCK: now also P1.4 (P4); no longer P1.3 (P3)
- net SW1: now also U3.20 (PB2/BOOT1)
- net SW2: now also U3.46 (PB9/TIM4_CH4)
- net HALL_0: now reaches U3.16 (PA6/SPI1_MISO)
- net HALL_0: now also Q7.D, R26.2
- net HALL_1: now reaches U3.17 (PA7/SPI1_MOSI)
- net HALL_1: now also Q8.D, R39.2
- net HALL_2: now reaches U3.19 (PB1/ADC12_IN9)
- net HALL_2: now also Q9.D, R40.2
- net at JP1.2: now also P1.2 (P2); no longer P1.5 (P5)
- new net: P2.3 (P3), Q7.G, R18.2
- new net: P2.4 (P4), Q8.G, R16.2
- new net: P2.5 (P5), Q9.G, R19.2
- new net: D27.2 (K), R26.1
- new net: D28.2 (K), R39.1
- new net: D29.2 (K), R40.1
- no-connect marks 13 -> 14
