File: KiCAD_Projects/STM32F103_mini_rev2.0/STM32F103_mini_rev2.0.sch (KiCad schematic (older format))
At the start: 44 parts, among them IC1 SP3485EN, P1 CONN_01X21, P2 CONN_01X04, P3 CONN_01X21, P4 USB_OTG, P5 CONN_01X06, P6 CONN_01X02, P7 CONN_01X04, SW1 SW_PUSH, U1 STM32F103_48, U2 NCP1117ST33T3G, U3 MAX3051, U4 78L05, U5 CH340, X1 ceralock, X2 ceralock

Commit message: BLDCもだいたい設計終わった
Parts:
- added D5, D6, D7: LED, LEDs:LED_0603, symbol LED
- added R10, R11, R12: 100, RP_KiCAD_Libs:C1608_WP, symbol R
Connections:
- net +12V: now also D5.1 (A)
- net +5V: now also D7.1 (A)
- net GND: now also R10.2, R11.2, R12.2
- net Vbus: now also D6.1 (A)
- new net: D5.2 (K), R10.1
- new net: D6.2 (K), R11.1
- new net: D7.2 (K), R12.1
Other:
- moved on the sheet: D1, D2, D3, D4, R3, R4, R8, R9
