File: KiCAD_Projects/_RoboconPCBs/for_MDdocument/for_MDdocument.sch (KiCad schematic (older format))
At the start: 26 parts, among them Q1 MOSFET_N, Q2 MOSFET_N, Q3 MOSFET_N, Q4 MOSFET_N, U1 SI8234, U2 SI8234

Commit message: no message
Parts:
- removed FB1, FB2, FB3, FB4: FILTER, RP_KiCAD_Libs:C1608_WP, symbol FILTER
Connections:
- net GNDPWR: now also C2.2, C4.2
- net OUT_A: now also C1.2
- net OUT_B: now also C3.2
- net at U1.10 (VOB): now also R4.2
- net at D2.1 (K), U1.11 (VDDB): now also C2.1
- net at U1.15 (VOA): now also R3.2
- net at D1.1 (K), U1.16 (VDDA): now also C1.1
- net at U2.10 (VOB): now also R8.2
- net at D4.1 (K), U2.11 (VDDB): now also C4.1
- net at U2.15 (VOA): now also R7.2
- net at D3.1 (K), U2.16 (VDDA): now also C3.1
Changed lines of the file:
@@
 LIBS:regul
 LIBS:stm32
-LIBS:user
 LIBS:Power_Management
 LIBS:powerint
@@
 $EndComp
 $Comp
-L FILTER FB1
-U 1 1 58D11CCA
-P 6100 2150
-F 0 "FB1" H 6100 2300 60  0000 C CNN
-F 1 "FILTER" H 6100 2050 60  0000 C CNN
-F 2 "RP_KiCAD_Libs:C1608_WP" H 6100 2150 60  0001 C CNN
-F 3 "" H 6100 2150 60  0000 C CNN
-	1    6100 2150
-	1    0    0    -1
-$EndComp
-$Comp
 L C C1
 U 1 1 58D11D28
@@
 	5450 2350 7250 2350
 Wire Wire Line
-	5750 2150 5300 2150
+	5300 2150 6550 2150
 $Comp
 L R R3
@@
 Wire Wire Line
 	6950 2150 6850 2150
-Wire Wire Line
-	6550 2150 6450 2150
 Connection ~ 5600 2350
 $Comp
@@
 $EndComp
 $Comp
-L FILTER FB2
-U 1 1 58D121A7
-P 6100 2900
-F 0 "FB2" H 6100 3050 60  0000 C CNN
-F 1 "FILTER" H 6100 2800 60  0000 C CNN
-F 2 "RP_KiCAD_Libs:C1608_WP" H 6100 2900 60  0001 C CNN
-F 3 "" H 6100 2900 60  0000 C CNN
-	1    6100 2900
-	1    0    0    -1
-$EndComp
-$Comp
 L C C2
 U 1 1 58D121AD
@@
 	5450 3100 7250 3100
 Wire Wire Line
-	5750 2900 5300 2900
+	5300 2900 6550 2900
 $Comp
 L R R4
@@
 Wire Wire Line
 	6950 2900 6850 2900
-Wire Wire Line
-	6550 2900 6450 2900
 Connection ~ 5600 3100
 $Comp
@@
 $EndComp
 $Comp
-L FILTER FB3
-U 1 1 58D1AA07
-P 6100 3850
-F 0 "FB3" H 6100 4000 60  0000 C CNN
-F 1 "FILTER" H 6100 3750 60  0000 C CNN
-F 2 "RP_KiCAD_Libs:C1608_WP" H 6100 3850 60  0001 C CNN
-F 3 "" H 6100 3850 60  0000 C CNN
-	1    6100 3850
-	1    0    0    -1
-$EndComp
-$Comp
 L C C3
 U 1 1 58D1AA0D
@@
 	5450 4050 7250 4050
 Wire Wire Line
-	5750 3850 5300 3850
+	5300 3850 6550 3850
 $Comp
 L R R7
@@
 Wire Wire Line
 	6950 3850 6850 3850
-Wire Wire Line
-	6550 3850 6450 3850
 Connection ~ 5600 4050
 $Comp
@@
 $EndComp
 $Comp
-L FILTER FB4
-U 1 1 58D1AA39
-P 6100 4600
-F 0 "FB4" H 6100 4750 60  0000 C CNN
-F 1 "FILTER" H 6100 4500 60  0000 C CNN
-F 2 "RP_KiCAD_Libs:C1608_WP" H 6100 4600 60  0001 C CNN
-F 3 "" H 6100 4600 60  0000 C CNN
-	1    6100 4600
-	1    0    0    -1
-$EndComp
-$Comp
 L C C4
 U 1 1 58D1AA3F
@@
 	5450 4800 7250 4800
 Wire Wire Line
-	5750 4600 5300 4600
+	5300 4600 6550 4600
 $Comp
 L R R8
@@
 Wire Wire Line
 	6950 4600 6850 4600
-Wire Wire Line
-	6550 4600 6450 4600
 Connection ~ 5600 4800
 $Comp
@@
 	1    0    0    -1
 $EndComp
+Wire Wire Line
+	5600 1950 5600 2000
+Wire Wire Line
+	5600 2300 5600 2350
+Wire Wire Line
+	5600 2700 5600 2750
+Wire Wire Line
+	5600 3050 5600 3100
+Wire Wire Line
+	5600 4000 5600 4050
+Wire Wire Line
+	5600 3650 5600 3700
+Wire Wire Line
+	5600 4750 5600 4800
+Wire Wire Line
+	5600 4400 5600 4450
 $EndSCHEMATC
