File: KiCAD_Projects/SSL_BLDC_ver0.0/SSL_BLDC_ver0.0.sch (KiCad schematic (older format))
At the start: 39 parts, among them P1 CONN_01X04, P2 CONN_01X04, P5 CONN_01X06, P6 CONN_01X02, Q1 MOSFET_N, Q2 MOSFET_N, Q3 MOSFET_N, Q4 MOSFET_N, Q5 MOSFET_N, Q6 MOSFET_N, SW1 SW_PUSH, U1 STM32F103_48, U2 NCP1117ST33T3G, U3 MAX3051, U4 NCP1117ST50T3G, X2 CRYSTAL

Commit message: bldc
Parts:
- removed D11: DIODE, Diodes_SMD:SMA_Standard, symbol DIODE
- removed U2: NCP1117ST33T3G, TO_SOT_Packages_SMD:SOT-223_reg, symbol NCP1117ST33T3G
- added C12, C14, C17: 0.1u, RP_KiCAD_Libs:C1608_WP_S, symbol C
- added C13: 4.7u, RP_KiCAD_Libs:C3216_S, symbol C
- added C15: 2.2u, RP_KiCAD_Libs:C3216_S, symbol C
- added C16, C28: 1u, RP_KiCAD_Libs:C1608_WP_S, symbol C
- added D3: LED, LEDs:LED_0805, symbol LED
- added ME1: AS504x, Housings_SSOP:SSOP-16_5.3x6.2mm_Pitch0.65mm, symbol AS504x
- added P3: CONN_02X04, symbol CONN_02X04
- added P4, P8: CONN_01X06, RP_KiCAD_Connector:ZH_6T, symbol CONN_01X06
- added P7, P9: CONN_01X02, Pin_Headers:Pin_Header_Straight_1x02, symbol CONN_01X02
- added R10, R12, R14, R16: 4.7k, RP_KiCAD_Libs:C1608_WP_S, symbol R
- added R11, R13, R15, R17: 1k, RP_KiCAD_Libs:C1608_WP_S, symbol R
- added R36: 100, RP_KiCAD_Libs:C1608_WP_S, symbol R
- added R9: 100, RP_KiCAD_Libs:C3216_S, symbol R
- added SW5, SW6: SW_PUSH, Buttons_Switches_SMD:SW_SPST_EVQPE1, symbol SW_PUSH
- added U2: DRV8305, Housings_QFP:TQFP-48-1EP_7x7mm_Pitch0.5mm, symbol DRV8305
- C1: value 0.1u -> 1u; footprint RP_KiCAD_Libs:C1608_WP -> RP_KiCAD_Libs:C1608_WP_S
- C10, C11, C4, C5, C6, C8, C9, R1, R3, R4, R5: footprint RP_KiCAD_Libs:C1608_WP -> RP_KiCAD_Libs:C1608_WP_S
- C2: value 4.7u -> 1u; footprint RP_KiCAD_Libs:C2012 -> RP_KiCAD_Libs:C1608_WP_S
- C3, C7: footprint RP_KiCAD_Libs:C2012 -> RP_KiCAD_Libs:C3216_S
- R2: value 10k -> 100; footprint RP_KiCAD_Libs:C1608_WP -> RP_KiCAD_Libs:C1608_WP_S
- R6, R7, R8: value R -> 10m; footprint Resistors_SMD:R_2010 -> Resistors_SMD:R_2512
Connections:
- net labels added: +BATT, AS_3.3V, AS_ENC_A, AS_ENC_B, AS_GND, AS_SPI_MISO, AS_SPI_NSS_ENC, AS_SPI_SCK, BATT_V, CS_U, CS_V, CS_W, ENC_A, ENC_B, GATE_U_H, GATE_U_L, GATE_V_H, GATE_V_L, GATE_W_H, GATE_W_L, GD_EN, GD_WAKE, GNDPWR, LED_A, LED_B, OUT_U, OUT_V, OUT_W, PWGD, PWM_U_H, PWM_U_L, PWM_V_H, PWM_V_L, PWM_W_H, PWM_W_L, SPI_MISO, SPI_MOSI, SPI_NSS_ENC, SPI_NSS_GD, SPI_SCK, SWO, S_U_L, S_V_L, S_W_L, VS_U, VS_V, VS_W, nFALUT
- net labels removed: +12V, BOOT0
- wire segments 17 -> 71
- no-connect marks 0 -> 9
Other:
- note removed: "LED"
- moved on the sheet: C10, C3, C4, C5, C6, C7, C8, C9, D1, D2, Q1, Q2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
