File: KiCAD_Projects/SSL_BST_ver1.0/SSL_BST_ver1.0.sch (KiCad schematic (older format))
At the start: 45 parts, among them P1 CONN_01X04, P2 CONN_01X04, P5 CONN_01X06, P6 CONN_01X02, Q1 MOSFET_N, Q2 MOSFET_N, Q3 MOSFET_N, Q4 MOSFET_N, Q5 MOSFET_N, Q6 MOSFET_N, SW1 SW_PUSH, U1 STM32F103_48, U2 NCP5359, U3 MAX3051, U4 NCP1117ST50T3G, U5 NCP5359, U6 OPTO-TRANSISTOR4, X1 ceralock

Commit message: BLMD_ver0.1仮
Parts:
- removed D11: DIODE, Diodes_SMD:SMA_Standard, symbol DIODE
- removed D3, D4: DIODE, Diodes_SMD:MiniMELF_Standard, symbol DIODE
- removed Q1, Q2, Q3, Q4, Q5, Q6: MOSFET_N, TO_SOT_Packages_SMD:SOT-428_GDS_compact, symbol MOSFET_N
- removed SW1: SW_PUSH, Buttons_Switches_SMD:SW_SPST_EVQPE1, symbol SW_PUSH
- removed U1: STM32F103_48, Housings_QFP:LQFP-48_7x7mm_Pitch0.5mm, symbol STM32F103_48-RESCUE-STM32F103_mini
- added C12, C13, C15, C16, C19, C20, C4, C5: 4.7u, RP_KiCAD_Libs:C3216_S, symbol C
- added C14: 20nF, RP_KiCAD_Libs:C1608_WP_S, symbol C
- added C17, C18: 470u, Capacitors_ThroughHole:C_Radial_D10_L13_P5, symbol C
- added D3: D, RP_KiCAD_Libs:C3216_S, symbol D
- added D4: BD9C601EFJ, Housings_SOIC:SOIC-8_3.9x4.9mm_Pitch1.27mm, symbol BD9C601EFJ
- added L1: 3.3uH, Inductors:NR4018, symbol L
- added Q1, Q2, Q3, Q4, Q5: Q_NMOS_GDS, TO_SOT_Packages_SMD:DFN56, symbol Q_NMOS_GDS
- added Q6, Q7, Q8, Q9: Q_PMOS_GDS, TO_SOT_Packages_SMD:DFN56, symbol Q_PMOS_GDS
- added R12, R13, R17: 1k, RP_KiCAD_Libs:C1608_WP_S, symbol R
- added R14: 1m, RP_KiCAD_Libs:C1608_WP_S, symbol R
- added R15: 10k, RP_KiCAD_Libs:C1608_WP_S, symbol R
- added R16: 15k, RP_KiCAD_Libs:C1608_WP_S, symbol R
- added U1: STM32F103_48, Housings_QFP:LQFP-48_7x7mm_Pitch0.5mm, symbol STM32F103_48
- C2: footprint RP_KiCAD_Libs:C2012 -> RP_KiCAD_Libs:C3216_S
- P1, P2: footprint RP_KiCAD_Connector:XA_4T -> Connectors_JST_PH:Connectors_JST_B4B-PH-K
- gave numbers to parts that had none: 2
Connections:
- net labels added: CS_N, CS_P, DCDC_EN, LED_1, OUT_EN, PW_OUT
- wire segments 62 -> 117
Other:
- note removed: "LED"
- moved on the sheet: C10, C2, C6, C7, C8, C9, D1, D2, R3, R4
